File: miniPCB/04/A/04A-005/X04A-005-B-XB.brd (EAGLE design)
At the start: 100 x 100 mm, 97 parts

Commit message: NM.14JAN2023
Parts:
- moved TP18 0.50 mm to (33.5, 93.0)
- moved TP28 0.50 mm to (83.5, 43.0)
- moved TP3 0.50 mm to (33.5, 43.0)
- moved TP38 0.50 mm to (83.5, 93.0)
Other:
- board text added: "INVERTING AMPLIFIER"
