File: miniPCB/04/A/04A-005/04A-005-A101.brd (EAGLE design)
At the start: 100 x 100 mm, 112 parts, among them J1 JUMPER, J2 JUMPER, J3 JUMPER, J4 JUMPER

Commit message: NM.07SEP2023
Parts:
- added R29, R30, R31, R33, R34, R36: (no value), minipcb:0207/10
- added R32, R35: (no value), minipcb:TRIM_0100
- R12, R19: device minipcb:TRIM_0100 -> minipcb:0207/10
- R14, R17, R23, R8: device minipcb:0207/10 -> minipcb:TRIM_0100
- moved R16 89.3 mm to (9.50, 68.5), turned to 0 degrees
- moved R15 81.5 mm to (34.5, 74.0), turned to 90 degrees
- moved R26 81.3 mm to (89.0, 12.5), turned to 0 degrees
- moved R25 79.7 mm to (59.5, 18.5), turned to 0 degrees
- moved R24 69.6 mm to (84.5, 24.0), turned to 90 degrees
- moved R27 67.3 mm to (90.5, 7.00), turned to 180 degrees
- moved R9 54.7 mm to (40.5, 7.00)
- moved R18 53.3 mm to (40.5, 57.0)
- moved R8 43.7 mm to (39.0, 12.5), turned to 0 degrees
- moved R10 38.7 mm to (27.0, 54.5)
- moved R19 38.5 mm to (77.0, 4.50)
- moved R11 34.7 mm to (27.0, 60.0)
- moved R17 31.2 mm to (39.0, 62.5), turned to 0 degrees
- moved R14 30.4 mm to (27.5, 93.0), turned to 180 degrees
- moved TP14 27.7 mm to (14.5, 72.5)
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Connections:
- new net N$1: R8.2, R9.1
- new net N$2: R17.2, R18.1
- new net N$3: R26.2, R27.1
- new net N$4: R35.2, R36.1
- net GND1: now also R13.1, R16.1; no longer R11.1, R14.1
- net GND2: now also R22.1, R25.1; no longer R18.1, R21.1
- net GND3: now also R31.1, R34.1; no longer R25.1, R28.1
- net IN-DC1: now also R10.2; no longer R8.2
- net IN-DC2: now also R19.2; no longer R15.2
- net IN-DC3: now also R28.2; no longer R22.2
- net OUT: now also R9.2
- net OUT1: now also R11.2, R16.2, R18.2; no longer R14.2, R9.2
- net OUT2: now also R20.2, R25.2, R27.2; no longer R16.2, R21.2
- net OUT3: now also R29.2, R34.2, R36.2; no longer R23.2, R28.2
- net P1.2: now also R12.1, R14.3; no longer R10.1, R12.3
- net P1.4: now also R13.2, R14.1; no longer R11.2, R12.1
- net P1.5: now also R21.1, R23.3; no longer R17.1, R19.3
- net P1.6: now also R22.2, R23.1; no longer R18.2, R19.1
- net P1.7: now also R30.1, R32.3; no longer R24.1, R26.3
- net P1.8: now also R31.2, R32.1; no longer R25.2, R26.1
- net V+1: now also R12.2; no longer R10.2
- net V+2: now also R21.2; no longer R17.2
- net V+3: now also R30.2; no longer R24.2
- net VFB: now also R8.1
- net VFB1: now also R10.1, R11.1, R17.1; no longer R8.1, R9.1
- net VFB2: now also R19.1, R20.1, R26.1; no longer R15.1, R16.1
- net VFB3: now also R28.1, R29.1, R35.1; no longer R22.1, R23.1
- net VR1: now also R14.2; no longer R12.2
- net VR2: now also R23.2; no longer R19.2
- net VR3: now also R32.2; no longer R26.2
- net VREF+1: now also R15.1; no longer R13.1
- net VREF+2: now also R24.1; no longer R20.1
- net VREF+3: now also R33.1; no longer R27.1
- net VREF1: now also R15.2; no longer R13.2
- net VREF2: now also R24.2; no longer R20.2
- net VREF3: now also R33.2; no longer R27.2
Routing:
- net VFB3: track 23.5 -> 39.1 mm
- net VFB2: track 23.5 -> 39.1 mm
- net VFB1: track 23.5 -> 39.1 mm
- net VFB: track 23.5 -> 39.1 mm
- net OUT2: track 45.1 -> 59.7 mm
- net OUT1: track 45.1 -> 59.7 mm
- net OUT3: track 45.1 -> 59.7 mm
- net OUT: track 45.1 -> 59.7 mm
- net N$4: track 0.00 -> 7.16 mm
- net N$3: track 0.00 -> 7.16 mm
- net N$2: track 0.00 -> 7.16 mm
- net N$1: track 0.00 -> 7.16 mm
Other:
- board text added: "R8"
- board text added: "R9"
