File: miniPCB/04/A/04A-005/04A-005.brd (EAGLE design)
At the start: 24 parts

Commit message: NM.14JAN2023
Parts:
- moved TP1 31.1 mm to (11.0, 6.50)
- moved TP9 17.0 mm to (23.0, 35.0), turned to 90 degrees
- moved TP6 14.8 mm to (28.5, 35.0), turned to 90 degrees
- moved TP4 13.5 mm to (29.5, 5.00)
- moved TP3 12.0 mm to (33.5, 43.5), turned to 180 degrees
- moved C1 11.1 mm to (42.5, 34.5), turned to 0 degrees
- moved C4 8.56 mm to (32.5, 35.0)
- moved TP10 7.52 mm to (2.50, 9.50)
- moved TP2 7.43 mm to (16.0, 43.5), turned to 180 degrees
- moved TP8 7.38 mm to (13.5, 10.5)
- moved TP7 6.95 mm to (38.5, 29.0)
- moved TP5 4.03 mm to (38.5, 19.0)
- moved R1 3.16 mm to (7.50, 43.0)
- moved R3 2.69 mm to (42.0, 43.0)
- moved C2 1.80 mm to (17.0, 30.5)
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Routing:
- net IN: track 34.6 -> 10.4 mm
- net VFB: track 33.6 -> 19.3 mm
- net OUT: track 33.0 -> 22.9 mm
- net N$1: track 38.7 -> 28.8 mm
- net P1.1: track 18.7 -> 9.91 mm
- net VREF: track 26.1 -> 18.1 mm
- net V+: track 69.6 -> 65.2 mm
- net P1.3: track 14.0 -> 10.4 mm
- net N$2: track 23.9 -> 21.5 mm

Commit message: NM.14JAN2023
Parts:
- moved TP3 0.50 mm to (33.5, 43.0)
Other:
- board text added: "INVERTING AMPLIFIER"
Changed lines of the file:
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@@
 <text x="9.50000625" y="7.7700125" size="1.499996875" layer="125" font="vector" ratio="12">TP1</text>
 <text x="17.499990625" y="42.229990625" size="1.499996875" layer="125" font="vector" ratio="12" rot="R180">TP2</text>
-<text x="35.00000625" y="42.229990625" size="1.499996875" layer="125" font="vector" ratio="12" rot="R180">TP3</text>
+<text x="35.00000625" y="41.729990625" size="1.499996875" layer="125" font="vector" ratio="12" rot="R180">TP3</text>
 <text x="27.99999375" y="6.269990625" size="1.499996875" layer="125" font="vector" ratio="12">TP4</text>
 <text x="37.000003125" y="20.2699875" size="1.499996875" layer="125" font="vector" ratio="12">TP5</text>
@@
 <text x="1.999996875" y="10.77000625" size="1.499996875" layer="125" font="vector" ratio="12">TP10</text>
 <text x="19.5000125" y="21.000009375" size="1.499996875" layer="125" font="vector" ratio="12" rot="R90">U1</text>
+<text x="45" y="44.5" size="1.778" layer="22" font="vector" ratio="12" rot="MR0">INVERTING AMPLIFIER</text>
 </plain>
 <attributes>
@@
 <attribute name="NAME" x="17.5" y="42.23" size="1.5" layer="25" font="vector" ratio="12" rot="R180"/>
 </element>
-<element name="TP3" library="minipcb" package="PINS_1_TESTPOINT_KE5000_NOTEXT" value="" x="33.5" y="43.5" smashed="yes" rot="R180">
-<attribute name="NAME" x="35" y="42.23" size="1.5" layer="25" font="vector" ratio="12" rot="R180"/>
+<element name="TP3" library="minipcb" package="PINS_1_TESTPOINT_KE5000_NOTEXT" value="" x="33.5" y="43" smashed="yes" rot="R180">
+<attribute name="NAME" x="35" y="41.73" size="1.5" layer="25" font="vector" ratio="12" rot="R180"/>
 </element>
 <element name="TP7" library="minipcb" package="PINS_1_TESTPOINT_KE5000_NOTEXT" value="" x="38.5" y="29" smashed="yes">
@@
 <contactref element="R3" pad="2"/>
 <contactref element="TP3" pad="1"/>
-<wire x1="27.5" y1="43" x2="31" y2="43" width="0.5" layer="16"/>
-<wire x1="31" y1="43" x2="31.5" y2="43.5" width="0.5" layer="16"/>
-<wire x1="31.5" y1="43.5" x2="33.5" y2="43.5" width="0.5" layer="16"/>
-<wire x1="33.5" y1="43.5" x2="35" y2="43.5" width="0.5" layer="16"/>
-<wire x1="35" y1="43.5" x2="35.5" y2="43" width="0.5" layer="16"/>
-<wire x1="35.5" y1="43" x2="37" y2="43" width="0.5" layer="16"/>
+<wire x1="27.5" y1="43" x2="33.5" y2="43" width="0.5" layer="16"/>
+<wire x1="33.5" y1="43" x2="37" y2="43" width="0.5" layer="16"/>
 </signal>
 <signal name="N$1">

Commit message: NM.16JAN2023
Parts:
- moved C3 7.38 mm to (37.0, 11.5), turned to 0 degrees
- moved TP2 0.50 mm to (16.0, 43.0)
Connections:
- removed net N$2: C3.2, R6.1, TP5.1, U1.3
- new net N$3: C3.1, R6.1, TP5.1, U1.3
- net GND: now also C3.2; no longer C3.1
Routing:
- net N$3: track 0.00 -> 23.1 mm
- net N$2: track 21.5 -> 0.00 mm
- net OUT: track 22.9 -> 28.8 mm
Changed lines of the file:
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@@
 <text x="38" y="37.000003125" size="1.499996875" layer="125" font="vector" ratio="13">C1</text>
 <text x="14.499996875" y="26" size="1.499996875" layer="125" font="vector" ratio="13" rot="R90">C2</text>
-<text x="35.00000625" y="12.5" size="1.499996875" layer="125" font="vector" ratio="13" rot="R180">C3</text>
+<text x="32.49999375" y="14" size="1.499996875" layer="125" font="vector" ratio="13">C3</text>
 <text x="29.999990625" y="30.499990625" size="1.499996875" layer="125" font="vector" ratio="13" rot="R90">C4</text>
 <text x="5.4999875" y="26" size="1.499996875" layer="125" font="vector" ratio="13" rot="R90">C5</text>
@@
 <text x="32.5000125" y="20.500009375" size="1.499996875" layer="125" font="vector" ratio="12" rot="R90">R6</text>
 <text x="9.50000625" y="7.7700125" size="1.499996875" layer="125" font="vector" ratio="12">TP1</text>
-<text x="17.499990625" y="42.229990625" size="1.499996875" layer="125" font="vector" ratio="12" rot="R180">TP2</text>
+<text x="17.499990625" y="41.729990625" size="1.499996875" layer="125" font="vector" ratio="12" rot="R180">TP2</text>
 <text x="35.00000625" y="41.729990625" size="1.499996875" layer="125" font="vector" ratio="12" rot="R180">TP3</text>
 <text x="27.99999375" y="6.269990625" size="1.499996875" layer="125" font="vector" ratio="12">TP4</text>
@@
 <attribute name="VALUE" x="26" y="12.5" size="1.5" layer="27" font="vector" ratio="13" rot="R180"/>
 </element>
-<element name="C3" library="minipcb" package="C050-024X044" value="" x="30.5" y="15" smashed="yes" rot="R180">
-<attribute name="NAME" x="35" y="12.5" size="1.5" layer="25" font="vector" ratio="13" rot="R180"/>
-<attribute name="VALUE" x="26" y="17.5" size="1.5" layer="27" font="vector" ratio="13"/>
+<element name="C3" library="minipcb" package="C050-024X044" value="" x="37" y="11.5" smashed="yes">
+<attribute name="NAME" x="32.5" y="14" size="1.5" layer="25" font="vector" ratio="13"/>
+<attribute name="VALUE" x="41.5" y="9" size="1.5" layer="27" font="vector" ratio="13" rot="R180"/>
 </element>
 <element name="R6" library="minipcb" package="0207/10" value="" x="34.5" y="24" smashed="yes" rot="R90">
@@
 <attribute name="NAME" x="2" y="10.77" size="1.5" layer="25" font="vector" ratio="12"/>
 </element>
-<element name="TP2" library="minipcb" package="PINS_1_TESTPOINT_KE5000_NOTEXT" value="" x="16" y="43.5" smashed="yes" rot="R180">
-<attribute name="NAME" x="17.5" y="42.23" size="1.5" layer="25" font="vector" ratio="12" rot="R180"/>
+<element name="TP2" library="minipcb" package="PINS_1_TESTPOINT_KE5000_NOTEXT" value="" x="16" y="43" smashed="yes" rot="R180">
+<attribute name="NAME" x="17.5" y="41.73" size="1.5" layer="25" font="vector" ratio="12" rot="R180"/>
 </element>
 <element name="TP3" library="minipcb" package="PINS_1_TESTPOINT_KE5000_NOTEXT" value="" x="33.5" y="43" smashed="yes" rot="R180">
@@
 </polygon>
 <contactref element="U1" pad="4"/>
-<contactref element="C3" pad="1"/>
 <contactref element="R3" pad="1"/>
 <contactref element="C4" pad="2"/>
@@
 <via x="6.5" y="17" extent="1-16" drill="0.5"/>
 <via x="25" y="8" extent="1-16" drill="0.5"/>
-<via x="15" y="8" extent="1-16" drill="0.5"/>
-<via x="30.5" y="12" extent="1-16" drill="0.5"/>
+<via x="26.5" y="13.5" extent="1-16" drill="0.5"/>
 <via x="28" y="8" extent="1-16" drill="0.5"/>
 <via x="16" y="13.5" extent="1-16" drill="0.5"/>
@@
 <via x="3.5" y="21" extent="1-16" drill="0.5"/>
 <via x="3.5" y="24.5" extent="1-16" drill="0.5"/>
-<via x="11" y="10" extent="1-16" drill="0.5"/>
 <via x="19.5" y="11.5" extent="1-16" drill="0.5"/>
 <via x="23.5" y="11.5" extent="1-16" drill="0.5"/>
-<via x="18.5" y="2.5" extent="1-16" drill="0.5"/>
+<contactref element="C3" pad="2"/>
+<via x="20.5" y="8" extent="1-16" drill="0.5"/>
+<via x="20.5" y="5" extent="1-16" drill="0.5"/>
+<via x="18.5" y="2" extent="1-16" drill="0.5"/>
+<via x="36" y="16.5" extent="1-16" drill="0.5"/>
+<via x="36" y="14.5" extent="1-16" drill="0.5"/>
+<via x="31.5" y="14.5" extent="1-16" drill="0.5"/>
+<via x="3.5" y="7.5" extent="1-16" drill="0.5"/>
+<via x="3.5" y="5" extent="1-16" drill="0.5"/>
 </signal>
 <signal name="NC">
@@
 <wire x1="19" y1="15" x2="19" y2="13" width="0.5" layer="16"/>
 <wire x1="19" y1="13" x2="16.5" y2="10.5" width="0.5" layer="16"/>
-<wire x1="12.7" y1="2.54" x2="12.7" y2="4.7" width="0.5" layer="16"/>
-<wire x1="12.7" y1="4.7" x2="13.5" y2="5.5" width="0.5" layer="16"/>
-<wire x1="13.5" y1="5.5" x2="13.5" y2="10.5" width="0.5" layer="16"/>
 <wire x1="13.5" y1="10.5" x2="16.5" y2="10.5" width="0.5" layer="16"/>
+<wire x1="12.7" y1="2.54" x2="17.04" y2="2.54" width="0.5" layer="16"/>
+<wire x1="17.04" y1="2.54" x2="19" y2="4.5" width="0.5" layer="16"/>
+<wire x1="19" y1="4.5" x2="19" y2="8" width="0.5" layer="16"/>
+<wire x1="19" y1="8" x2="16.5" y2="10.5" width="0.5" layer="16"/>
 </signal>
 <signal name="VFB">
@@
 <contactref element="R1" pad="1"/>
 <contactref element="TP2" pad="1"/>
-<wire x1="12.5" y1="43" x2="14" y2="43" width="0.5" layer="16"/>
-<wire x1="14" y1="43" x2="14.5" y2="43.5" width="0.5" layer="16"/>
-<wire x1="14.5" y1="43.5" x2="16" y2="43.5" width="0.5" layer="16"/>
-<wire x1="16" y1="43.5" x2="18" y2="43.5" width="0.5" layer="16"/>
-<wire x1="18" y1="43.5" x2="18.5" y2="43" width="0.5" layer="16"/>
-<wire x1="18.5" y1="43" x2="22.5" y2="43" width="0.5" layer="16"/>
+<wire x1="12.5" y1="43" x2="16" y2="43" width="0.5" layer="16"/>
+<wire x1="16" y1="43" x2="22.5" y2="43" width="0.5" layer="16"/>
 </signal>
 <signal name="VREF">
@@
 <wire x1="34.5" y1="34.5" x2="40" y2="34.5" width="0.5" layer="16"/>
 </signal>
-<signal name="N$2">
-<contactref element="U1" pad="3"/>
-<contactref element="R6" pad="1"/>
-<contactref element="C3" pad="2"/>
-<contactref element="TP5" pad="1"/>
-<wire x1="26.27" y1="20.19" x2="26.27" y2="21.77" width="0.5" layer="16"/>
-<wire x1="26.27" y1="21.77" x2="27" y2="22.5" width="0.5" layer="16"/>
-<wire x1="27" y1="22.5" x2="31" y2="22.5" width="0.5" layer="16"/>
-<wire x1="31" y1="22.5" x2="34.5" y2="19" width="0.5" layer="16"/>
-<wire x1="34.5" y1="19" x2="38.5" y2="19" width="0.5" layer="16"/>
-<wire x1="28" y1="15" x2="26.27" y2="16.73" width="0.5" layer="16"/>
-<wire x1="26.27" y1="16.73" x2="26.27" y2="20.19" width="0.5" layer="16"/>
-</signal>
 <signal name="IN">
 <contactref element="R4" pad="2"/>
@@
 <wire x1="10.16" y1="2.54" x2="10.16" y2="5.66" width="0.5" layer="16"/>
 <wire x1="10.16" y1="5.66" x2="11" y2="6.5" width="0.5" layer="16"/>
-<wire x1="11" y1="6.5" x2="15" y2="6.5" width="0.5" layer="1"/>
-<wire x1="15" y1="6.5" x2="16.5" y2="5" width="0.5" layer="1"/>
+<wire x1="11" y1="6.5" x2="15" y2="6.5" width="0.5" layer="16"/>
+<wire x1="15" y1="6.5" x2="16.5" y2="5" width="0.5" layer="16"/>
+</signal>
+<signal name="N$3">
+<contactref element="R6" pad="1"/>
+<contactref element="TP5" pad="1"/>
+<wire x1="34.5" y1="19" x2="38.5" y2="19" width="0.5" layer="16"/>
+<contactref element="U1" pad="3"/>
+<wire x1="26.27" y1="20.19" x2="26.27" y2="21.77" width="0.5" layer="16"/>
+<wire x1="26.27" y1="21.77" x2="27" y2="22.5" width="0.5" layer="16"/>
+<wire x1="27" y1="22.5" x2="31" y2="22.5" width="0.5" layer="16"/>
+<contactref element="C3" pad="1"/>
+<wire x1="34.5" y1="19" x2="34.5" y2="11.5" width="0.5" layer="16"/>
+<wire x1="31" y1="22.5" x2="34.5" y2="19" width="0.5" layer="16"/>
 </signal>
 </signals>

Commit message: NM.04FEB2023
Parts:
- C1, C5: device minipcb:C050-024X044 -> minipcb:C5MM
Connections:
- net GND: now also C1.-, C5.-; no longer C1.2, C5.2
- net N$1: now also C1.+; no longer C1.1
- net V+: now also C5.+; no longer C5.1
Changed lines of the file:
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@@
 <board>
 <plain>
-<text x="38" y="37.000003125" size="1.499996875" layer="125" font="vector" ratio="13">C1</text>
+<text x="44.5" y="27.500003125" size="1.499996875" layer="125" font="vector" ratio="13">C1</text>
 <text x="14.499996875" y="26" size="1.499996875" layer="125" font="vector" ratio="13" rot="R90">C2</text>
 <text x="32.49999375" y="14" size="1.499996875" layer="125" font="vector" ratio="13">C3</text>
 <text x="29.999990625" y="30.499990625" size="1.499996875" layer="125" font="vector" ratio="13" rot="R90">C4</text>
-<text x="5.4999875" y="26" size="1.499996875" layer="125" font="vector" ratio="13" rot="R90">C5</text>
+<text x="10" y="24.0000125" size="1.499996875" layer="125" font="vector" ratio="13">C5</text>
 <text x="16.999990625" y="17.499990625" size="1.499996875" layer="125" font="vector" ratio="13">C6</text>
 <text x="11.000003125" y="40.99999375" size="1.499996875" layer="125" font="vector" ratio="12" rot="R180">R1</text>
 <text x="29.499990625" y="40.49999375" size="1.499996875" layer="125" font="vector" ratio="12" rot="R180">R2</text>
-<text x="45.500009375" y="40.99999375" size="1.499996875" layer="125" font="vector" ratio="12" rot="R180">R3</text>
+<text x="48.000009375" y="40.99999375" size="1.499996875" layer="125" font="vector" ratio="12" rot="R180">R3</text>
 <text x="25" y="2.99999375" size="1.499996875" layer="125" font="vector" ratio="12" rot="R180">R4</text>
 <text x="25" y="8.500009375" size="1.499996875" layer="125" font="vector" ratio="12" rot="R180">R5</text>
@@
 <text x="35.00000625" y="41.729990625" size="1.499996875" layer="125" font="vector" ratio="12" rot="R180">TP3</text>
 <text x="27.99999375" y="6.269990625" size="1.499996875" layer="125" font="vector" ratio="12">TP4</text>
-<text x="37.000003125" y="20.2699875" size="1.499996875" layer="125" font="vector" ratio="12">TP5</text>
+<text x="37" y="20.5" size="1.499996875" layer="125" font="vector" ratio="12">TP5</text>
 <text x="27.22999375" y="33.500009375" size="1.499996875" layer="125" font="vector" ratio="12" rot="R90">TP6</text>
-<text x="37.000003125" y="30.26999375" size="1.499996875" layer="125" font="vector" ratio="12">TP7</text>
+<text x="37.000003125" y="25.76999375" size="1.499996875" layer="125" font="vector" ratio="12">TP7</text>
 <text x="12" y="11.770003125" size="1.499996875" layer="125" font="vector" ratio="12">TP8</text>
 <text x="21.73000625" y="33.500009375" size="1.499996875" layer="125" font="vector" ratio="12" rot="R90">TP9</text>
@@
 <attribute name="VALUE" x="19.5" y="35" size="1.5" layer="27" font="vector" ratio="13" rot="R270"/>
 </element>
-<element name="C5" library="minipcb" package="C050-024X044" value="" x="8" y="30.5" smashed="yes" rot="R90">
-<attribute name="NAME" x="5.5" y="26" size="1.5" layer="25" font="vector" ratio="13" rot="R90"/>
+<element name="C5" library="minipcb" package="C5MM" value="" x="8" y="30.5" smashed="yes" rot="R90">
+<attribute name="NAME" x="10" y="24" size="1.5" layer="25" font="vector" ratio="13"/>
 <attribute name="VALUE" x="10.5" y="35" size="1.5" layer="27" font="vector" ratio="13" rot="R270"/>
 </element>
@@
 </element>
 <element name="R3" library="minipcb" package="0207/10" value="" x="42" y="43" smashed="yes" rot="R180">
-<attribute name="NAME" x="45.5" y="41" size="1.5" layer="25" font="vector" ratio="12" rot="R180"/>
+<attribute name="NAME" x="48" y="41" size="1.5" layer="25" font="vector" ratio="12" rot="R180"/>
 <attribute name="VALUE" x="42" y="43" size="1.5" layer="27" font="vector" ratio="12" align="center"/>
 </element>
@@
 <attribute name="NAME" x="29.5" y="40.5" size="1.5" layer="25" font="vector" ratio="12" rot="R180"/>
 </element>
-<element name="C1" library="minipcb" package="C050-024X044" value="" x="42.5" y="34.5" smashed="yes">
-<attribute name="NAME" x="38" y="37" size="1.5" layer="25" font="vector" ratio="13"/>
+<element name="C1" library="minipcb" package="C5MM" value="" x="42.5" y="34.5" smashed="yes">
+<attribute name="NAME" x="44.5" y="27.5" size="1.5" layer="25" font="vector" ratio="13"/>
 <attribute name="VALUE" x="47" y="32" size="1.5" layer="27" font="vector" ratio="13" rot="R180"/>
 </element>
@@
 </element>
 <element name="TP7" library="minipcb" package="PINS_1_TESTPOINT_KE5000_NOTEXT" value="" x="38.5" y="29" smashed="yes">
-<attribute name="NAME" x="37" y="30.27" size="1.5" layer="25" font="vector" ratio="12"/>
+<attribute name="NAME" x="37" y="25.77" size="1.5" layer="25" font="vector" ratio="12"/>
 </element>
 <element name="TP5" library="minipcb" package="PINS_1_TESTPOINT_KE5000_NOTEXT" value="" x="38.5" y="19" smashed="yes">
-<attribute name="NAME" x="37" y="20.27" size="1.5" layer="25" font="vector" ratio="12"/>
+<attribute name="NAME" x="37" y="20.5" size="1.5" layer="25" font="vector" ratio="12"/>
 </element>
 </elements>
@@
 <contactref element="P1-" pad="1"/>
 <contactref element="C2" pad="2"/>
-<contactref element="C5" pad="2"/>
-<contactref element="C1" pad="2"/>
+<contactref element="C5" pad="-"/>
+<contactref element="C1" pad="-"/>
 <polygon width="0.6" layer="1">
 <vertex x="1" y="1"/>
@@
 <via x="3.5" y="7.5" extent="1-16" drill="0.5"/>
 <via x="3.5" y="5" extent="1-16" drill="0.5"/>
+<wire x1="45" y1="34.5" x2="47" y2="43" width="0" layer="19" extent="1-1"/>
+<wire x1="36" y1="36" x2="45" y2="34.5" width="0" layer="19" extent="1-1"/>
+<wire x1="36" y1="33" x2="36" y2="36" width="0" layer="19" extent="1-1"/>
+<wire x1="32.5" y1="37.5" x2="36" y2="36" width="0" layer="19" extent="1-1"/>
+<wire x1="26.5" y1="39" x2="32.5" y2="37.5" width="0" layer="19" extent="1-1"/>
+<wire x1="23.5" y1="39" x2="26.5" y2="39" width="0" layer="19" extent="1-1"/>
+<wire x1="31.5" y1="28.5" x2="36" y2="33" width="0" layer="19" extent="1-1"/>
+<wire x1="32" y1="24" x2="31.5" y2="28.5" width="0" layer="19" extent="1-1"/>
+<wire x1="28.81" y1="20.19" x2="32" y2="24" width="0" layer="19" extent="1-1"/>
+<wire x1="31.5" y1="18.5" x2="28.81" y2="20.19" width="0" layer="19" extent="1-1"/>
+<wire x1="31.5" y1="14.5" x2="31.5" y2="18.5" width="0" layer="19" extent="1-1"/>
+<wire x1="36" y1="14.5" x2="31.5" y2="14.5" width="0" layer="19" extent="1-1"/>
+<wire x1="36" y1="16.5" x2="36" y2="14.5" width="0" layer="19" extent="1-1"/>
+<wire x1="39.5" y1="11.5" x2="36" y2="14.5" width="0" layer="19" extent="1-1"/>
+<wire x1="26" y1="24" x2="28.81" y2="20.19" width="0" layer="19" extent="1-1"/>
+<wire x1="26.5" y1="13.5" x2="31.5" y2="14.5" width="0" layer="19" extent="1-1"/>
+<wire x1="23.5" y1="11.5" x2="26.5" y2="13.5" width="0" layer="19" extent="1-1"/>
+<wire x1="25" y1="8" x2="23.5" y2="11.5" width="0" layer="19" extent="1-1"/>
+<wire x1="28" y1="8" x2="25" y2="8" width="0" layer="19" extent="1-1"/>
+<wire x1="19.5" y1="11.5" x2="23.5" y2="11.5" width="0" layer="19" extent="1-1"/>
+<wire x1="20.5" y1="8" x2="19.5" y2="11.5" width="0" layer="19" extent="1-1"/>
+<wire x1="20.5" y1="5" x2="20.5" y2="8" width="0" layer="19" extent="1-1"/>
+<wire x1="18.5" y1="2" x2="20.5" y2="5" width="0" layer="19" extent="1-1"/>
+<wire x1="16" y1="13.5" x2="19.5" y2="11.5" width="0" layer="19" extent="1-1"/>
+<wire x1="25" y1="32" x2="26.5" y2="39" width="0" layer="19" extent="1-1"/>
+<wire x1="17" y1="33" x2="25" y2="32" width="0" layer="19" extent="1-1"/>
+<wire x1="13.5" y1="29.5" x2="17" y2="33" width="0" layer="19" extent="1-1"/>
+<wire x1="11" y1="29.5" x2="13.5" y2="29.5" width="0" layer="19" extent="1-1"/>
+<wire x1="8" y1="33" x2="11" y2="29.5" width="0" layer="19" extent="1-1"/>
+<wire x1="6" y1="37" x2="8" y2="33" width="0" layer="19" extent="1-1"/>
+<wire x1="6" y1="40" x2="6" y2="37" width="0" layer="19" extent="1-1"/>
+<wire x1="3" y1="40" x2="6" y2="40" width="0" layer="19" extent="1-1"/>
+<wire x1="3" y1="37" x2="6" y2="37" width="0" layer="19" extent="1-1"/>
+<wire x1="3" y1="34" x2="3" y2="37" width="0" layer="19" extent="1-1"/>
+<wire x1="6.5" y1="24.5" x2="11" y2="29.5" width="0" layer="19" extent="1-1"/>
+<wire x1="3.5" y1="24.5" x2="6.5" y2="24.5" width="0" layer="19" extent="1-1"/>
+<wire x1="6.5" y1="21" x2="6.5" y2="24.5" width="0" layer="19" extent="1-1"/>
+<wire x1="3.5" y1="21" x2="6.5" y2="21" width="0" layer="19" extent="1-1"/>
+<wire x1="6.5" y1="17" x2="6.5" y2="21" width="0" layer="19" extent="1-1"/>
+<wire x1="3.5" y1="17" x2="6.5" y2="17" width="0" layer="19" extent="1-1"/>
+<wire x1="6.5" y1="13.5" x2="6.5" y2="17" width="0" layer="19" extent="1-1"/>
+<wire x1="3.5" y1="13.5" x2="6.5" y2="13.5" width="0" layer="19" extent="1-1"/>
+<wire x1="2.5" y1="9.5" x2="3.5" y2="13.5" width="0" layer="19" extent="1-1"/>
+<wire x1="3.5" y1="7.5" x2="2.5" y2="9.5" width="0" layer="19" extent="1-1"/>
+<wire x1="3.5" y1="5" x2="3.5" y2="7.5" width="0" layer="19" extent="1-1"/>
+<wire x1="2.54" y1="2.54" x2="3.5" y2="5" width="0" layer="19" extent="1-1"/>
+<wire x1="6.5" y1="5.5" x2="3.5" y2="5" width="0" layer="19" extent="1-1"/>
+<wire x1="6.5" y1="9" x2="3.5" y2="7.5" width="0" layer="19" extent="1-1"/>
+<wire x1="47.5" y1="5.5" x2="39.5" y2="11.5" width="0" layer="19" extent="1-1"/>
+<wire x1="47.5" y1="2.5" x2="47.5" y2="5.5" width="0" layer="19" extent="1-1"/>
+<wire x1="44" y1="2.5" x2="47.5" y2="2.5" width="0" layer="19" extent="1-1"/>
 </signal>
 <signal name="NC">
@@
 <contactref element="P1-" pad="2"/>
 <contactref element="C2" pad="1"/>
-<contactref element="C5" pad="1"/>
+<contactref element="C5" pad="+"/>
 <contactref element="R1" pad="2"/>
 <contactref element="U1" pad="8"/>
@@
 <signal name="N$1">
 <contactref element="R2" pad="2"/>
-<contactref element="C1" pad="1"/>
+<contactref element="C1" pad="+"/>
 <contactref element="C4" pad="1"/>
 <contactref element="U1" pad="5"/>

Commit message: NM.03SEP2023
Parts:
- removed P1-: (no value), minipcb:MINIPCB_5P_50X50MM
- added C7: (no value), minipcb:C050-024X044
- added J1: JUMPER, minipcb:PINS_2
- added P1: (no value), minipcb:PINS_1X5
- added R7, R9: (no value), minipcb:0207/10
- added R8: (no value), minipcb:TRIM_0100
- added U$1: MINIPCB_50X50, minipcb:MINIPCB_0P_50X50MM
- moved TP4 23.0 mm to (14.5, 22.5)
- moved C3 9.01 mm to (42.0, 19.0)
- moved TP8 7.38 mm to (20.0, 14.0), turned to 90 degrees
- moved TP1 7.28 mm to (18.0, 4.50)
- moved TP5 6.02 mm to (34.5, 14.5)
- moved C6 5.52 mm to (27.0, 14.5)
- moved R4 5.52 mm to (27.0, 4.50)
- moved R5 5.52 mm to (27.0, 10.0)
- moved TP7 5.15 mm to (41.0, 24.5)
- moved R1 4.47 mm to (9.50, 39.0)
- moved C1 2.06 mm to (43.0, 32.5)
- moved R3 1.58 mm to (41.5, 41.5)
- moved TP10 1.00 mm to (3.50, 9.50)
Connections:
- net N$1 renamed VR
- net N$3 renamed VREF+
- new net IN-DC: C7.2, J1.2, R4.2, TP1.1
- new net N$1: R8.2, R9.1
- net GND: now also P1.1, R7.1; no longer P1-.1
- net IN: now also C7.1, J1.1, P1.4; no longer P1-.4, R4.2, TP1.1
- net NC: now also P1.3; no longer P1-.3
- net OUT: now also P1.5, R7.2, R9.2; no longer P1-.5
- net V+: now also P1.2; no longer P1-.2
- net VFB: now also R8.1
Routing:
- net OUT: track 28.8 -> 59.7 mm
- net IN-DC: track 0.00 -> 20.5 mm
- net VFB: track 19.3 -> 39.1 mm
- net N$1: track 0.00 -> 7.16 mm
- net V+: track 65.2 -> 60.4 mm
- net VREF+: track 23.1 -> 18.6 mm
- net VREF: track 18.1 -> 22.5 mm
- net IN: track 10.4 -> 12.8 mm
- net VR: track 28.8 -> 30.8 mm
- net P1.3: track 10.0 -> 11.1 mm
Other:
- board text added: "C7"
- board text added: "J1"
- board text added: "R7"
- board text added: "R8"
- board text added: "R9"
- board text removed: "INVERTING AMPLIFIER"
