File: miniPCB/04/A/04A-005/04A-005.brd (EAGLE design)
At the start: 30 parts, among them J1 JUMPER

Commit message: NM.07SEP2023
Changed lines of the file:
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@@
 <attribute name="CIRCUIT_CATEGORY" value="04A, OPERATIONAL AMPLIFIER" x="11" y="46.2" size="1.3" layer="1" font="vector" ratio="12" align="center-left"/>
 <attribute name="CIRCUIT_CATEGORY" value="04A, OPERATIONAL AMPLIFIER" x="11" y="46.2" size="1.3" layer="21" font="vector" ratio="12" align="center-left"/>
+<attribute name="PART_NUMBER" value="04A-005" x="43" y="48" size="1.3" layer="16" font="vector" ratio="13" rot="MR180" align="center-right"/>
 <attribute name="PART_NUMBER" value="04A-005" x="43" y="48" size="1.3" layer="22" font="vector" ratio="13" rot="MR180" align="center-right"/>
-<attribute name="PART_NUMBER" value="04A-005" x="43" y="48" size="1.3" layer="16" font="vector" ratio="13" rot="MR180" align="center-right"/>
+<attribute name="REVISION" value="A1-01" x="37" y="46" size="1.3" layer="22" font="vector" ratio="13" rot="MR180" align="center-right"/>
 <attribute name="REVISION" value="A1-01" x="37" y="46" size="1.3" layer="16" font="vector" ratio="13" rot="MR180" align="center-right"/>
-<attribute name="REVISION" value="A1-01" x="37" y="46" size="1.3" layer="22" font="vector" ratio="13" rot="MR180" align="center-right"/>
 <attribute name="TITLE" value="INVERTING AMPLIFIER" x="11" y="48" size="1.3" layer="1" font="vector" ratio="12" align="center-left"/>
 <attribute name="TITLE" value="INVERTING AMPLIFIER" x="11" y="48" size="1.3" layer="21" font="vector" ratio="12" align="center-left"/>

Commit message: NM.21SEP2023
Changed lines of the file:
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@@
 <attribute name="CIRCUIT_CATEGORY" value="04A, OPERATIONAL AMPLIFIER" x="11" y="46.2" size="1.3" layer="1" font="vector" ratio="12" align="center-left"/>
 <attribute name="CIRCUIT_CATEGORY" value="04A, OPERATIONAL AMPLIFIER" x="11" y="46.2" size="1.3" layer="21" font="vector" ratio="12" align="center-left"/>
+<attribute name="PART_NUMBER" value="04A-005" x="43" y="48" size="1.3" layer="22" font="vector" ratio="13" rot="MR180" align="center-right"/>
 <attribute name="PART_NUMBER" value="04A-005" x="43" y="48" size="1.3" layer="16" font="vector" ratio="13" rot="MR180" align="center-right"/>
-<attribute name="PART_NUMBER" value="04A-005" x="43" y="48" size="1.3" layer="22" font="vector" ratio="13" rot="MR180" align="center-right"/>
+<attribute name="REVISION" value="A1-01" x="37" y="46" size="1.3" layer="16" font="vector" ratio="13" rot="MR180" align="center-right"/>
 <attribute name="REVISION" value="A1-01" x="37" y="46" size="1.3" layer="22" font="vector" ratio="13" rot="MR180" align="center-right"/>
-<attribute name="REVISION" value="A1-01" x="37" y="46" size="1.3" layer="16" font="vector" ratio="13" rot="MR180" align="center-right"/>
 <attribute name="TITLE" value="INVERTING AMPLIFIER" x="11" y="48" size="1.3" layer="1" font="vector" ratio="12" align="center-left"/>
 <attribute name="TITLE" value="INVERTING AMPLIFIER" x="11" y="48" size="1.3" layer="21" font="vector" ratio="12" align="center-left"/>

Commit message: NM.03OCT2023
Parts:
- moved R3 85.9 mm to (5.50, -36.5), turned to 0 degrees
- moved TP2 85.1 mm to (26.5, -41.5), turned to 0 degrees
- moved TP3 84.5 mm to (32.0, -41.5), turned to 0 degrees
- moved TP6 84.1 mm to (12.0, -47.5), turned to 0 degrees
- moved TP9 82.7 mm to (28.5, -47.5), turned to 0 degrees
- moved TP7 75.7 mm to (17.5, -47.5)
- moved R1 72.6 mm to (30.5, -30.5), turned to 0 degrees
- moved TP4 71.3 mm to (1.00, -47.5)
- moved TP5 68.0 mm to (6.50, -47.5)
- moved R2 64.6 mm to (3.50, -17.0), turned to 0 degrees
- moved C4 61.7 mm to (14.5, -24.0), turned to 0 degrees
- moved TP8 61.6 mm to (23.0, -47.5), turned to 0 degrees
- moved J1 61.4 mm to (33.5, -47.0), turned to 0 degrees
- moved R9 60.6 mm to (5.50, -42.5), turned to 0 degrees
- moved R7 58.9 mm to (30.5, -36.5)
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Routing:
- net V+: track 60.4 -> 0.00 mm
- net OUT: track 59.7 -> 0.00 mm
- net VFB: track 39.1 -> 0.00 mm
- net VR: track 30.8 -> 0.00 mm
- net VREF: track 22.5 -> 0.00 mm
- net IN-DC: track 20.5 -> 0.00 mm
- net VREF+: track 18.6 -> 0.00 mm
- net IN: track 12.8 -> 0.00 mm
- net P1.3: track 11.1 -> 0.00 mm
- net P1.1: track 9.62 -> 0.00 mm
- net N$1: track 7.16 -> 0.00 mm
