File: miniPCB/04/A/04A-005/04A-005.sch (EAGLE design)
At the start: 24 parts

Commit message: NM.14JAN2023
Parts:
- P1-: PART_NUMBER X04A-005-B -> X04A-005-B-XB
Connections:
- net GND: now also U1-PWR.V-; no longer U1P.V-
- net V+: now also U1-PWR.V+; no longer U1P.V+

Commit message: NM.16JAN2023
Connections:
- removed net N$2: C3.-, R6.1, TP5.1, U1A.+IN
- new net N$3: C3.+, R6.1, TP5.1, U1A.+IN
- net GND: now also C3.-; no longer C3.+
Other:
- moved on the sheet: C3
Changed lines of the file:
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@@
 <attribute name="NAME" x="80.01" y="129.54" size="1.778" layer="95" rot="R270"/>
 </instance>
-<instance part="C3" gate="C" x="66.04" y="91.44" smashed="yes" rot="MR180">
-<attribute name="NAME" x="68.58" y="90.17" size="1.778" layer="95" rot="MR180"/>
+<instance part="C3" gate="C" x="66.04" y="91.44" smashed="yes" rot="MR0">
+<attribute name="NAME" x="63.5" y="92.71" size="1.778" layer="95" rot="MR0"/>
 </instance>
 <instance part="GND8" gate="1" x="66.04" y="83.82" smashed="yes"/>
@@
 </segment>
 <segment>
-<pinref part="C3" gate="C" pin="+"/>
-<pinref part="GND8" gate="1" pin="GND"/>
-</segment>
-<segment>
 <pinref part="R3" gate="R" pin="1"/>
 <pinref part="GND5" gate="1" pin="GND"/>
@@
 <pinref part="TP10" gate="TP" pin="1"/>
 <wire x1="109.22" y1="167.64" x2="109.22" y2="162.56" width="0.1524" layer="91"/>
+</segment>
+<segment>
+<pinref part="GND8" gate="1" pin="GND"/>
+<pinref part="C3" gate="C" pin="-"/>
 </segment>
 </net>
@@
 </segment>
 </net>
-<net name="N$2" class="0">
-<segment>
-<pinref part="U1" gate="A" pin="+IN"/>
-<wire x1="66.04" y1="114.3" x2="68.58" y2="114.3" width="0.1524" layer="91"/>
-<pinref part="R6" gate="R" pin="1"/>
-<wire x1="76.2" y1="96.52" x2="71.12" y2="96.52" width="0.1524" layer="91"/>
-<pinref part="C3" gate="C" pin="-"/>
-<junction x="66.04" y="96.52"/>
-<wire x1="71.12" y1="96.52" x2="66.04" y2="96.52" width="0.1524" layer="91"/>
-<wire x1="66.04" y1="96.52" x2="66.04" y2="114.3" width="0.1524" layer="91"/>
-<pinref part="TP5" gate="TP" pin="1"/>
-<junction x="71.12" y="96.52"/>
-</segment>
-</net>
 <net name="IN" class="0">
 <segment>
@@
 </segment>
 </net>
+<net name="N$3" class="0">
+<segment>
+<pinref part="R6" gate="R" pin="1"/>
+<wire x1="76.2" y1="96.52" x2="71.12" y2="96.52" width="0.1524" layer="91"/>
+<pinref part="TP5" gate="TP" pin="1"/>
+<pinref part="U1" gate="A" pin="+IN"/>
+<wire x1="66.04" y1="114.3" x2="68.58" y2="114.3" width="0.1524" layer="91"/>
+<wire x1="66.04" y1="96.52" x2="66.04" y2="114.3" width="0.1524" layer="91"/>
+<wire x1="71.12" y1="96.52" x2="66.04" y2="96.52" width="0.1524" layer="91"/>
+<junction x="71.12" y="96.52"/>
+<pinref part="C3" gate="C" pin="+"/>
+<junction x="66.04" y="96.52"/>
+</segment>
+</net>

Commit message: NM.04FEB2023
Parts:
- C1, C5: device minipcb:CAPACITORTHD -> minipcb:CAPACITOR_10
Changed lines of the file:
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@@
 <grid distance="0.1" unitdist="inch" unit="inch" style="lines" multiple="1" display="no" altdistance="0.01" altunitdist="inch" altunit="inch"/>
 <layers>
-<layer number="1" name="Top" color="4" fill="1" visible="no" active="no"/>
-<layer number="2" name="Route2" color="1" fill="3" visible="no" active="no"/>
-<layer number="3" name="Route3" color="4" fill="3" visible="no" active="no"/>
-<layer number="4" name="Route4" color="1" fill="4" visible="no" active="no"/>
-<layer number="5" name="Route5" color="4" fill="4" visible="no" active="no"/>
-<layer number="6" name="Route6" color="1" fill="8" visible="no" active="no"/>
-<layer number="7" name="Route7" color="4" fill="8" visible="no" active="no"/>
-<layer number="8" name="Route8" color="1" fill="2" visible="no" active="no"/>
-<layer number="9" name="Route9" color="4" fill="2" visible="no" active="no"/>
-<layer number="10" name="Route10" color="1" fill="7" visible="no" active="no"/>
-<layer number="11" name="Route11" color="4" fill="7" visible="no" active="no"/>
-<layer number="12" name="Route12" color="1" fill="5" visible="no" active="no"/>
-<layer number="13" name="Route13" color="4" fill="5" visible="no" active="no"/>
-<layer number="14" name="Route14" color="1" fill="6" visible="no" active="no"/>
-<layer number="15" name="Route15" color="4" fill="6" visible="no" active="no"/>
-<layer number="16" name="Bottom" color="1" fill="1" visible="no" active="no"/>
-<layer number="17" name="Pads" color="2" fill="1" visible="no" active="no"/>
-<layer number="18" name="Vias" color="2" fill="1" visible="no" active="no"/>
-<layer number="19" name="Unrouted" color="6" fill="1" visible="no" active="no"/>
-<layer number="20" name="Dimension" color="15" fill="1" visible="no" active="no"/>
-<layer number="21" name="tPlace" color="7" fill="1" visible="no" active="no"/>
-<layer number="22" name="bPlace" color="7" fill="1" visible="no" active="no"/>
-<layer number="23" name="tOrigins" color="15" fill="1" visible="no" active="no"/>
-<layer number="24" name="bOrigins" color="15" fill="1" visible="no" active="no"/>
-<layer number="25" name="tNames" color="7" fill="1" visible="no" active="no"/>
-<layer number="26" name="bNames" color="7" fill="1" visible="no" active="no"/>
-<layer number="27" name="tValues" color="7" fill="1" visible="no" active="no"/>
-<layer number="28" name="bValues" color="7" fill="1" visible="no" active="no"/>
+<layer number="1" name="Top" color="4" fill="1" visible="yes" active="no"/>
+<layer number="2" name="Route2" color="1" fill="3" visible="yes" active="no"/>
+<layer number="3" name="Route3" color="4" fill="3" visible="yes" active="no"/>
+<layer number="4" name="Route4" color="1" fill="4" visible="yes" active="no"/>
+<layer number="5" name="Route5" color="4" fill="4" visible="yes" active="no"/>
+<layer number="6" name="Route6" color="1" fill="8" visible="yes" active="no"/>
+<layer number="7" name="Route7" color="4" fill="8" visible="yes" active="no"/>
+<layer number="8" name="Route8" color="1" fill="2" visible="yes" active="no"/>
+<layer number="9" name="Route9" color="4" fill="2" visible="yes" active="no"/>
+<layer number="10" name="Route10" color="1" fill="7" visible="yes" active="no"/>
+<layer number="11" name="Route11" color="4" fill="7" visible="yes" active="no"/>
+<layer number="12" name="Route12" color="1" fill="5" visible="yes" active="no"/>
+<layer number="13" name="Route13" color="4" fill="5" visible="yes" active="no"/>
+<layer number="14" name="Route14" color="1" fill="6" visible="yes" active="no"/>
+<layer number="15" name="Route15" color="4" fill="6" visible="yes" active="no"/>
+<layer number="16" name="Bottom" color="1" fill="1" visible="yes" active="no"/>
+<layer number="17" name="Pads" color="2" fill="1" visible="yes" active="no"/>
+<layer number="18" name="Vias" color="2" fill="1" visible="yes" active="no"/>
+<layer number="19" name="Unrouted" color="6" fill="1" visible="yes" active="no"/>
+<layer number="20" name="Dimension" color="15" fill="1" visible="yes" active="no"/>
+<layer number="21" name="tPlace" color="7" fill="1" visible="yes" active="no"/>
+<layer number="22" name="bPlace" color="7" fill="1" visible="yes" active="no"/>
+<layer number="23" name="tOrigins" color="15" fill="1" visible="yes" active="no"/>
+<layer number="24" name="bOrigins" color="15" fill="1" visible="yes" active="no"/>
+<layer number="25" name="tNames" color="7" fill="1" visible="yes" active="no"/>
+<layer number="26" name="bNames" color="7" fill="1" visible="yes" active="no"/>
+<layer number="27" name="tValues" color="7" fill="1" visible="yes" active="no"/>
+<layer number="28" name="bValues" color="7" fill="1" visible="yes" active="no"/>
 <layer number="29" name="tStop" color="7" fill="3" visible="no" active="no"/>
 <layer number="30" name="bStop" color="7" fill="6" visible="no" active="no"/>
@@
 <layer number="35" name="tGlue" color="7" fill="4" visible="no" active="no"/>
 <layer number="36" name="bGlue" color="7" fill="5" visible="no" active="no"/>
-<layer number="37" name="tTest" color="7" fill="1" visible="no" active="no"/>
-<layer number="38" name="bTest" color="7" fill="1" visible="no" active="no"/>
+<layer number="37" name="tTest" color="7" fill="1" visible="yes" active="no"/>
+<layer number="38" name="bTest" color="7" fill="1" visible="yes" active="no"/>
 <layer number="39" name="tKeepout" color="4" fill="11" visible="no" active="no"/>
 <layer number="40" name="bKeepout" color="1" fill="11" visible="no" active="no"/>
@@
 <layer number="44" name="Drills" color="7" fill="1" visible="no" active="no"/>
 <layer number="45" name="Holes" color="7" fill="1" visible="no" active="no"/>
-<layer number="46" name="Milling" color="3" fill="1" visible="no" active="no"/>
-<layer number="47" name="Measures" color="7" fill="1" visible="no" active="no"/>
-<layer number="48" name="Document" color="7" fill="1" visible="no" active="no"/>
-<layer number="49" name="Reference" color="7" fill="1" visible="no" active="no"/>
-<layer number="50" name="dxf" color="7" fill="1" visible="no" active="no"/>
-<layer number="51" name="tDocu" color="7" fill="1" visible="no" active="no"/>
-<layer number="52" name="bDocu" color="7" fill="1" visible="no" active="no"/>
-<layer number="53" name="tGND_GNDA" color="7" fill="9" visible="no" active="no"/>
-<layer number="54" name="bGND_GNDA" color="1" fill="9" visible="no" active="no"/>
-<layer number="56" name="wert" color="7" fill="1" visible="no" active="no"/>
-<layer number="57" name="tCAD" color="7" fill="1" visible="no" active="no"/>
-<layer number="59" name="tCarbon" color="7" fill="1" visible="no" active="no"/>
-<layer number="60" name="bCarbon" color="7" fill="1" visible="no" active="no"/>
+<layer number="46" name="Milling" color="3" fill="1" visible="yes" active="no"/>
+<layer number="47" name="Measures" color="7" fill="1" visible="yes" active="no"/>
+<layer number="48" name="Document" color="7" fill="1" visible="yes" active="no"/>
+<layer number="49" name="Reference" color="7" fill="1" visible="yes" active="no"/>
+<layer number="50" name="dxf" color="7" fill="1" visible="yes" active="no"/>
+<layer number="51" name="tDocu" color="7" fill="1" visible="yes" active="no"/>
+<layer number="52" name="bDocu" color="7" fill="1" visible="yes" active="no"/>
+<layer number="53" name="tGND_GNDA" color="7" fill="9" visible="yes" active="no"/>
+<layer number="54" name="bGND_GNDA" color="1" fill="9" visible="yes" active="no"/>
+<layer number="56" name="wert" color="7" fill="1" visible="yes" active="no"/>
+<layer number="57" name="tCAD" color="7" fill="1" visible="yes" active="no"/>
+<layer number="59" name="tCarbon" color="7" fill="1" visible="yes" active="no"/>
+<layer number="60" name="bCarbon" color="7" fill="1" visible="yes" active="no"/>
 <layer number="88" name="SimResults" color="9" fill="1" visible="no" active="yes"/>
 <layer number="89" name="SimProbes" color="9" fill="1" visible="no" active="yes"/>
@@
 <part name="NC1" library="minipcb" deviceset="NC" device="" value="NC"/>
 <part name="C2" library="minipcb" deviceset="CAPACITOR" device="THD"/>
-<part name="C5" library="minipcb" deviceset="CAPACITOR" device="THD"/>
+<part name="C5" library="minipcb" deviceset="CAPACITOR" device="_10"/>
 <part name="GND2" library="minipcb" deviceset="GND" device=""/>
 <part name="GND3" library="minipcb" deviceset="GND" device=""/>
@@
 <part name="R2" library="minipcb" deviceset="TRIMPOT" device="0.100THD"/>
 <part name="P+5" library="minipcb" deviceset="V+" device=""/>
-<part name="C1" library="minipcb" deviceset="CAPACITOR" device="THD"/>
+<part name="C1" library="minipcb" deviceset="CAPACITOR" device="_10"/>
 <part name="GND6" library="minipcb" deviceset="GND" device=""/>
 <part name="C4" library="minipcb" deviceset="CAPACITOR" device="THD"/>

Commit message: NM.03SEP2023
Parts:
- removed P1-: (no value), minipcb:MINIPCB_5P50X50
- added C7: (no value), minipcb:CAPACITORTHD
- added J1: JUMPER, minipcb:PINS_2
- added P1: (no value), minipcb:MINIPCB_5P5P
- added R7, R9: (no value), minipcb:RESISTOR10MM
- added R8: (no value), minipcb:TRIMPOT0.100THD
- added U$1: MINIPCB_50X50, minipcb:MINIPCB_50X50
Connections:
- net N$1 renamed VR
- net N$3 renamed VREF+
- new net IN-DC: C7.-, J1.2, R4.2, TP1.1
- new net N$1: R8.S, R9.1
- net GND: now also P1-1.1, R7.1; no longer P1-1.1
- net IN: now also C7.+, J1.1, P1-4.1; no longer P1-4.1, R4.2, TP1.1
- net NC: now also P1-3.1; no longer P1-3.1
- net OUT: now also P1-5.1, R7.2, R9.2; no longer P1-5.1
- net V+: now also P1-2.1; no longer P1-2.1
- net VFB: now also R8.A
Other:
- note added: "NOTES: 1. DIMENSIONS ARE IN MILLIMETERS. 2. MANUFACTURING SPECIFICATIONS: ADDITIONAL OPTIONS AVAILABLE UPON REQUEST. 2.1 BASE MATERIAL: FR4-TG130 2.2 LAYERS: TWO (2) 2.3 COPPER WEIGHT: DEFAULT: - ONE OUNCE (1 oz) AVAILABLE UPON REQUEST: - TWO OUNCE (2 oz) 2.4 PIECES PER PANEL: FOUR (4) 2.5 PCB THICKNESS: DEFAULT: - 1.60 MM AVAILABLE UPON REQUEST: - 0.6 MM - 0.8 MM - 1.0 MM - 1.2 MM - 2.0 MM 2.6 P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"
- note added: "NOTES: 3. PERFORMANCE FUNCTIONS: 3.1 GAIN CONTROL: - ADJUSTING RESISTOR R8 CONTROLS OUTPUT GAIN. 3.2 DC BIAS CONTROL: - ADJUSTING RESISTOR R2 CONTROLS DC BIAS VOLTAGE. 3.3 JUMPER SELECTION: - WITH: DC BIAS AMPLIFIED. - WITHOUT: DC BIAS BLOCKED, ONLY AC COMPONENT AMPLIFIED. 4. CALIBRATION ADJUSTMENT PROCEDURE: 4.1 PURPOSE - SET OUTPUT DC BIAS TO HALF OF SUPPLY VOLTAGE. 4.2 SCOPE - PERFORM DURING C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"

Commit message: NM.21SEP2023
Other:
- note added: "NOTES: 3. PERFORMANCE FUNCTIONS: 3.1 GAIN CONTROL: - ADJUSTING RESISTOR R8 CONTROLS OUTPUT GAIN. 3.2 DC BIAS CONTROL: - ADJUSTING RESISTOR R2 CONTROLS DC BIAS VOLTAGE. 3.3 JUMPER SELECTION: - WITH: DC BIAS AMPLIFIED. - WITHOUT: DC BIAS BLOCKED, ONLY AC AMPLIFIED. 4. CALIBRATION ADJUSTMENT PROCEDURE: 4.1 PURPOSE - SET OUTPUT DC BIAS TO HALF OF SUPPLY VOLTAGE. 4.2 SCOPE - PERFORM DURING CALIBRATION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"
- note removed: "NOTES: 3. PERFORMANCE FUNCTIONS: 3.1 GAIN CONTROL: - ADJUSTING RESISTOR R8 CONTROLS OUTPUT GAIN. 3.2 DC BIAS CONTROL: - ADJUSTING RESISTOR R2 CONTROLS DC BIAS VOLTAGE. 3.3 JUMPER SELECTION: - WITH: DC BIAS AMPLIFIED. - WITHOUT: DC BIAS BLOCKED, ONLY AC COMPONENT AMPLIFIED. 4. CALIBRATION ADJUSTMENT PROCEDURE: 4.1 PURPOSE - SET OUTPUT DC BIAS TO HALF OF SUPPLY VOLTAGE. 4.2 SCOPE - PERFORM DURING C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"
- moved on the sheet: C1, C2, C3, C4, C5, C6, C7, J1, P1-1, P1-2, P1-3, P1-4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

Commit message: NM.03OCT2023
Other:
- note added: "NOTES: 1. DIMENSIONS ARE IN MILLIMETERS."
- note removed: "NOTES: 1. DIMENSIONS ARE IN MILLIMETERS. 2. MANUFACTURING SPECIFICATIONS: ADDITIONAL OPTIONS AVAILABLE UPON REQUEST. 2.1 BASE MATERIAL: FR4-TG130 2.2 LAYERS: TWO (2) 2.3 COPPER WEIGHT: DEFAULT: - ONE OUNCE (1 oz) AVAILABLE UPON REQUEST: - TWO OUNCE (2 oz) 2.4 PIECES PER PANEL: FOUR (4) 2.5 PCB THICKNESS: DEFAULT: - 1.60 MM AVAILABLE UPON REQUEST: - 0.6 MM - 0.8 MM - 1.0 MM - 1.2 MM - 2.0 MM 2.6 P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"
- note removed: "NOTES: 3. PERFORMANCE FUNCTIONS: 3.1 GAIN CONTROL: - ADJUSTING RESISTOR R8 CONTROLS OUTPUT GAIN. 3.2 DC BIAS CONTROL: - ADJUSTING RESISTOR R2 CONTROLS DC BIAS VOLTAGE. 3.3 JUMPER SELECTION: - WITH: DC BIAS AMPLIFIED. - WITHOUT: DC BIAS BLOCKED, ONLY AC AMPLIFIED. 4. CALIBRATION ADJUSTMENT PROCEDURE: 4.1 PURPOSE - SET OUTPUT DC BIAS TO HALF OF SUPPLY VOLTAGE. 4.2 SCOPE - PERFORM DURING CALIBRATION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"
