File: miniPCB/04/A/04A-015/X04A-015-B-XB.brd (EAGLE design)
At the start: 100 x 100 mm, 113 parts

Commit message: NM.14JAN2023
Other:
- board text added: "DIFFERENTIAL AMPLIFIER"
Changed lines of the file:
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@@
 <text x="42.7299875" y="28.49999375" size="1.499996875" layer="125" font="vector" ratio="12" rot="R90">TP12</text>
 <text x="23.500003125" y="27.99999375" size="1.499996875" layer="125" font="vector" ratio="12" rot="R90">U1</text>
+<text x="45" y="44" size="1.778" layer="22" font="vector" ratio="12" rot="MR0">DIFFERENTIAL AMPLIFIER</text>
 <text x="35.50000625" y="84.50000625" size="1.499996875" layer="125" font="vector" ratio="13" rot="R90">C1</text>
 <text x="13" y="76" size="1.499996875" layer="125" font="vector" ratio="13" rot="R180">C2</text>
@@
 <text x="42.7299875" y="78.49999375" size="1.499996875" layer="125" font="vector" ratio="12" rot="R90">TP12</text>
 <text x="23.500003125" y="77.99999375" size="1.499996875" layer="125" font="vector" ratio="12" rot="R90">U1</text>
+<text x="45" y="94" size="1.778" layer="22" font="vector" ratio="12" rot="MR0">DIFFERENTIAL AMPLIFIER</text>
 <text x="85.50000625" y="34.50000625" size="1.499996875" layer="125" font="vector" ratio="13" rot="R90">C1</text>
 <text x="63" y="26" size="1.499996875" layer="125" font="vector" ratio="13" rot="R180">C2</text>
@@
 <text x="92.7299875" y="28.49999375" size="1.499996875" layer="125" font="vector" ratio="12" rot="R90">TP12</text>
 <text x="73.500003125" y="27.99999375" size="1.499996875" layer="125" font="vector" ratio="12" rot="R90">U1</text>
+<text x="95" y="44" size="1.778" layer="22" font="vector" ratio="12" rot="MR0">DIFFERENTIAL AMPLIFIER</text>
 <text x="85.50000625" y="84.50000625" size="1.499996875" layer="125" font="vector" ratio="13" rot="R90">C1</text>
 <text x="63" y="76" size="1.499996875" layer="125" font="vector" ratio="13" rot="R180">C2</text>
@@
 <text x="92.7299875" y="78.49999375" size="1.499996875" layer="125" font="vector" ratio="12" rot="R90">TP12</text>
 <text x="73.500003125" y="77.99999375" size="1.499996875" layer="125" font="vector" ratio="12" rot="R90">U1</text>
+<text x="95" y="94" size="1.778" layer="22" font="vector" ratio="12" rot="MR0">DIFFERENTIAL AMPLIFIER</text>
 <wire x1="0" y1="0" x2="0" y2="100" width="0" layer="20"/>
 <wire x1="0" y1="100" x2="100" y2="100" width="0" layer="20"/>
