File: miniPCB/04/A/04A-015/04A-015.sch (EAGLE design)
At the start: 28 parts

Commit message: NM.14JAN2023
Parts:
- P1-: PART_NUMBER X04A-015-B -> X04A-015-B-XB
Connections:
- net GND: now also U1-PWR.V-; no longer U1P.V-
- net V+: now also U1-PWR.V+; no longer U1P.V+

Commit message: NM.07SEP2023
Parts:
- removed P1-: (no value), minipcb:MINIPCB_7P50
- added P1: (no value), minipcb:MINIPCB_5P5P
- added R10: (no value), minipcb:TRIMPOT0.100THD
- added R11, R9: (no value), minipcb:RESISTOR10MM
- added U$1: MINIPCB_50X50, minipcb:MINIPCB_50X50
- C4, C6: device minipcb:CAPACITORTHD -> minipcb:CAPACITOR_10
Connections:
- new net N$5: R8.2, TP12.1
- new net N$6: R10.S, R11.2
- net GND: now also P1-1.1; no longer P1-1.1
- net IN: now also P1-4.1; no longer P1-4.1
- net N$2: now also R9.1, U1B.-IN, U1B.OUT; no longer C6.-, R6.2, R8.1, TP8.1
- net N$4: no longer P1-6.1
- net NC: now also P1-3.1; no longer P1-3.1
- net OUT: now also P1-5.1, R10.A; no longer P1-5.1
- net V+: now also P1-2.1; no longer P1-2.1
- net VFB: now also R11.1
- net VREF: now also C6.-, R6.2, R8.1, R9.2, TP8.1; no longer P1-7.1, R8.2, TP12.1, U1B.-IN, U1B.OUT
Other:
- note added: "NOTES: 1. DIMENSIONS ARE IN MILLIMETERS. 2."

Commit message: NM.15SEP2023
Parts:
- removed P1: (no value), minipcb:MINIPCB_5P5P
- added P2: (no value), minipcb:MINIPCB_7P
- C3: device minipcb:CAPACITORTHD -> minipcb:CAPACITOR_10
- C6: device minipcb:CAPACITOR_10 -> minipcb:CAPACITORTHD
- U$1: value MINIPCB_50X50 -> CLASSIC-50; device minipcb:MINIPCB_50X50 -> miniPCB_BOARDS:CLASSIC-50; CIRCUIT_CATEGORY OPERATIONAL AMPLIFIERS -> (none); REVISION A1-01 -> (none); TITLE DIFFERENCE AMPLIFIER -> miniPCB, DIFFERENCE AMPLIFIER
Connections:
- net N$1 renamed REF
- net N$2 renamed VFBREF
- net N$3 renamed VPOS
- removed net IN: P1-4.1, R4.2, TP1.1
- removed net N$4: R5.2, TP2.1
- removed net N$5: R8.2, TP12.1
- new net IN+: P2-4.1, R4.2, TP1.1
- new net IN-: P2-6.1, R5.2, TP2.1
- new net OUTREF: P2-7.1, R8.2, TP12.1
- net GND: now also P2-1.1; no longer P1-1.1
- net NC: now also P2-3.1; no longer P1-3.1
- net OUT: now also P2-5.1; no longer P1-5.1
- net V+: now also P2-2.1; no longer P1-2.1
Changed lines of the file:
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@@
 <part name="C1" library="minipcb" deviceset="CAPACITOR" device="THD"/>
 <part name="GND6" library="minipcb" deviceset="GND" device=""/>
-<part name="C3" library="minipcb" deviceset="CAPACITOR" device="THD"/>
+<part name="C3" library="minipcb" deviceset="CAPACITOR" device="_10"/>
 <part name="U1" library="minipcb" deviceset="OPAMP_DUAL" device="THD"/>
 <part name="C5" library="minipcb" deviceset="CAPACITOR" device="THD"/>
-<part name="C6" library="minipcb" deviceset="CAPACITOR" device="_10"/>
+<part name="C6" library="minipcb" deviceset="CAPACITOR" device="THD"/>
 <part name="GND8" library="minipcb" deviceset="GND" device=""/>
 <part name="GND5" library="minipcb" deviceset="GND" device=""/>
@@
 <attribute name="TITLE" value="DIFFERENCE AMPLIFIER"/>
 </part>
-<part name="P1" library="minipcb" deviceset="MINIPCB_5P" device="5P"/>
-<part name="U$1" library="minipcb" deviceset="MINIPCB_50X50" device="">
-<attribute name="CIRCUIT_CATEGORY" value="OPERATIONAL AMPLIFIERS"/>
-<attribute name="PART_NUMBER" value="04A-015"/>
-<attribute name="REVISION" value="A1-01"/>
-<attribute name="TITLE" value="DIFFERENCE AMPLIFIER"/>
-</part>
 <part name="U$2" library="minipcb" deviceset="DRAWING_PWR_IN_OUT" device=""/>
 <part name="R9" library="minipcb" deviceset="RESISTOR" device="10MM"/>
@@
 <part name="R11" library="minipcb" deviceset="RESISTOR" device="10MM"/>
 <part name="NC2" library="minipcb" deviceset="NC" device="" value="NC"/>
+<part name="P2" library="minipcb" deviceset="MINIPCB_7P" device=""/>
+<part name="U$1" library="miniPCB_BOARDS" deviceset="CLASSIC" device="-50">
+<attribute name="PART_NUMBER" value="04A-015"/>
+<attribute name="TITLE" value="miniPCB, DIFFERENCE AMPLIFIER"/>
+</part>
 </parts>
 <sheets>
@@
 <attribute name="QA_DATE" x="295" y="7" size="2.5" layer="97" rot="R180" align="center-left"/>
 </instance>
-<instance part="U$1" gate="G$1" x="193.04" y="109.22" smashed="yes">
-<attribute name="TITLE" x="203.54" y="157.22" size="1.5" layer="94" font="vector" ratio="12" align="center-left"/>
-<attribute name="TITLE" x="203.54" y="157.22" size="1.5" layer="94" font="vector" ratio="12" align="center-left"/>
-<attribute name="CIRCUIT_CATEGORY" x="203.54" y="155.42" size="1.5" layer="94" font="vector" ratio="12" align="center-left"/>
-<attribute name="CIRCUIT_CATEGORY" x="203.54" y="155.42" size="1.5" layer="94" font="vector" ratio="12" align="center-left"/>
-</instance>
 <instance part="DWG1" gate="DWG" x="329.86" y="63" smashed="yes"/>
+<instance part="U$1" gate="G$5" x="170.18" y="106.68" smashed="yes">
+<attribute name="TITLE" x="172.18" y="154.68" size="1" layer="94" font="vector" ratio="12"/>
+<attribute name="TITLE" x="172.18" y="154.68" size="1" layer="94" font="vector" ratio="12"/>
+</instance>
 </instances>
 <busses>
@@
 <attribute name="NAME" x="261.62" y="127" size="1.778" layer="94" rot="R90" align="center-left"/>
 </instance>
-<instance part="P1" gate="-1" x="109.22" y="198.12" smashed="yes">
-<attribute name="NAME" x="102.87" y="198.12" size="1.778" layer="95" ratio="13" rot="MR0" align="center-left"/>
-</instance>
-<instance part="P1" gate="-2" x="109.22" y="190.5" smashed="yes">
-<attribute name="NAME" x="102.87" y="190.5" size="1.778" layer="95" ratio="13" rot="MR0" align="center-left"/>
-</instance>
-<instance part="P1" gate="-3" x="109.22" y="182.88" smashed="yes">
-<attribute name="NAME" x="102.87" y="182.88" size="1.778" layer="95" ratio="13" rot="MR0" align="center-left"/>
-</instance>
-<instance part="P1" gate="-4" x="109.22" y="137.16" smashed="yes">
-<attribute name="NAME" x="102.87" y="137.16" size="1.778" layer="95" ratio="13" rot="MR0" align="center-left"/>
-</instance>
-<instance part="P1" gate="-5" x="281.94" y="134.62" smashed="yes" rot="R180">
-<attribute name="NAME" x="288.29" y="134.62" size="1.778" layer="95" ratio="13" rot="MR180" align="center-left"/>
-</instance>
 <instance part="SHEET2" gate="G$3" x="0" y="0" smashed="yes">
 <attribute name="DRAWING_NAME" x="312.5" y="16" size="5" layer="97" align="top-left"/>
@@
 </instance>
 <instance part="NC2" gate="NC" x="246.38" y="170.18" smashed="yes"/>
+<instance part="P2" gate="-1" x="109.22" y="198.12" smashed="yes">
+<attribute name="NAME" x="102.87" y="198.12" size="1.778" layer="95" ratio="13" rot="MR0" align="center-left"/>
+</instance>
+<instance part="P2" gate="-2" x="109.22" y="190.5" smashed="yes">
+<attribute name="NAME" x="102.87" y="190.5" size="1.778" layer="95" ratio="13" rot="MR0" align="center-left"/>
+</instance>
+<instance part="P2" gate="-3" x="109.22" y="182.88" smashed="yes">
+<attribute name="NAME" x="102.87" y="182.88" size="1.778" layer="95" ratio="13" rot="MR0" align="center-left"/>
+</instance>
+<instance part="P2" gate="-4" x="109.22" y="137.16" smashed="yes">
+<attribute name="NAME" x="102.87" y="137.16" size="1.778" layer="95" ratio="13" rot="MR0" align="center-left"/>
+</instance>
+<instance part="P2" gate="-5" x="281.94" y="134.62" smashed="yes" rot="R180">
+<attribute name="NAME" x="288.29" y="134.62" size="1.778" layer="95" ratio="13" rot="MR180" align="center-left"/>
+</instance>
+<instance part="P2" gate="-6" x="109.22" y="121.92" smashed="yes">
+<attribute name="NAME" x="102.87" y="121.92" size="1.778" layer="95" ratio="13" rot="MR0" align="center-left"/>
+</instance>
+<instance part="P2" gate="-7" x="281.94" y="121.92" smashed="yes" rot="R180">
+<attribute name="NAME" x="288.29" y="121.92" size="1.778" layer="95" ratio="13" rot="MR180" align="center-left"/>
+</instance>
 </instances>
 <busses>
@@
 <pinref part="GND1" gate="1" pin="GND"/>
 <wire x1="111.76" y1="198.12" x2="109.22" y2="198.12" width="0.1524" layer="91"/>
-<pinref part="P1" gate="-1" pin="1"/>
+<pinref part="P2" gate="-1" pin="1"/>
 </segment>
 <segment>
@@
 <segment>
 <wire x1="109.22" y1="182.88" x2="114.3" y2="182.88" width="0.1524" layer="91"/>
-<pinref part="P1" gate="-3" pin="1"/>
+<pinref part="P2" gate="-3" pin="1"/>
 </segment>
 </net>
@@
 <pinref part="P+1" gate="1" pin="V+"/>
 <wire x1="119.38" y1="190.5" x2="109.22" y2="190.5" width="0.1524" layer="91"/>
-<pinref part="P1" gate="-2" pin="1"/>
+<pinref part="P2" gate="-2" pin="1"/>
 </segment>
 <segment>
@@
 <pinref part="TP9" gate="TP" pin="1"/>
 <junction x="251.46" y="134.62"/>
-<pinref part="P1" gate="-5" pin="1"/>
 <pinref part="R10" gate="R" pin="A"/>
 <wire x1="246.38" y1="160.02" x2="246.38" y2="157.48" width="0.1524" layer="91"/>
 <junction x="246.38" y="157.48"/>
+<label x="266.7" y="134.62" size="1.778" layer="95"/>
+<pinref part="P2" gate="-5" pin="1"/>
 </segment>
 </net>
@@
 <wire x1="218.44" y1="165.1" x2="218.44" y2="157.48" width="0.1524" layer="91"/>
 <junction x="218.44" y="157.48"/>
+<label x="210.82" y="137.16" size="1.778" layer="95"/>
 </segment>
 </net>
@@
 <wire x1="210.82" y1="86.36" x2="246.38" y2="86.36" width="0.1524" layer="91"/>
 <pinref part="R9" gate="R" pin="2"/>
+<label x="218.44" y="86.36" size="1.778" layer="95"/>
 </segment>
 </net>
@@
 </segment>
 </net>
-<net name="N$1" class="0">
+<net name="REF" class="0">
 <segment>
 <pinref part="C1" gate="C" pin="+"/>
@@
 <wire x1="162.56" y1="88.9" x2="154.94" y2="88.9" width="0.1524" layer="91"/>
 <junction x="162.56" y="88.9"/>
-</segment>
-</net>
-<net name="IN" class="0">
+<label x="137.16" y="88.9" size="1.778" layer="95"/>
+</segment>
+</net>
+<net name="IN+" class="0">
 <segment>
 <pinref part="R4" gate="R" pin="2"/>
@@
 <wire x1="187.96" y1="137.16" x2="109.22" y2="137.16" width="0.1524" layer="91"/>
 <junction x="187.96" y="137.16"/>
-<pinref part="P1" gate="-4" pin="1"/>
-</segment>
-</net>
-<net name="N$3" class="0">
+<label x="170.18" y="137.16" size="1.778" layer="95"/>
+<pinref part="P2" gate="-4" pin="1"/>
+</segment>
+</net>
+<net name="VPOS" class="0">
 <segment>
 <pinref part="U1" gate="A" pin="+IN"/>
@@
 <wire x1="203.2" y1="121.92" x2="208.28" y2="121.92" width="0.1524" layer="91"/>
 <junction x="208.28" y="121.92"/>
-</segment>
-</net>
-<net name="N$4" class="0">
+<label x="210.82" y="121.92" size="1.778" layer="95"/>
+</segment>
+</net>
+<net name="IN-" class="0">
 <segment>
 <wire x1="109.22" y1="121.92" x2="187.96" y2="121.92" width="0.1524" layer="91"/>
@@
 <wire x1="187.96" y1="121.92" x2="193.04" y2="121.92" width="0.1524" layer="91"/>
 <junction x="187.96" y="121.92"/>
-</segment>
-</net>
-<net name="N$5" class="0">
+<label x="170.18" y="121.92" size="1.778" layer="95"/>
+<pinref part="P2" gate="-6" pin="1"/>
+</segment>
+</net>
+<net name="OUTREF" class="0">
 <segment>
 <pinref part="R8" gate="R" pin="2"/>
@@
 <junction x="261.62" y="121.92"/>
 <wire x1="261.62" y1="121.92" x2="259.08" y2="121.92" width="0.1524" layer="91"/>
-</segment>
-</net>
-<net name="N$2" class="0">
+<label x="266.7" y="121.92" size="1.778" layer="95"/>
+<pinref part="P2" gate="-7" pin="1"/>
+</segment>
+</net>
+<net name="VFBREF" class="0">
 <segment>
 <pinref part="U1" gate="B" pin="OUT"/>
@@
 <wire x1="170.18" y1="83.82" x2="170.18" y2="78.74" width="0.1524" layer="91"/>
 <pinref part="R9" gate="R" pin="1"/>
-</segment>
-</net>
+<label x="185.42" y="78.74" size="1.778" layer="95"/>
+</segment>
+</net>

Commit message: NM.03OCT2023
Parts:
- added R12: (no value), minipcb:RESISTOR10MM
Connections:
- new net OUTPUT: P2-5.1, R12.2
- net OUT: now also R12.1; no longer P2-5.1
Other:
- moved on the sheet: R8, TP12, TP8

Commit message: NM.07MAR2024
Parts:
- added TP13: (no value), minipcb:TESTPOINTKE5000-SMTEXT
Connections:
- net OUTPUT: now also TP13.1
Other:
- note removed: "NOTES: 1. DIMENSIONS ARE IN MILLIMETERS. 2."
