File: miniPCB/00/A/00A-001/00A-001.sch (EAGLE design)
At the start: 5 parts

Commit message: NM.28JAN2023
Parts:
- removed U$1: MINIPCB_LOGO, minipcb:MINIPCB_LOGO
Changed lines of the file:
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@@
 <?xml version="1.0" encoding="utf-8"?>
 <!DOCTYPE eagle SYSTEM "eagle.dtd">
-<eagle version="6.3">
+<eagle version="9.6.2">
 <drawing>
 <settings>
 <setting alwaysvectorfont="no"/>
+<setting keepoldvectorfont="yes"/>
 <setting verticaltext="up"/>
 </settings>
@@
 <attribute name="CIRCUIT_NAME" value="PROBE BOARD"/>
 </part>
-<part name="U$1" library="minipcb" deviceset="MINIPCB_LOGO" device=""/>
 </parts>
 <sheets>
@@
 </plain>
 <instances>
-<instance part="P1" gate="P" x="111.76" y="124.46"/>
-<instance part="P2" gate="P" x="111.76" y="109.22"/>
-<instance part="P3" gate="P" x="139.7" y="124.46" rot="MR0"/>
-<instance part="P4" gate="P" x="139.7" y="109.22" rot="MR0"/>
-<instance part="SHEET1" gate="SH" x="0" y="0"/>
-<instance part="SHEET1" gate="G$1" x="182.88" y="177.8"/>
-<instance part="U$1" gate="G$1" x="124.46" y="132.08"/>
+<instance part="P1" gate="P" x="111.76" y="124.46" smashed="yes">
+<attribute name="NAME" x="111.76" y="129.54" size="1.778" layer="95" ratio="13"/>
+<attribute name="VALUE" x="111.76" y="127" size="1.778" layer="96" ratio="13"/>
+</instance>
+<instance part="P2" gate="P" x="111.76" y="109.22" smashed="yes">
+<attribute name="NAME" x="111.76" y="114.3" size="1.778" layer="95" ratio="13"/>
+<attribute name="VALUE" x="111.76" y="111.76" size="1.778" layer="96" ratio="13"/>
+</instance>
+<instance part="P3" gate="P" x="139.7" y="124.46" smashed="yes" rot="MR0">
+<attribute name="NAME" x="139.7" y="129.54" size="1.778" layer="95" ratio="13" rot="MR0"/>
+<attribute name="VALUE" x="139.7" y="127" size="1.778" layer="96" ratio="13" rot="MR0"/>
+</instance>
+<instance part="P4" gate="P" x="139.7" y="109.22" smashed="yes" rot="MR0">
+<attribute name="NAME" x="139.7" y="114.3" size="1.778" layer="95" ratio="13" rot="MR0"/>
+<attribute name="VALUE" x="139.7" y="111.76" size="1.778" layer="96" ratio="13" rot="MR0"/>
+</instance>
+<instance part="SHEET1" gate="SH" x="0" y="0" smashed="yes">
+<attribute name="DRAWING_NAME" x="166.37" y="21.59" size="2.54" layer="97"/>
+<attribute name="REVISION" x="194.31" y="16.51" size="5.08" layer="97" align="center"/>
+<attribute name="SHEET" x="194.31" y="8.89" size="5.08" layer="97" align="center"/>
+<attribute name="VALUE" x="166.37" y="36.83" size="2.54" layer="97"/>
+<attribute name="LAST_DATE_TIME" x="210.82" y="6.35" size="2.54" layer="97"/>
+<attribute name="CIRCUIT_NAME" x="166.37" y="29.21" size="2.54" layer="97"/>
+<attribute name="CIRCUIT_CATEGORY" x="186.69" y="21.59" size="2.54" layer="97"/>
+</instance>
+<instance part="SHEET1" gate="G$1" x="182.88" y="177.8" smashed="yes"/>
 </instances>
 <busses>
