File: miniPCB/00/A/00A-004/00A-004.brd (EAGLE design)
At the start: 17 parts

Commit message: NM.28JAN2023
Parts:
- U$1: value MINIPCB_LOGO -> (none)
- moved U$1 3.00 mm to (67.0, 7.00)
Other:
- board text added: "00A-004-B"
- board text removed: "miniPCB.com #00A-004"
Changed lines of the file:
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@@
 <?xml version="1.0" encoding="utf-8"?>
 <!DOCTYPE eagle SYSTEM "eagle.dtd">
-<eagle version="6.3">
+<eagle version="9.6.2">
 <drawing>
 <settings>
 <setting alwaysvectorfont="no"/>
+<setting keepoldvectorfont="yes"/>
 <setting verticaltext="up"/>
 </settings>
@@
 <layer number="59" name="tCarbon" color="7" fill="1" visible="no" active="no"/>
 <layer number="60" name="bCarbon" color="7" fill="1" visible="no" active="no"/>
-<layer number="88" name="SimResults" color="9" fill="1" visible="yes" active="yes"/>
-<layer number="89" name="SimProbes" color="9" fill="1" visible="yes" active="yes"/>
-<layer number="90" name="Modules" color="7" fill="1" visible="yes" active="yes"/>
+<layer number="88" name="SimResults" color="9" fill="1" visible="no" active="no"/>
+<layer number="89" name="SimProbes" color="9" fill="1" visible="no" active="no"/>
+<layer number="90" name="Modules" color="7" fill="1" visible="no" active="no"/>
 <layer number="91" name="Nets" color="2" fill="1" visible="no" active="no"/>
 <layer number="92" name="Busses" color="1" fill="1" visible="no" active="no"/>
@@
 <hole x="9" y="18" drill="1.6"/>
 <hole x="16" y="18" drill="1.6"/>
-<hole x="3" y="17" drill="2.8"/>
-<hole x="3" y="3" drill="2.8"/>
-<hole x="67" y="3" drill="2.8"/>
-<hole x="67" y="17" drill="2.8"/>
+<hole x="3" y="17" drill="3.2"/>
+<hole x="67" y="17" drill="3.2"/>
 <wire x1="0" y1="0" x2="70" y2="0" width="0" layer="48"/>
 <wire x1="70" y1="0" x2="70" y2="20" width="0" layer="48"/>
 <wire x1="70" y1="20" x2="0" y2="20" width="0" layer="48"/>
 <wire x1="0" y1="20" x2="0" y2="0" width="0" layer="48"/>
-<rectangle x1="1" y1="5" x2="6.5" y2="15" layer="21"/>
-<text x="64" y="1" size="1.27" layer="16" font="vector" ratio="12" rot="MR0">miniPCB.com
-#00A-004</text>
+<text x="64" y="1" size="1.27" layer="16" font="vector" ratio="12" rot="MR0">00A-004-B</text>
 <text x="9.00000625" y="3.9599875" size="2.1844" layer="121" font="vector" ratio="12" rot="R180" align="bottom-center">P1</text>
 <text x="15.99999375" y="3.9599875" size="2.1844" layer="121" font="vector" ratio="12" rot="R180" align="bottom-center">P2</text>
@@
 <hole x="54" y="18" drill="1.6"/>
 <hole x="61" y="18" drill="1.6"/>
+<rectangle x1="1" y1="1" x2="6" y2="13" layer="21"/>
 </plain>
 <attributes>
@@
 <param name="dpMaxLengthDifference" value="10mm"/>
 <param name="dpGapFactor" value="2.5"/>
-<param name="checkGrid" value="0"/>
 <param name="checkAngle" value="0"/>
 <param name="checkFont" value="1"/>
 <param name="checkRestrict" value="1"/>
+<param name="checkStop" value="0"/>
+<param name="checkValues" value="0"/>
+<param name="checkNames" value="1"/>
+<param name="checkWireStubs" value="1"/>
+<param name="checkPolygonWidth" value="0"/>
 <param name="useDiameter" value="13"/>
 <param name="maxErrors" value="50"/>
@@
 <pass name="Default">
 <param name="RoutingGrid" value="50mil"/>
+<param name="AutoGrid" value="1"/>
+<param name="Efforts" value="0"/>
+<param name="TopRouterVariant" value="1"/>
 <param name="tpViaShape" value="round"/>
 <param name="PrefDir.1" value="|"/>
@@
 </autorouter>
 <elements>
-<element name="P1" library="nolan-utsa" package="PINS_1_TESTPOINT_KE5000" value="" x="9" y="6" rot="R180"/>
-<element name="P2" library="nolan-utsa" package="PINS_1_TESTPOINT_KE5000" value="" x="16" y="6" rot="R180"/>
-<element name="P3" library="nolan-utsa" package="PINS_1_1MM" value="" x="9" y="12" rot="R90"/>
-<element name="P4" library="nolan-utsa" package="PINS_1_1MM" value="" x="16" y="12" rot="R90"/>
-<element name="P5" library="nolan-utsa" package="PINS_1_TESTPOINT_KE5000" value="" x="24" y="6" rot="R180"/>
-<element name="P6" library="nolan-utsa" package="PINS_1_TESTPOINT_KE5000" value="" x="31" y="6" rot="R180"/>
-<element name="P7" library="nolan-utsa" package="PINS_1_1MM" value="" x="24" y="12" rot="R90"/>
-<element name="P8" library="nolan-utsa" package="PINS_1_1MM" value="" x="31" y="12" rot="R90"/>
-<element name="P9" library="nolan-utsa" package="PINS_1_TESTPOINT_KE5000" value="" x="39" y="6" rot="R180"/>
-<element name="P10" library="nolan-utsa" package="PINS_1_TESTPOINT_KE5000" value="" x="46" y="6" rot="R180"/>
-<element name="P11" library="nolan-utsa" package="PINS_1_1MM" value="" x="39" y="12" rot="R90"/>
-<element name="P12" library="nolan-utsa" package="PINS_1_1MM" value="" x="46" y="12" rot="R90"/>
-<element name="P13" library="nolan-utsa" package="PINS_1_TESTPOINT_KE5000" value="" x="54" y="6" rot="R180"/>
-<element name="P14" library="nolan-utsa" package="PINS_1_TESTPOINT_KE5000" value="" x="61" y="6" rot="R180"/>
-<element name="P15" library="nolan-utsa" package="PINS_1_1MM" value="" x="54" y="12" rot="R90"/>
-<element name="P16" library="nolan-utsa" package="PINS_1_1MM" value="" x="61" y="12" rot="R90"/>
-<element name="U$1" library="minipcb" package="MINIPCB-LOGO" value="MINIPCB_LOGO" x="67" y="10" rot="R90"/>
+<element name="P1" library="nolan-utsa" package="PINS_1_TESTPOINT_KE5000" value="" x="9" y="6" smashed="yes" rot="R180">
+<attribute name="NAME" x="9" y="3.96" size="2.1844" layer="25" font="vector" ratio="12" rot="R180" align="bottom-center"/>
+</element>
+<element name="P2" library="nolan-utsa" package="PINS_1_TESTPOINT_KE5000" value="" x="16" y="6" smashed="yes" rot="R180">
+<attribute name="NAME" x="16" y="3.96" size="2.1844" layer="25" font="vector" ratio="12" rot="R180" align="bottom-center"/>
+</element>
+<element name="P3" library="nolan-utsa" package="PINS_1_1MM" value="" x="9" y="12" smashed="yes" rot="R90"/>
+<element name="P4" library="nolan-utsa" package="PINS_1_1MM" value="" x="16" y="12" smashed="yes" rot="R90"/>
+<element name="P5" library="nolan-utsa" package="PINS_1_TESTPOINT_KE5000" value="" x="24" y="6" smashed="yes" rot="R180">
+<attribute name="NAME" x="24" y="3.96" size="2.1844" layer="25" font="vector" ratio="12" rot="R180" align="bottom-center"/>
+</element>
+<element name="P6" library="nolan-utsa" package="PINS_1_TESTPOINT_KE5000" value="" x="31" y="6" smashed="yes" rot="R180">
+<attribute name="NAME" x="31" y="3.96" size="2.1844" layer="25" font="vector" ratio="12" rot="R180" align="bottom-center"/>
+</element>
+<element name="P7" library="nolan-utsa" package="PINS_1_1MM" value="" x="24" y="12" smashed="yes" rot="R90"/>
+<element name="P8" library="nolan-utsa" package="PINS_1_1MM" value="" x="31" y="12" smashed="yes" rot="R90"/>
+<element name="P9" library="nolan-utsa" package="PINS_1_TESTPOINT_KE5000" value="" x="39" y="6" smashed="yes" rot="R180">
+<attribute name="NAME" x="39" y="3.96" size="2.1844" layer="25" font="vector" ratio="12" rot="R180" align="bottom-center"/>
+</element>
+<element name="P10" library="nolan-utsa" package="PINS_1_TESTPOINT_KE5000" value="" x="46" y="6" smashed="yes" rot="R180">
+<attribute name="NAME" x="46" y="3.96" size="2.1844" layer="25" font="vector" ratio="12" rot="R180" align="bottom-center"/>
+</element>
+<element name="P11" library="nolan-utsa" package="PINS_1_1MM" value="" x="39" y="12" smashed="yes" rot="R90"/>
+<element name="P12" library="nolan-utsa" package="PINS_1_1MM" value="" x="46" y="12" smashed="yes" rot="R90"/>
+<element name="P13" library="nolan-utsa" package="PINS_1_TESTPOINT_KE5000" value="" x="54" y="6" smashed="yes" rot="R180">
+<attribute name="NAME" x="54" y="3.96" size="2.1844" layer="25" font="vector" ratio="12" rot="R180" align="bottom-center"/>
+</element>
+<element name="P14" library="nolan-utsa" package="PINS_1_TESTPOINT_KE5000" value="" x="61" y="6" smashed="yes" rot="R180">
+<attribute name="NAME" x="61" y="3.96" size="2.1844" layer="25" font="vector" ratio="12" rot="R180" align="bottom-center"/>
+</element>
+<element name="P15" library="nolan-utsa" package="PINS_1_1MM" value="" x="54" y="12" smashed="yes" rot="R90"/>
+<element name="P16" library="nolan-utsa" package="PINS_1_1MM" value="" x="61" y="12" smashed="yes" rot="R90"/>
+<element name="U$1" library="minipcb" package="MINIPCB-LOGO" value="" x="67" y="7" smashed="yes" rot="R90"/>
 </elements>
 <signals>
@@
 </signal>
 </signals>
+<mfgpreviewcolors>
+<mfgpreviewcolor name="soldermaskcolor" color="0xC8008000"/>
+<mfgpreviewcolor name="silkscreencolor" color="0xFFFEFEFE"/>
+<mfgpreviewcolor name="backgroundcolor" color="0xFF282828"/>
+<mfgpreviewcolor name="coppercolor" color="0xFFFFBF00"/>
+<mfgpreviewcolor name="substratecolor" color="0xFF786E46"/>
+</mfgpreviewcolors>
 </board>
 </drawing>
-<compatibility>
-<note version="6.3" minversion="6.2.2" severity="warning">
-Since Version 6.2.2 text objects can contain more than one line,
-which will not be processed correctly with this version.
-</note>
-</compatibility>
 </eagle>
