File: miniPCB/00/A/00A-004/00A-004.sch (EAGLE design)
At the start: 17 parts

Commit message: NM.28JAN2023
Parts:
- removed U$1: MINIPCB_LOGO, minipcb:MINIPCB_LOGO
Changed lines of the file:
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@@
 <?xml version="1.0" encoding="utf-8"?>
 <!DOCTYPE eagle SYSTEM "eagle.dtd">
-<eagle version="6.3">
+<eagle version="9.6.2">
 <drawing>
 <settings>
 <setting alwaysvectorfont="no"/>
+<setting keepoldvectorfont="yes"/>
 <setting verticaltext="up"/>
 </settings>
@@
 <attribute name="CIRCUIT_NAME" value="PROBE BOARD"/>
 </part>
-<part name="U$1" library="minipcb" deviceset="MINIPCB_LOGO" device=""/>
 </parts>
 <sheets>
@@
 </plain>
 <instances>
-<instance part="P1" gate="P" x="116.84" y="157.48"/>
-<instance part="P2" gate="P" x="116.84" y="142.24"/>
-<instance part="P3" gate="P" x="144.78" y="157.48" rot="MR0"/>
-<instance part="P4" gate="P" x="144.78" y="142.24" rot="MR0"/>
-<instance part="P5" gate="P" x="116.84" y="121.92"/>
-<instance part="P6" gate="P" x="116.84" y="106.68"/>
-<instance part="P7" gate="P" x="144.78" y="121.92" rot="MR0"/>
-<instance part="P8" gate="P" x="144.78" y="106.68" rot="MR0"/>
-<instance part="P9" gate="P" x="116.84" y="83.82"/>
-<instance part="P10" gate="P" x="116.84" y="68.58"/>
-<instance part="P11" gate="P" x="144.78" y="83.82" rot="MR0"/>
-<instance part="P12" gate="P" x="144.78" y="68.58" rot="MR0"/>
-<instance part="P13" gate="P" x="116.84" y="48.26"/>
-<instance part="P14" gate="P" x="116.84" y="33.02"/>
-<instance part="P15" gate="P" x="144.78" y="48.26" rot="MR0"/>
-<instance part="P16" gate="P" x="144.78" y="33.02" rot="MR0"/>
-<instance part="SHEET1" gate="SH" x="0" y="0"/>
-<instance part="SHEET1" gate="G$1" x="182.88" y="177.8"/>
-<instance part="U$1" gate="G$1" x="129.54" y="162.56"/>
+<instance part="P1" gate="P" x="116.84" y="157.48" smashed="yes">
+<attribute name="NAME" x="116.84" y="162.56" size="1.778" layer="95" ratio="13"/>
+<attribute name="VALUE" x="116.84" y="160.02" size="1.778" layer="96" ratio="13"/>
+</instance>
+<instance part="P2" gate="P" x="116.84" y="142.24" smashed="yes">
+<attribute name="NAME" x="116.84" y="147.32" size="1.778" layer="95" ratio="13"/>
+<attribute name="VALUE" x="116.84" y="144.78" size="1.778" layer="96" ratio="13"/>
+</instance>
+<instance part="P3" gate="P" x="144.78" y="157.48" smashed="yes" rot="MR0">
+<attribute name="NAME" x="144.78" y="162.56" size="1.778" layer="95" ratio="13" rot="MR0"/>
+<attribute name="VALUE" x="144.78" y="160.02" size="1.778" layer="96" ratio="13" rot="MR0"/>
+</instance>
+<instance part="P4" gate="P" x="144.78" y="142.24" smashed="yes" rot="MR0">
+<attribute name="NAME" x="144.78" y="147.32" size="1.778" layer="95" ratio="13" rot="MR0"/>
+<attribute name="VALUE" x="144.78" y="144.78" size="1.778" layer="96" ratio="13" rot="MR0"/>
+</instance>
+<instance part="P5" gate="P" x="116.84" y="121.92" smashed="yes">
+<attribute name="NAME" x="116.84" y="127" size="1.778" layer="95" ratio="13"/>
+<attribute name="VALUE" x="116.84" y="124.46" size="1.778" layer="96" ratio="13"/>
+</instance>
+<instance part="P6" gate="P" x="116.84" y="106.68" smashed="yes">
+<attribute name="NAME" x="116.84" y="111.76" size="1.778" layer="95" ratio="13"/>
+<attribute name="VALUE" x="116.84" y="109.22" size="1.778" layer="96" ratio="13"/>
+</instance>
+<instance part="P7" gate="P" x="144.78" y="121.92" smashed="yes" rot="MR0">
+<attribute name="NAME" x="144.78" y="127" size="1.778" layer="95" ratio="13" rot="MR0"/>
+<attribute name="VALUE" x="144.78" y="124.46" size="1.778" layer="96" ratio="13" rot="MR0"/>
+</instance>
+<instance part="P8" gate="P" x="144.78" y="106.68" smashed="yes" rot="MR0">
+<attribute name="NAME" x="144.78" y="111.76" size="1.778" layer="95" ratio="13" rot="MR0"/>
+<attribute name="VALUE" x="144.78" y="109.22" size="1.778" layer="96" ratio="13" rot="MR0"/>
+</instance>
+<instance part="P9" gate="P" x="116.84" y="83.82" smashed="yes">
+<attribute name="NAME" x="116.84" y="88.9" size="1.778" layer="95" ratio="13"/>
+<attribute name="VALUE" x="116.84" y="86.36" size="1.778" layer="96" ratio="13"/>
+</instance>
+<instance part="P10" gate="P" x="116.84" y="68.58" smashed="yes">
+<attribute name="NAME" x="116.84" y="73.66" size="1.778" layer="95" ratio="13"/>
+<attribute name="VALUE" x="116.84" y="71.12" size="1.778" layer="96" ratio="13"/>
+</instance>
+<instance part="P11" gate="P" x="144.78" y="83.82" smashed="yes" rot="MR0">
+<attribute name="NAME" x="144.78" y="88.9" size="1.778" layer="95" ratio="13" rot="MR0"/>
+<attribute name="VALUE" x="144.78" y="86.36" size="1.778" layer="96" ratio="13" rot="MR0"/>
+</instance>
+<instance part="P12" gate="P" x="144.78" y="68.58" smashed="yes" rot="MR0">
+<attribute name="NAME" x="144.78" y="73.66" size="1.778" layer="95" ratio="13" rot="MR0"/>
+<attribute name="VALUE" x="144.78" y="71.12" size="1.778" layer="96" ratio="13" rot="MR0"/>
+</instance>
+<instance part="P13" gate="P" x="116.84" y="48.26" smashed="yes">
+<attribute name="NAME" x="116.84" y="53.34" size="1.778" layer="95" ratio="13"/>
+<attribute name="VALUE" x="116.84" y="50.8" size="1.778" layer="96" ratio="13"/>
+</instance>
+<instance part="P14" gate="P" x="116.84" y="33.02" smashed="yes">
+<attribute name="NAME" x="116.84" y="38.1" size="1.778" layer="95" ratio="13"/>
+<attribute name="VALUE" x="116.84" y="35.56" size="1.778" layer="96" ratio="13"/>
+</instance>
+<instance part="P15" gate="P" x="144.78" y="48.26" smashed="yes" rot="MR0">
+<attribute name="NAME" x="144.78" y="53.34" size="1.778" layer="95" ratio="13" rot="MR0"/>
+<attribute name="VALUE" x="144.78" y="50.8" size="1.778" layer="96" ratio="13" rot="MR0"/>
+</instance>
+<instance part="P16" gate="P" x="144.78" y="33.02" smashed="yes" rot="MR0">
+<attribute name="NAME" x="144.78" y="38.1" size="1.778" layer="95" ratio="13" rot="MR0"/>
+<attribute name="VALUE" x="144.78" y="35.56" size="1.778" layer="96" ratio="13" rot="MR0"/>
+</instance>
+<instance part="SHEET1" gate="SH" x="0" y="0" smashed="yes">
+<attribute name="DRAWING_NAME" x="166.37" y="21.59" size="2.54" layer="97"/>
+<attribute name="REVISION" x="194.31" y="16.51" size="5.08" layer="97" align="center"/>
+<attribute name="SHEET" x="194.31" y="8.89" size="5.08" layer="97" align="center"/>
+<attribute name="VALUE" x="166.37" y="36.83" size="2.54" layer="97"/>
+<attribute name="LAST_DATE_TIME" x="210.82" y="6.35" size="2.54" layer="97"/>
+<attribute name="CIRCUIT_NAME" x="166.37" y="29.21" size="2.54" layer="97"/>
+<attribute name="CIRCUIT_CATEGORY" x="186.69" y="21.59" size="2.54" layer="97"/>
+</instance>
+<instance part="SHEET1" gate="G$1" x="182.88" y="177.8" smashed="yes"/>
 </instances>
 <busses>
