File: miniPCB/13/A/13A-777/13A-777.sch (EAGLE design)
At the start: 38 parts, among them Q1 JFET-N2N5484, Q2 JFET-N2N5484, Q3 JFET-N2N5484, Q4 JFET-N2N5484, SW1 PEL12T, U2 MCP4451-502E/ML

Commit message: NM.17JAN2023
Parts:
- added C16, C18, C19, C20, C21, C22, C23, C24, C25, C26, C27, C29, C31, C32: 100n, minipcb:CAPACITORSMD
- added C17, C28, C30: 1u, minipcb:CAPACITORSMD
- added Q5, Q6: NTR2101P, minipcb:MOSFET-PNTR2101PT1G
- added R14, R16, R18, R19, R23, R24, R27, R28, R31, R32, R35, R36, R37, R38, R39, R40, R41, R42: 10k, minipcb:RESISTORSMD
- added R15, R17: 499K, minipcb:RESISTORSMD
- added R20, R21, R25, R29, R33, R43: 10K, minipcb:RESISTORSMD
- added R22, R26, R30, R34: 149K, minipcb:RESISTORSMD
- added R44: 149, minipcb:RESISTORSMD
- added U3, U4, U5, U6: (no value), minipcb:OPAMP_SINGLESMD
- C1, C11, C7: value (none) -> 1u
- C10, C12, C13, C14, C15, C6, C8, C9: value (none) -> 100n
- Q1, Q2, Q3, Q4: value JFET-N2N5484 -> JFET-N, SOT23
- R1, R8, R9: value (none) -> 10k
- R10, R11, R12, R3, R4, R5, R6, R7: value (none) -> 149
- R13: value (none) -> 499K
- R2: value (none) -> 10K
Connections:
- removed net Q1_SIGNAL: Q1.SOURCE, R3.2
- removed net Q2_SIGNAL: Q2.SOURCE, R4.2
- removed net Q4_SIGNAL: Q4.SOURCE, R6.2
- new net B1: B1.2, R2.1, R43.2
- new net ELECTROSCOPE_BIAS: R40.1, U1.21.RA2
- new net ELECTROSCOPE_VCC: C7.+, C8.+, Q1.DRAIN, Q2.DRAIN, Q3.DRAIN, Q4.DRAIN, Q5.D
- new net ELECTROSCOPE_VCC1: Q6.D, SW1.5.+
- new net ENCODER_RESET: R16.2, U1.2.RD4
- new net N$10: R37.1, R38.2
- new net N$11: R38.1, R39.2
- new net N$12: C32.+, R39.1, R40.2
- new net N$13: R44.2, U$1.1.MCLR/VPP
- new net N$4: Q5.G, R14.1, R15.2
- new net N$7: Q6.G, R16.1, R17.2
- new net N$8: R19.1, SW1.A
- new net N$9: R20.2, SW1.3.SW
- new net Q1-ADC: C19.+, R24.2, U1.19.RA0
- new net Q1.1: Q1.SOURCE, R21.2, R3.2
- new net Q2-ADC: C22.+, R28.2, U1.20.RA1
- new net Q2.1: Q2.SOURCE, R25.2, R4.2
- new net Q3-ADC: C26.+, R36.2, U1.22.RA3
- new net Q4-ADC: C24.+, R32.2, U1.23.RA4
- new net Q4.1: Q4.SOURCE, R29.2, R6.2
- new net U3.1: R23.1, R24.1, U3A.OUT
- new net U3.3: C16.+, R21.1, U3A.+IN
- new net U3.4: C16.-, C9.+, R22.1, R23.2, U3A.-IN
- new net U4.1: R27.1, R28.1, U4A.OUT
- new net U4.2: C21.+, R25.1, U4A.+IN
- new net U4.4: C20.+, C21.-, R26.1, R27.2, U4A.-IN
- new net U5.1: R31.1, R32.1, U5A.OUT
- new net U5.3: C23.+, R29.1, U5A.+IN
- new net U5.4: C10.+, C23.-, R30.1, R31.2, U5A.-IN
- new net U6.1: R35.1, R36.1, U6A.OUT
- new net U6.3: C25.+, R33.1, U6A.+IN
- new net U6.4: C12.+, C25.-, R34.1, R35.2, U6A.-IN
- net +3V3: now also C11.+, C17.+, C18.+, C27.+, C28.+, C29.+, C30.+, C31.+, Q5.S, Q6.S, R15.1, R17.1, R41.2, R42.2, U3-PWR.V+, U4-PWR.V+, U5-PWR.V+, U6-PWR.V+
- net BUTTON: now also R43.1; no longer B1.2, R2.1
- net ELECTROSCOPE_ENABLE: now also U2.!RESET; no longer C7.+, C8.+, Q1.DRAIN, Q2.DRAIN, Q3.DRAIN, Q4.DRAIN
- net ELECTROSCOPE_RESET: now also R14.2; no longer U2.!RESET
- net ENC_A: now also R19.2, U1.4.RD6; no longer SW1.A
- net ENC_B: now also R18.2, U1.5.RD7; no longer SW1.B
- net ENC_BLUE: now also U1.25.RE0
- net ENC_GREEN: now also U1.11.RB3
- net ENC_RED: now also U1.8.RB0
- net ENC_SW: now also R20.1, U1.3.RD5; no longer SW1.3.SW
- net GND: now also C17.-, C18.-, C19.-, C20.-, C22.-, C24.-, C26.-, C27.-, C28.-, C29.-, C30.-, C31.-, C32.-, U3-PWR.V-, U4-PWR.V-, U5-PWR.V-, U6-PWR.V-
- net MCLR: now also R44.1; no longer U$1.1.MCLR/VPP
- net N$6: now also R18.1, SW1.B; no longer SW1.5.+
- net Q1_W: now also R22.2; no longer C9.+
- net Q2_W: now also R26.2; no longer C10.+
- net Q3_SIGNAL: now also R33.2
- net Q3_W: now also R34.2; no longer C11.+
- net Q4_W: now also R30.2; no longer C12.+
- net SCL: now also R41.1
- net SDA: now also R42.1
Other:
- note added: "QUADRANT 1"
- note added: "QUADRANT 2"
- note added: "QUADRANT 3"
- note added: "QUADRANT 4"

Commit message: NM.17JAN2023
Parts:
- R23, R27, R31, R35: value 10k -> 149K
Connections:
- net GND: no longer C10.-, C12.-, C20.-, C9.-
- net U3.1: now also C9.-
- net U4.1: now also C20.-
- net U5.1: now also C10.-
- net U6.1: now also C12.-
Other:
- moved on the sheet: C10, C12, C20, C9

Commit message: NM.18JAN2023
Parts:
- removed C23, C24, C25, C26, C27, C29, C31, C32: 100n, minipcb:CAPACITORSMD
- removed C28, C30: 1u, minipcb:CAPACITORSMD
- removed Q4: JFET-N, SOT23, minipcb:JFET-N2N5484
- removed Q5, Q6: NTR2101P, minipcb:MOSFET-PNTR2101PT1G
- removed R28, R32, R36, R37, R38, R39, R40, R41, R42: 10k, minipcb:RESISTORSMD
- removed R29, R33: 10K, minipcb:RESISTORSMD
- removed R30, R31, R34, R35: 149K, minipcb:RESISTORSMD
- removed U6: (no value), minipcb:OPAMP_SINGLESMD
- added B2: 18650, minipcb:BATTERY18650-NOHOLES
- added F1: 1A, minipcb:FUSE-1812-1A
- added J1: (no value), minipcb:USB
- added LED2: (no value), minipcb:LEDCHIP-LED0805
- added X1: HD44780LCD-VIVA, minipcb:HD44780LCD-VIVA
- C1, C11, C17, C2, C5: value 1u -> 680n
- C10, C12, C13, C14, C15, C18, C19, C21, C22, C6, C8, C9: value 100n -> 680n
- C16, C20: value 100n -> 4u7
- C3, C4: value 10n -> 680n
- C7: value 1u -> 4u7
- Q1, Q2: value JFET-N, SOT23 -> NTR2101P; device minipcb:JFET-N2N5484 -> minipcb:MOSFET-PNTR2101PT1G
- Q3: value JFET-N, SOT23 -> 2N7002; device minipcb:JFET-N2N5484 -> minipcb:MOSFET-NSOT23
- R10, R11, R12, R3, R44, R7: value 149 -> 150
- R14: value 10k -> 4K7
- R15: value 499K -> 4K7
- R16: value 10k -> 499K
- R17: value 499K -> 4K99
- R21: value 10K -> 1K
- R22: value 149K -> 4K99
- R23: value 149K -> 10k
- R25: value 10K -> 150
- R26: value 149K -> 2K
- R27: value 149K -> 1K
- R4, R5: value 149 -> 10k
- R6: value 149 -> 499K
- U1: value (none) -> PIC16F1789T-I/PT
- U2: value MCP4451-502E/ML -> MCP4017T-502E/LT; device minipcb:MCP4451-502E/MLQFN20_4X4MC_MCH -> minipcb:MCP4017T-502E/LTSC70-6_MC_MCH
- U3, U5: value (none) -> ADP150AUJZ-3.3-R7; device minipcb:OPAMP_SINGLESMD -> minipcb:ADP150
- U4: device minipcb:OPAMP_SINGLESMD -> minipcb:MCP73831T-2ATI/OTSOT-23-5_MC_MCH
Connections:
- net N$2 renamed SW1.1
- net N$3 renamed SW1.2
- net N$5 renamed SW1.4
- net N$9 renamed SW1.3
- removed net A0: U1.41.RD3, U2.HVC/A0
- removed net A1: U1.40.RD2, U2.A1
- removed net ELECTROSCOPE_BIAS: R40.1, U1.21.RA2
- removed net ELECTROSCOPE_ENABLE: U1.38.RD0, U2.!RESET
- removed net ELECTROSCOPE_RESET: R14.2, U1.39.RD1
- removed net ELECTROSCOPE_VCC: C7.+, C8.+, Q1.DRAIN, Q2.DRAIN, Q3.DRAIN, Q4.DRAIN, Q5.D
- removed net ELECTROSCOPE_VCC1: Q6.D, SW1.5.+
- removed net N$8: R19.1, SW1.A
- removed net Q1-ADC: C19.+, R24.2, U1.19.RA0
- removed net Q1.1: Q1.SOURCE, R21.2, R3.2
- removed net Q1_W: R22.2, R3.1, U2.P0W
- removed net Q2-ADC: C22.+, R28.2, U1.20.RA1
- removed net Q2.1: Q2.SOURCE, R25.2, R4.2
- removed net Q2_W: R26.2, R4.1, U2.P1W
- removed net Q3-ADC: C26.+, R36.2, U1.22.RA3
- removed net Q3_SIGNAL: Q3.SOURCE, R33.2, R5.2
- removed net Q3_W: R34.2, R5.1, U2.P2W
- removed net Q4-ADC: C24.+, R32.2, U1.23.RA4
- removed net Q4.1: Q4.SOURCE, R29.2, R6.2
- removed net Q4_W: R30.2, R6.1, U2.P3W
- removed net U3.1: C9.-, R23.1, R24.1, U3A.OUT
- removed net U3.3: C16.+, R21.1, U3A.+IN
- removed net U3.4: C16.-, C9.+, R22.1, R23.2, U3A.-IN
- removed net U4.1: C20.-, R27.1, R28.1, U4A.OUT
- removed net U4.2: C21.+, R25.1, U4A.+IN
- removed net U4.4: C20.+, C21.-, R26.1, R27.2, U4A.-IN
- removed net U5.1: C10.-, R31.1, R32.1, U5A.OUT
- removed net U5.3: C23.+, R29.1, U5A.+IN
- removed net U5.4: C10.+, C23.-, R30.1, R31.2, U5A.-IN
- removed net U6.1: C12.-, R35.1, R36.1, U6A.OUT
- removed net U6.3: C25.+, R33.1, U6A.+IN
- removed net U6.4: C12.+, C25.-, R34.1, R35.2, U6A.-IN
- new net DAC1: R21.2, U1.21.RA2
- new net DAC1OUT1: U2.W, X1.VO
- new net DAC1_OUT1: C11.+, R21.1, R27.1, U1.22.RA3
- new net LCD-D0: U1.8.RB0, X1.DB0
- new net LCD-D1: U1.9.RB1, X1.DB1
- new net LCD-D2: U1.10.RB2, X1.DB2
- new net LCD-D3: U1.11.RB3, X1.DB3
- new net LCD-RE: U1.40.RD2, X1.E
- new net LCD-RS: U1.38.RD0, X1.RS
- new net LCD-RW: U1.39.RD1, X1.RW
- new net LCD_BACKLIGHT_RESET: R5.2, U1.41.RD3
- new net LCD_ENABLE: R3.2, U1.43.RC5
- new net N$14: R26.1, U4.PROG
- new net N$15: R3.1, U3.EN
- new net N$2: Q1.G, R16.2, R4.1
- new net N$3: Q3.D, R23.2, R24.1, R4.2, U1.20.RA1
- new net N$5: R17.1, R22.2, U1.19.RA0
- new net N$9: R25.1, U4.STAT
- new net OPA1IN-: U1.24.RA5
- new net SW1.A: R19.1, R8.1, SW1.A
- new net SW1.B: R18.1, R9.1, SW1.B
- new net VDD1: C8.+, Q2.D, X1.A
- new net VSS: X1.VSS
- net +3V3: now also C12.+, C16.+, C19.+, C20.+, C21.+, C22.+, C7.+, F1.2, Q1.S, Q2.S, R14.2, R15.2, R16.1, R6.1, SW1.5.+, U1.28.VDD, U1.7.VDD, U3.VIN, U3.VOUT, U4.VBAT, U5.EN, U5.VIN, U5.VOUT, X1.VDD; no longer C11.+, C27.+, C28.+, C29.+, C30.+, C31.+, Q5.S, Q6.S, R15.1, R17.1, R41.2, R42.2, U3-PWR.V+, U4-PWR.V+, U5-PWR.V+, U6-PWR.V+
- net ENCODER_RESET: no longer R16.2
- net ENC_A: no longer R8.1
- net ENC_B: no longer R9.1
- net ENC_GREEN: now also U1.35.RC1; no longer U1.11.RB3
- net ENC_RED: now also U1.36.RC2; no longer U1.8.RB0
- net GND: now also B2.-, C10.-, C12.-, C16.-, C20.-, C21.-, C9.-, J1.5.GND, Q3.S, R22.1, R24.2, R26.2, R27.2, U2.B, U3.GND, U4.VSS, U5.GND, X1.K; no longer C24.-, C26.-, C27.-, C28.-, C29.-, C30.-, C31.-, C32.-, U2.EPAD, U2.P0B, U2.P1B, U2.P2B, U2.P3B, U3-PWR.V-, U4-PWR.V-, U5-PWR.V-, U6-PWR.V-
- net N$10: now also C10.+, Q2.G, R5.1, R6.2; no longer R37.1, R38.2
- net N$11: now also B2.+, F1.1; no longer R38.1, R39.2
- net N$12: now also LED2.C, R25.2; no longer C32.+, R39.1, R40.2
- net N$4: now also C9.+, Q1.D, R17.2; no longer Q5.G, R14.1, R15.2
- net N$6: now also Q3.G, R23.1; no longer R18.1, SW1.B
- net N$7: now also J1.1.VCC, LED2.A, U4.VDD; no longer Q6.G, R16.1, R17.2
- net SCL: now also R14.1; no longer R41.1
- net SDA: now also R15.1; no longer R42.1
Other:
- note removed: "QUADRANT 1"
- note removed: "QUADRANT 2"
- note removed: "QUADRANT 3"
- note removed: "QUADRANT 4"

Commit message: NM.28JAN2023
Parts:
- removed B2: 18650, minipcb:BATTERY18650-NOHOLES
- removed C22: 680n, minipcb:CAPACITORSMD
- removed R43: 10K, minipcb:RESISTORSMD
- removed R44: 150, minipcb:RESISTORSMD
- removed U5: ADP150AUJZ-3.3-R7, minipcb:ADP150
- added BT1: 18650, minipcb:BATTERY18650-NOHOLES
- added LED3: (no value), minipcb:LEDCHIP-LED0805
- added PCB: PCB-50/100-0, minipcb:MINIPCB_0P50X100MM
- added Q4: NTR2101P, minipcb:MOSFET-PNTR2101PT1G
- added R28, R29, R30: 10k, minipcb:RESISTORSMD
- added R31: 499K, minipcb:RESISTORSMD
- added R32: 150, minipcb:RESISTORSMD
- C1, C11, C13, C14, C15, C19, C2, C21, C4, C5, C6, C8, C9: device minipcb:CAPACITORSMD -> minipcb:CAPACITOR1206
- C10: value 680n -> 4u7; device minipcb:CAPACITORSMD -> minipcb:CAPACITOR1206
- C12: value 680n -> 22u 25V; device minipcb:CAPACITORSMD -> minipcb:CAPACITOR_10
- C16: value 4u7 -> 22u 25V; device minipcb:CAPACITORSMD -> minipcb:CAPACITOR_10
- C17, C18, C3: value 680n -> 6n8; device minipcb:CAPACITORSMD -> minipcb:CAPACITOR1206
- C20: value 4u7 -> 680n; device minipcb:CAPACITORSMD -> minipcb:CAPACITOR1206
- C7: value 4u7 -> 6n8; device minipcb:CAPACITORSMD -> minipcb:CAPACITOR1206
- Q1: value NTR2101P -> 2N7002; device minipcb:MOSFET-PNTR2101PT1G -> minipcb:MOSFET-NSOT23
- R10, R3: value 150 -> 10K
- R11: value 150 -> 499K
- R13: value 499K -> 150
- R14, R15: value 4K7 -> 150
- R16, R6: value 499K -> 10k
- R17: value 4K99 -> 10k
- R18: value 10k -> 2K
- R2: value 10K -> 10k
- R20: value 10K -> 499K
- R21: value 1K -> 4K99
- R23, R4, R8: value 10k -> 150
- R24: value 10k -> 1K
- R25: value 150 -> 1K
- R26: value 2K -> 1K
- R27: value 1K -> 150
- R5: value 10k -> 10K
- R7: value 150 -> 10k
- U2: value MCP4017T-502E/LT -> MCP73831; device minipcb:MCP4017T-502E/LTSC70-6_MC_MCH -> minipcb:MCP73831T-2ATI/OTSOT-23-5_MC_MCH
- U4: value (none) -> ADP150AUJZ-3.3-R7; device minipcb:MCP73831T-2ATI/OTSOT-23-5_MC_MCH -> minipcb:ADP150
- X1: value HD44780LCD-VIVA -> HD44780LCD-1602; device minipcb:HD44780LCD-VIVA -> minipcb:HD44780LCD-1602
Connections:
- removed net DAC1: R21.2, U1.21.RA2
- removed net DAC1OUT1: U2.W, X1.VO
- removed net DAC1_OUT1: C11.+, R21.1, R27.1, U1.22.RA3
- removed net ENCODER_RESET: U1.2.RD4
- removed net LCD_BACKLIGHT_RESET: R5.2, U1.41.RD3
- removed net N$1: LED1.C, R7.2
- removed net N$10: C10.+, Q2.G, R5.1, R6.2
- removed net N$11: B2.+, F1.1
- removed net N$12: LED2.C, R25.2
- removed net N$13: R44.2, U$1.1.MCLR/VPP
- removed net N$14: R26.1, U4.PROG
- removed net N$15: R3.1, U3.EN
- removed net N$2: Q1.G, R16.2, R4.1
- removed net N$3: Q3.D, R23.2, R24.1, R4.2, U1.20.RA1
- removed net N$4: C9.+, Q1.D, R17.2
- removed net N$5: R17.1, R22.2, U1.19.RA0
- removed net N$6: Q3.G, R23.1
- removed net N$7: J1.1.VCC, LED2.A, U4.VDD
- removed net N$9: R25.1, U4.STAT
- removed net OPA1IN-: U1.24.RA5
- removed net SCL: R14.1, U1.37.RC3, U2.SCL
- removed net SDA: R15.1, U1.42.RC4, U2.SDA
- removed net UART_MCU_RX: U1.1.RC7
- removed net UART_MCU_TX: U1.44.RC6
- removed net VDD1: C8.+, Q2.D, X1.A
- removed net VSS: X1.VSS
- new net +3V3-LCD: C16.+, C18.+, C21.+, Q4.S, R31.1, R6.2, R7.2, SW1.5.+, U4.VOUT, X1.VDD
- new net BT+: BT1.+, F1.1, LED3.A
- new net LCD-BACKLIGHT-A: R32.2, X1.A
- new net LCD-BACKLIGHT-ENABLE: R28.1, R29.2, U1.11.RB3
- new net LCD-D4: U1.3.RD5, X1.DB4
- new net LCD-D5: U1.4.RD6, X1.DB5
- new net LCD-D6: U1.5.RD7, X1.DB6
- new net LCD-D7: U1.8.RB0, X1.DB7
- new net LCD-V0: C13.+, R24.1, R25.1, R26.1, X1.VO
- new net LED1.K: LED1.C, R4.2
- new net LED2.K: LED2.C, R12.2
- new net LED3K: LED3.C, R23.2
- new net P1-1: R8.2, U$1.1.MCLR/VPP
- new net PROG: R18.1, U2.PROG
- new net Q1.D: Q1.D, R19.2
- new net Q1.G: Q1.G, R17.1
- new net Q2.G: Q2.G, R19.1, R20.2
- new net Q2.S: C11.+, Q2.D, R21.2
- new net Q3.D: Q3.D, R30.2
- new net Q3.G: Q3.G, R29.1
- new net Q4.G: C19.+, Q4.G, R30.1, R31.2
- new net Q4.S: Q4.D, R32.1
- new net RA0: R21.1, R22.2, U1.19.RA0
- new net RA1: R16.1, R17.2, U1.20.RA1
- new net RA2: R25.2, U1.21.RA2
- new net RA3: R24.2, U1.22.RA3
- new net U4.1: R12.1, U2.STAT
- new net U4.3: R27.1, U4.EN
- new net VBAT: C10.+, C12.+, C14.+, C15.+, F1.2, Q2.S, R20.1, R23.1, U2.VBAT, U3.EN, U3.VIN, U4.VIN
- new net VUSB: J1.1.VCC, LED2.A, U2.VDD
- net +3V3: now also C1.+, C6.+, R3.2; no longer C12.+, C16.+, C18.+, C19.+, C2.+, C21.+, C22.+, C4.+, C5.+, F1.2, Q1.S, Q2.S, R1.2, R14.2, R15.2, R16.1, R2.2, R6.1, R8.2, SW1.5.+, U2.VDD, U3.VIN, U4.VBAT, U5.EN, U5.VIN, U5.VOUT, X1.VDD
- net B1: now also C5.+, R3.1, R5.2; no longer R2.1, R43.2
- net BUTTON: now also R5.1; no longer C6.+, R43.1
- net ENC_A: now also R1.2, U1.38.RD0; no longer C13.+, R19.2, U1.4.RD6
- net ENC_B: now also R2.2, U1.37.RC3; no longer C14.+, R18.2, U1.5.RD7
- net ENC_BLUE: now also R15.1, U1.36.RC2; no longer R12.1, U1.25.RE0
- net ENC_GREEN: now also R14.1; no longer R11.1
- net ENC_RED: now also R13.1, U1.25.RE0; no longer R10.1, U1.36.RC2
- net ENC_SW: now also C9.+, R10.1, R11.2, U1.39.RD1; no longer C15.+, R13.2, R20.1, U1.3.RD5
- net GND: now also BT1.-, Q1.S, R11.1, R16.2, R18.2, R28.2, U4.GND, X1.VSS; no longer B2.-, C22.-, R13.1, R24.2, R27.2, U2.B, U4.VSS, U5.GND
- net LCD-D0: now also U1.43.RC5; no longer U1.8.RB0
- net LCD-D1: now also U1.44.RC6; no longer U1.9.RB1
- net LCD-D2: now also U1.1.RC7; no longer U1.10.RB2
- net LCD-D3: now also U1.2.RD4; no longer U1.11.RB3
- net LCD-RE: now also U1.42.RC4; no longer U1.40.RD2
- net LCD-RS: now also U1.40.RD2; no longer U1.38.RD0
- net LCD-RW: now also U1.41.RD3; no longer U1.39.RD1
- net LCD_ENABLE: now also R27.2, U1.10.RB2; no longer R3.2, U1.43.RC5
- net LED1: now also R4.1, U1.14.RB4; no longer R7.1
- net MCLR: now also C8.+, R8.1, R9.1; no longer C1.+, R1.1, R44.1
- net SW1.1: now also R13.2; no longer R10.2
- net SW1.2: now also R14.2; no longer R11.2
- net SW1.3: now also R10.2; no longer R20.2
- net SW1.4: now also R15.2; no longer R12.2
- net SW1.A: now also C2.+, R1.1, R6.1, SW1.B; no longer R19.1, R8.1, SW1.A
- net SW1.B: now also C4.+, R2.1, R7.1, SW1.A; no longer R18.1, R9.1, SW1.B
Other:
- moved on the sheet: C1, C10, C11, C12, C13, C14, C15, C16, C17, C18, C19, C2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

Commit message: NM.24FEB2023
Parts:
- removed LED3: (no value), minipcb:LEDCHIP-LED0805
- removed R23: 150, minipcb:RESISTORSMD
- C12, C16: device minipcb:CAPACITOR_10 -> minipcb:CAPACITOR3.5MM
- J1: device minipcb:USB -> minipcb:USB2LUG
- PCB: PART_NUMBER 13A-777-A-XA -> 13A-777-A-XB
Connections:
- removed net LED3K: LED3.C, R23.2
- net BT+: no longer LED3.A
- net ENC_A: now also U1.27.RE2; no longer U1.38.RD0
- net ENC_B: now also U1.26.RE1; no longer U1.37.RC3
- net ENC_SW: now also U1.24.RA5; no longer U1.39.RD1
- net GND: now also J1.6.SHIELD
- net LCD_ENABLE: now also U1.23.RA4; no longer U1.10.RB2
- net VBAT: no longer R23.1
