File: miniPCB/13/A/13A-777/13A-777.brd (EAGLE design)
At the start: 100 x 50 mm, 72 parts, among them Q1 2N7002, Q2 NTR2101P, Q3 2N7002, Q4 NTR2101P, SW1 PEL12T, U1 PIC16F1789T-I/PT, U2 MCP73831, U3 ADP150AUJZ-3.3-R7, U4 ADP150AUJZ-3.3-R7, X1 HD44780LCD-1602

Commit message: NM.24FEB2023
Parts:
- removed LED3: (no value), minipcb:CHIP-LED0805
- removed R23: 150, minipcb:R0805
- C12, C16: device minipcb:C5MM -> minipcb:C3-5MM
- J1: device minipcb:USB_MICRO -> minipcb:USB_MICRO_B
- moved R27 33.4 mm to (51.0, 25.0), turned to 0 degrees
- moved R11 24.7 mm to (4.50, 16.6), turned to 180 degrees
- moved C9 24.4 mm to (4.50, 19.1), turned to 0 degrees
- moved R10 19.7 mm to (4.50, 21.6), turned to 0 degrees
- moved C18 13.3 mm to (74.5, 37.0), turned to 0 degrees
- moved C21 12.5 mm to (74.5, 34.5), turned to 0 degrees
- moved Q1 12.4 mm to (56.2, 31.0)
- moved R19 12.3 mm to (57.0, 34.5), turned to 270 degrees
- moved C6 11.9 mm to (28.7, 32.3), turned to 90 degrees
- moved R24 11.0 mm to (14.4, 21.9), turned to 180 degrees
- moved C7 10.4 mm to (31.1, 32.3), turned to 90 degrees
- moved LED2 9.63 mm to (90.1, 25.6), turned to 180 degrees
- moved R25 9.16 mm to (14.4, 19.9), turned to 180 degrees
- moved R20 8.80 mm to (59.0, 34.5), turned to 90 degrees
- moved C17 8.20 mm to (73.5, 26.5), turned to 270 degrees
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Connections:
- removed net LED3K: LED3.C, R23.2
- net BT+: no longer LED3.A
- net ENC_A: now also U1.27; no longer U1.38
- net ENC_B: now also U1.26; no longer U1.37
- net ENC_SW: now also U1.24; no longer U1.39
- net GND: now also J1.GND10, J1.GND5, J1.GND6, J1.GND7, J1.GND8, J1.GND9, J1.XPAD3, J1.XPAD4
- net LCD_ENABLE: now also U1.23; no longer U1.10
- net VBAT: no longer R23.1
Routing:
- net LCD_ENABLE: track 44.2 -> 16.4 mm, vias 2 -> 0
- net U4.3: track 4.89 -> 30.0 mm
- net ICSPCLK: track 66.0 -> 41.1 mm
- net +3V3-LCD: track 15.9 -> 39.7 mm, vias 6 -> 3
- net RA0: track 32.3 -> 56.0 mm, vias 0 -> 2
- net LCD-V0: track 75.5 -> 52.8 mm, vias 0 -> 1
- net BUTTON: track 41.7 -> 63.9 mm, vias 0 -> 2
- net RA1: track 14.7 -> 36.8 mm, vias 0 -> 2
- net ICSPDAT: track 60.9 -> 43.6 mm, vias 2 -> 0
- net SW1.B: track 47.2 -> 30.8 mm
- net SW1.A: track 39.2 -> 23.8 mm
- net LED1: track 74.0 -> 59.7 mm, vias 0 -> 2
- net ENC_SW: track 23.6 -> 37.8 mm
- net ENC_RED: track 46.0 -> 32.5 mm
- net VBAT: track 51.0 -> 62.0 mm, vias 0 -> 1
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Other:
- board text removed: "LED3"
- board text removed: "R23"

Commit message: NM.26NOV2024
Changed lines of the file:
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@@
 </layers>
 <board>
-<fusionsync huburn="a.cGVyc29uYWw6dWUyYTE3NGFm" projecturn="a.cGVyc29uYWw6dWUyYTE3NGFmIzIwMjMwMTIzNjAwOTI1NDUx" f3durn="urn:adsk.wipprod:dm.lineage:8F-dwzJJS3-J1EJKGrBEVg" pcbguid="" lastpulledtime="" lastsyncedchangeguid="" latestrevisionid="3a7591c4-de92-4145-851f-6bdf0c000477" lastsyncedrevisionid="3a7591c4-de92-4145-851f-6bdf0c000477" lastboardhashguid="51ed9cf1-2ef0-75af-49c9-db2a46c9702f" lastpushedtime="2023-01-23T02:27:52Z" linktopcb3d="true"/>
 <plain>
 <text x="60.00000625" y="13.81000625" size="0.9" layer="122" font="vector" ratio="12" rot="MR0">BT1</text>
@@
 <param name="checkFont" value="1"/>
 <param name="checkRestrict" value="1"/>
-<param name="checkStop" value="0"/>
-<param name="checkValues" value="0"/>
-<param name="checkNames" value="1"/>
-<param name="checkWireStubs" value="1"/>
-<param name="checkPolygonWidth" value="0"/>
 <param name="useDiameter" value="13"/>
 <param name="maxErrors" value="50"/>
@@
 <pass name="Default">
 <param name="RoutingGrid" value="50mil"/>
-<param name="AutoGrid" value="1"/>
-<param name="Efforts" value="0"/>
-<param name="TopRouterVariant" value="1"/>
 <param name="tpViaShape" value="round"/>
-<param name="PrefDir.1" value="a"/>
 <param name="PrefDir.2" value="0"/>
 <param name="PrefDir.3" value="0"/>
@@
 <param name="PrefDir.14" value="0"/>
 <param name="PrefDir.15" value="0"/>
-<param name="PrefDir.16" value="a"/>
 <param name="cfVia" value="8"/>
 <param name="cfNonPref" value="5"/>
@@
 <element name="PCB" library="minipcb" package="MINIPCB_0P_50X100MM" value="PCB-50/100-0" x="0" y="0" smashed="yes">
 <attribute name="PART_NUMBER" value="13A-777-A-XB" x="94.5" y="47.5" size="1.5" layer="16" font="vector" ratio="13" rot="MR180" align="center-right"/>
-<attribute name="PART_NUMBER" value="13A-777-A-XA" x="94.5" y="47.5" size="1.5" layer="22" font="vector" ratio="13" rot="MR180" align="center-right" display="off"/>
 <attribute name="REVISION" value="A" x="0" y="0" size="1.778" layer="27" display="off"/>
 </element>
