File: miniPCB/11/A/11A-001/VIVA_PIC16/Rev 5.3/v5.3.brd (EAGLE design)
At the start: 100 x 100 mm, 69 parts, among them J1 VDD SELECTOR, J3 ICSP, J4 PICKIT3, J7 2.1 MM, U1 VIVA_UTSA-KEYPADV5, U2 VIVA_USB-TTL, U3 PIC16F1829, U4 VIVA-HEADER-I2C-RA, U5 VIVA_PIC16BOARD, U6 ATMEGA328-AU, U7 VIVA_USB-TTL, U8 3.3V, U9 5.0V

Commit message: NM.28JUL2023
Parts:
- added C20, C21: (no value), utsa:C0805
- added R12, R17: 10k, utsa:R0805
- moved D4 15.9 mm to (34.5, 54.0), turned to 180 degrees
- moved D2 12.0 mm to (34.5, 57.0), turned to 180 degrees
- moved LED3 7.07 mm to (22.5, 40.5), turned to 90 degrees
- moved C7 4.74 mm to (61.1, 61.3), turned to 180 degrees
- moved R15 4.61 mm to (20.0, 40.5), turned to 270 degrees
- moved A1 4.24 mm to (86.0, 85.0)
- moved C16 4.03 mm to (28.5, 80.5)
- moved C17 4.03 mm to (28.5, 82.5)
- moved U9 4.03 mm to (21.5, 80.5)
- moved C14 3.61 mm to (29.5, 91.5)
- moved C15 3.61 mm to (29.5, 89.5)
- moved U8 3.35 mm to (22.5, 89.5)
- moved J1 3.04 mm to (5.00, 39.0), turned to 0 degrees
- moved D6 3.00 mm to (13.0, 88.5)
- moved J7 3.00 mm to (4.50, 82.0)
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Connections:
- new net B1-CAP: B1.3.B, B1.4.B, C4.1, R12.2, R4.2
- new net PD4-CAP: B4.3.B, B4.4.B, C19.1, R16.2, R17.2
- net GND: now also C20.2, C21.2
- net MCLR: no longer B2.3.B, B2.4.B
- net MCLR_CAP: now also B2.3.B, B2.4.B
- net PD4: now also R17.1; no longer B4.3.B, B4.4.B, C19.1, R16.2
- net RB7: now also R12.1; no longer B1.3.B, B1.4.B, C4.1, R4.2
- net VDD: now also C20.1, C21.1
Routing:
- net +5V: track 0.00 -> 97.7 mm
- net VDD: track 64.7 -> 142.2 mm, vias 19 -> 20
- net N$46: track 0.00 -> 56.1 mm, vias 0 -> 2
- net +3V3: track 0.00 -> 53.4 mm
- net MCLR: track 0.00 -> 42.5 mm
- net N$45: track 0.00 -> 37.4 mm
- net N$36: track 0.00 -> 36.3 mm
- net RC5: track 0.00 -> 27.9 mm
- net MCLR_CAP: track 0.00 -> 23.5 mm
- net N$48: track 0.00 -> 21.0 mm
- net RA5: track 0.00 -> 18.9 mm, vias 0 -> 2
- net N$49: track 0.00 -> 18.5 mm
- net RC4: track 0.00 -> 16.7 mm
- net N$47: track 0.00 -> 14.5 mm
- net RA2: track 0.00 -> 14.3 mm
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