File: miniPCB/11/A/11A-001/VIVA_PIC16/Rev 5.3/v5.3.sch (EAGLE design)
At the start: 69 parts, among them J1 VDD SELECTOR, J3 ICSP, J4 PICKIT3, J7 2.1 MM, U1 VIVA_UTSA-KEYPADV5, U2 VIVA_USB-TTL, U3 PIC16F1829, U4 VIVA-HEADER-I2C-RA, U5 VIVA_PIC16BOARD, U6 ATMEGA328-AU, U7 VIVA_USB-TTL, U8 3.3V, U9 5.0V

Commit message: NM.28JUL2023
Parts:
- added C20, C21: (no value), utsa:C0805
- added R12, R17: 10k, utsa:R-EU__R0805
Connections:
- new net B1-CAP: B1.2, C4.+, R12.2, R4.2
- new net PD4-CAP: B4.2, C19.+, R16.2, R17.2
- net GND: now also C20.-, C21.-
- net MCLR: no longer B2.2
- net MCLR_CAP: now also B2.2
- net PD4: now also R17.1; no longer B4.2, C19.+, R16.2
- net RB7: now also R12.1; no longer B1.2, C4.+, R4.2
- net VDD: now also C20.+, C21.+
Other:
- note added: "ATmega MICROCONTROLLER"
- note added: "GENERAL PURPOSE BUTTON"
- note added: "HELLO WORLD! LED"
- note added: "PIC MICROCONTROLLER"
- note added: "PIC16 HEADERS"
- note added: "PROGRAMMING HEADER"
- note added: "RESET BUTTON"
- note added: "UTSA CAPACITANCE KEYPAD"
- note added: "VIVA HEADERS"
- note removed: "Capacitance Keypad"
- note removed: "General Purpose Button"
- note removed: "Hello World LED"
- note removed: "PIC Microcontroller"
- note removed: "PIC16 Headers"
- note removed: "Programming Header"
- note removed: "Reset Button"
- moved on the sheet: B1, B2, B3, B4, C1, C10, C11, C12, C13, C14, C15, C16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
