File: miniPCB/04/A/04A-010/04A-010.sch (EAGLE design)
At the start: 29 parts

Commit message: NM.14JAN2023
Connections:
- net GND: now also U1-PWR.V-; no longer U1P.V-
- net V+: now also U1-PWR.V+; no longer U1P.V+

Commit message: NM.14JAN2023
Parts:
- P1-: PART_NUMBER X04A-010-B -> X04A-010-B-XB
Changed lines of the file:
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@@
 <part name="TP6" library="minipcb" deviceset="TESTPOINT" device="KE5000-SMTEXT"/>
 <part name="P1-" library="minipcb" deviceset="MINIPCB_7P" device="50">
-<attribute name="PART_NUMBER" value="X04A-010-B"/>
+<attribute name="PART_NUMBER" value="X04A-010-B-XB"/>
 <attribute name="REVISION" value="B"/>
 </part>

Commit message: NM.03SEP2023
Parts:
- removed C6: (no value), minipcb:CAPACITORTHD
- removed P1-: (no value), minipcb:MINIPCB_7P50
- added P1: (no value), minipcb:MINIPCB_7P
- added R10: (no value), minipcb:TRIMPOT0.100THD
- added R11, R12, R9: (no value), minipcb:RESISTOR10MM
- added U$1: MINIPCB_50X50, minipcb:MINIPCB_50X50
- C3, C4: device minipcb:CAPACITORTHD -> minipcb:CAPACITOR_10
- R2: device minipcb:RESISTOR10MM -> minipcb:TRIMPOT0.100THD
- R3: device minipcb:TRIMPOT0.100THD -> minipcb:RESISTOR10MM
Connections:
- new net N$1: R10.S, R9.2
- net BIAS: now also C3.+, R2.S, R4.1; no longer C4.+, R1.1, R3.S
- net BIAS_CONTROL: now also P1-6.1, R4.2; no longer P1-6.1, R1.2
- net GND: now also P1-1.1, R11.2, R12.2, R3.1; no longer C6.-, P1-1.1, R4.1
- net IN: now also P1-4.1, R6.2; no longer P1-4.1, R5.2
- net IN+: now also R12.1, R6.1; no longer R5.1
- net NC: now also P1-3.1; no longer P1-3.1
- net OUT: now also P1-5.1, R10.A, R11.1, R8.2; no longer P1-5.1, R7.2
- net POT.1: now also R2.A, R3.2; no longer R3.A, R4.2
- net POT.3: now also R1.1, R2.E; no longer R2.1, R3.E
- net V+: now also C4.+, P1-2.1, R1.2; no longer C6.+, P1-2.1, R2.2
- net VFB: now also R8.1, R9.1; no longer R6.1
- net VREF: now also R5.2; no longer P1-7.1, R8.2
- net VREF_FILTERED: now also P1-7.1, R5.1, R7.2; no longer C3.+, R6.2, R8.1
Other:
- note added: "NOTES: 1. DIMENSIONS ARE IN MILLIMETERS. 2. MANUFACTURING SPECIFICATIONS: ADDITIONAL OPTIONS AVAILABLE UPON REQUEST. 2.1 BASE MATERIAL: FR4-TG130 2.2 LAYERS: TWO (2) 2.3 COPPER WEIGHT: DEFAULT: - ONE OUNCE (1 oz) AVAILABLE UPON REQUEST: - TWO OUNCE (2 oz) 2.4 PIECES PER PANEL: FOUR (4) 2.5 PCB THICKNESS: DEFAULT: - 1.60 MM AVAILABLE UPON REQUEST: - 0.6 MM - 0.8 MM - 1.0 MM - 1.2 MM - 2.0 MM 2.6 P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"
- note added: "NOTES: 3. PERFORMANCE FUNCTIONS: 3.1 GAIN CONTROL: - ADJUSTING RESISTOR R10 CONTROLS OUTPUT GAIN. 3.2 DC BIAS CONTROL: - ADJUSTING RESISTOR R2 CONTROLS DC BIAS VOLTAGE. 4. CALIBRATION ADJUSTMENT PROCEDURE: 4.1 PURPOSE - SET OUTPUT DC BIAS TO HALF OF SUPPLY VOLTAGE. 4.2 SCOPE - PERFORM DURING CALIBRATION PROCEDURE. 4.3 PROCEDURAL NOTES - PERFORM AFTER SAFE TO TURN ON (STTO) TEST PASSES. 4.4 PROCED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"

Commit message: NM.07SEP2023
Other:
- note added: "NOTES: 1. DIMENSIONS ARE IN MILLIMETERS. 2. MANUFACTURING SPECIFICATIONS: - ADDITIONAL OPTIONS AVAILABLE UPON REQUEST. 2.1 BASE MATERIAL: FR4-TG130 2.2 LAYERS: TWO (2) 2.3 COPPER WEIGHT: DEFAULT: - ONE OUNCE (1 oz) AVAILABLE UPON REQUEST: - TWO OUNCE (2 oz) 2.4 PIECES PER PANEL: FOUR (4) 2.5 PCB THICKNESS: DEFAULT: - 1.60 MM AVAILABLE UPON REQUEST: - 0.6 MM - 0.8 MM - 1.0 MM - 1.2 MM - 2.0 MM 2.6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"
- note added: "NOTES: 3. PROCEDURE: SAFE TO TURN ON (STTO) TEST: - PERFORM BEFORE APPLYING POWER. 3.1 MEASURE RESISTANCE: - MEASURE RESISTANCE BETWEEN TP10 AND TP11. 3.2 DETERMINE RESULT: - LOWER LIMIT: 100 OHMS - TARGET VALUE: TBD - UPPER LIMIT: N/A 4. PROCEDURE: DC VOLTAGE BIAS ADJUSTMENT: - PERFORM AFTER SAFE TO TURN ON (STTO) TEST. - PERFORM BEFORE ADJUSTING AC VOLTAGE GAIN. 4.1 APPLY POWER: - DO NOT VIOLAT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"
- note removed: "NOTES: 1. DIMENSIONS ARE IN MILLIMETERS. 2. MANUFACTURING SPECIFICATIONS: ADDITIONAL OPTIONS AVAILABLE UPON REQUEST. 2.1 BASE MATERIAL: FR4-TG130 2.2 LAYERS: TWO (2) 2.3 COPPER WEIGHT: DEFAULT: - ONE OUNCE (1 oz) AVAILABLE UPON REQUEST: - TWO OUNCE (2 oz) 2.4 PIECES PER PANEL: FOUR (4) 2.5 PCB THICKNESS: DEFAULT: - 1.60 MM AVAILABLE UPON REQUEST: - 0.6 MM - 0.8 MM - 1.0 MM - 1.2 MM - 2.0 MM 2.6 P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"
- note removed: "NOTES: 3. PERFORMANCE FUNCTIONS: 3.1 GAIN CONTROL: - ADJUSTING RESISTOR R10 CONTROLS OUTPUT GAIN. 3.2 DC BIAS CONTROL: - ADJUSTING RESISTOR R2 CONTROLS DC BIAS VOLTAGE. 4. CALIBRATION ADJUSTMENT PROCEDURE: 4.1 PURPOSE - SET OUTPUT DC BIAS TO HALF OF SUPPLY VOLTAGE. 4.2 SCOPE - PERFORM DURING CALIBRATION PROCEDURE. 4.3 PROCEDURAL NOTES - PERFORM AFTER SAFE TO TURN ON (STTO) TEST PASSES. 4.4 PROCED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"
- moved on the sheet: C1, C2, C3, C4, C5, C7, P1-1, P1-2, P1-3, P1-4, P1-5, P1-6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

Commit message: NM.21SEP2023
Other:
- moved on the sheet: C1, C2, C3, C4, C5, C7, P1-1, P1-2, P1-3, P1-4, P1-5, P1-6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

Commit message: NM.07MAR2024
Other:
- note added: "NOTES:"
- note removed: "NOTES: 1. DIMENSIONS ARE IN MILLIMETERS. 2. MANUFACTURING SPECIFICATIONS: - ADDITIONAL OPTIONS AVAILABLE UPON REQUEST. 2.1 BASE MATERIAL: FR4-TG130 2.2 LAYERS: TWO (2) 2.3 COPPER WEIGHT: DEFAULT: - ONE OUNCE (1 oz) AVAILABLE UPON REQUEST: - TWO OUNCE (2 oz) 2.4 PIECES PER PANEL: FOUR (4) 2.5 PCB THICKNESS: DEFAULT: - 1.60 MM AVAILABLE UPON REQUEST: - 0.6 MM - 0.8 MM - 1.0 MM - 1.2 MM - 2.0 MM 2.6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"
- note removed: "NOTES: 3. PROCEDURE: SAFE TO TURN ON (STTO) TEST: - PERFORM BEFORE APPLYING POWER. 3.1 MEASURE RESISTANCE: - MEASURE RESISTANCE BETWEEN TP10 AND TP11. 3.2 DETERMINE RESULT: - LOWER LIMIT: 100 OHMS - TARGET VALUE: TBD - UPPER LIMIT: N/A 4. PROCEDURE: DC VOLTAGE BIAS ADJUSTMENT: - PERFORM AFTER SAFE TO TURN ON (STTO) TEST. - PERFORM BEFORE ADJUSTING AC VOLTAGE GAIN. 4.1 APPLY POWER: - DO NOT VIOLAT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"
