File: miniPCB/04/A/04A-010/X04A-010-B-XB.brd (EAGLE design)
At the start: 100 x 100 mm, 116 parts

Commit message: NM.14JAN2023
Parts:
- added E$1: (no value), minipcb:MINIPCB_PANEL_IMAGEFRAME
- moved C11 1.50 mm to (45.5, 90.5)
- moved C18 1.50 mm to (95.5, 40.5)
- moved C25 1.50 mm to (95.5, 90.5)
- moved C4 1.50 mm to (45.5, 40.5)
- moved C1 1.00 mm to (38.0, 40.5)
- moved C10 1.00 mm to (38.0, 90.5)
- moved C17 1.00 mm to (88.0, 40.5)
- moved C24 1.00 mm to (88.0, 90.5)
Routing:
- net BIAS3: track 35.6 -> 36.5 mm
- net BIAS2: track 35.6 -> 36.5 mm
- net BIAS1: track 35.6 -> 36.5 mm
- net BIAS: track 35.6 -> 36.5 mm
Other:
- board text added: "NON-INVERTING AMPLIFIER"

Commit message: NM.07MAR2024
Changed lines of the file:
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@@
 </element>
 <element name="E$1" library="minipcb" package="MINIPCB_PANEL_IMAGEFRAME" value="" x="-25" y="-30" smashed="yes">
-<attribute name="DRAWING_NAME" x="64" y="-26.31" size="5" layer="210" align="center-left"/>
+<attribute name="DRAWING_NAME" x="56" y="-26.31" size="5" layer="210" align="center-left"/>
 </element>
 </elements>
