File: miniPCB/14/A/14A-010/14A-010.sch (EAGLE design)
At the start: 9 parts

Commit message: NM.03OCT2023
Parts:
- removed U$1: PICKIT3ARROW, minipcb:PICKIT3ARROW
- added J1, J2: 615008144221, SIG_CONNECTORS:615008144221
- added Q1: (no value), minipcb:BJT_NPNBCE
- added R5: (no value), minipcb:RESISTORSMD
- U$2: value BMD-350 -> ARDUINOMICRO; device SIG_ICS:BMD-350 -> SIG_ICS:ARDUINOMICRO
- U1: device minipcb:PIC16F1789 -> SIG_ICS:DCDC_ISOLATORRFM-XXXXS
Connections:
- removed net ICSPCLK: U$1.5.ICSPCLK/PGC, U1.16.ICSPCLK
- removed net ICSPDAT: U$1.4.ICSPDAT/PGD, U1.17.ICSPDAT
- removed net MCLR: R3.1, U$1.1.MCLR/VPP, U1.18.MCLR
- removed net N$2: C2.+, R2.1, SW1.B, U1.20.RA1
- new net ENCA: C1.+, R1.1, SW1.A
- new net ENCB: C2.+, R2.1, SW1.B
- new net OUT: R3.1, R5.2
- net GND: now also Q1.E, R5.1; no longer U$1.3.VSS, U1.29.VSS, U1.6.VSS
- net N$1: now also Q1.B, R3.2; no longer C1.+, R1.1, SW1.A, U1.19.RA0
- net VDD: no longer R3.2, U$1.2.VDD, U1.28.VDD, U1.7.VDD
Other:
- moved on the sheet: C1, C2, R1, R2, R3, SW1
