File: miniPCB/00/B/00B-003/00B-003.sch (EAGLE design)
At the start: 28 parts, among them Q1 2N7002, U1 INA290

Commit message: NM.23OCT2023
Parts:
- removed C10: 22u, nolan-utsa:C-EUC1210
- removed C11, C3, C7: 1n, nolan-utsa:C-EUC0805
- removed C4: 22u, nolan-utsa:C-EUC1210K
- removed C6, C8: 1u, nolan-utsa:C-EUC0805
- removed Q1: 2N7002, nolan-utsa:MOSFET-NSOT23
- added C12, C14: 100n, minipcb:CAPACITORSMD
- added C13: 1n, minipcb:CAPACITORSMD
- added C15: 1u, minipcb:CAPACITORSMD
- added J1: (no value), minipcb:BNC_RA
- added LED1: GREEN, minipcb:LEDCHIP-LED0805
- C1: device nolan-utsa:C-EUC0805 -> minipcb:CAPACITORSMD
- C2: value 1n -> 100p; device nolan-utsa:C-EUC0805 -> minipcb:CAPACITORSMD
- C5: device nolan-utsa:C-EUC1210 -> nolan-utsa:C-EUPCR-8X10
- C9: device nolan-utsa:C-EUC0805 -> nolan-utsa:C-EUPCR-8X10
- D1: device nolan-utsa:DIODE-SOD123-K -> minipcb:DIODESMD
- D2: value 18V -> 1N5819; device nolan-utsa:ZENER-DIODESOT23 -> minipcb:DIODESMD
- R1: device nolan-utsa:R-EU_R0805 -> minipcb:RESISTOR2512
- R2: value 270 -> 250; device nolan-utsa:R-EU_R0805 -> minipcb:RESISTORSMD
- R3: value (none) -> 22000; device nolan-utsa:R-EU_R0805 -> minipcb:RESISTORSMD
- R4: value (none) -> 1200; device nolan-utsa:R-EU_R0805 -> minipcb:RESISTORSMD
- R5: value 10k -> 250; device nolan-utsa:R-EU_R0805 -> minipcb:RESISTORSMD
- U2: value (none) -> AP3012
Connections:
- net N$1 renamed P
- net N$2 renamed N
- net N$3 renamed OUTSIGNAL
- removed net HV_DCDC: C8.1, C9.1, D1.C, Q1.D, R3.2, R5.2
- removed net N$13: C10.1, C11.1, D2.C, Q1.G, R5.1
- new net BSW: D1.A, SW1.2
- new net N$1: LED1.A, R5.1
- net B+: now also C14.+, C15.+, D1.C, R5.2; no longer C4.1, C6.1, C7.1, SW1.2
- net GND: now also C1.-, C12.-, C13.-, C14.-, C15.-, C2.-, J1.GND, LED1.C; no longer C1.2, C10.2, C11.2, C2.2, C3.2, C4.2, C6.2, C7.2, C8.2, D2.A
- net HV: now also C1.+, C12.+, C2.+, C9.1, D2.C, R3.2; no longer C1.1, C2.1, Q1.S
- net HV_SW: now also D2.A; no longer D1.A
- net SIGNAL: now also C13.+, J1.1; no longer C3.1
Other:
- note added: "NOTES: 1. MAXIMUM SENSE CURRENT LIMITED BY SHUNT RESISTANCE AND INA290 SUPPLY VOLTAGE. 2. INDUCTOR L1: SUMIDA CDTH3D14/HPNP-100NC OR EQUIVALENT. 3. AP3012 NOTES: 3.1 VIN = 2V6 to 16V 3.2 VFB = 1.25 3.3 VOUT = SET BY RESISTORS, UP TO 29V 4. INA290 GAIN VARIANTS 4.1 A1 = 20 4.2 A2 = 50 4.3 A3 = 100 4.4 A4 = 200 4.5 A5 = 500"
- note removed: "0.5 Ohm SHUNT"
- note removed: "1"
- note removed: "100"
- note removed: "1mOhm SHUNT"
- note removed: "20"
- note removed: "200"
- note removed: "50"
- note removed: "500"
- note removed: "A1"
- note removed: "A2"
- note removed: "A3"
- note removed: "A4"
- note removed: "A5"
- note removed: "AP3012 NOTES: (1) VIN = 2V6 to 16V (2) VFB = 1.25 (3) VOUT = SET BY RESISTORS, UP TO 29V"
- note removed: "ASSUME: (1) 1mOhm shunt (2) HV=18V (3) A2 variant (50x GAIN) THEN: (1) MAX CURRENT = 360A (2) CURRENT (A) = SIGNAL (mV) * (1/50)"
- note removed: "GAIN"
- note removed: "INA290 GAIN VARIANTS - A1 = 20 - A2 = 50 - A3 = 100 - A4 = 200 - A5 = 500"
- note removed: "INA290 VARIANT"
- note removed: "L: SUMIDA CDTH3D14/HPNP-100NC or Equivalent"
- note removed: "OUTPUT (mV) INPUT (uA)"
