File: miniPCB/04/B/04B-005/04B-005.brd (EAGLE design)
At the start: 28 parts

Commit message: NM.03OCT2023
Parts:
- moved TP4 12.9 mm to (17.5, 23.5)
- moved TP2 9.92 mm to (27.5, 8.50), turned to 180 degrees
- moved TP1 7.43 mm to (14.5, 12.0)
- moved C2 5.15 mm to (18.5, 8.50), turned to 0 degrees
Routing:
- net N$5: track 31.4 -> 35.0 mm
- net N$10: track 16.2 -> 13.7 mm
- net N$9: track 46.2 -> 47.3 mm

Commit message: NM.23OCT2023
Changed lines of the file:
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@@
 <elements>
 <element name="P1-" library="minipcb" package="MINIPCB_5P_50X50MM" value="" x="0" y="0" smashed="yes">
+<attribute name="CIRCUIT_CATEGORY" value="TRANSISTOR AMPLIFIERS" x="10.5" y="46.4" size="1.5" layer="21" font="vector" ratio="12" align="center-left"/>
+<attribute name="CIRCUIT_CATEGORY" value="TRANSISTOR AMPLIFIERS" x="10.5" y="46.4" size="1.5" layer="1" font="vector" ratio="12" align="center-left"/>
 <attribute name="PART_NUMBER" value="04B-005" x="45" y="48" size="1.5" layer="16" font="vector" ratio="13" rot="MR180" align="center-right"/>
 <attribute name="PART_NUMBER" value="04B-005" x="45" y="48" size="1.5" layer="22" font="vector" ratio="13" rot="MR180" align="center-right"/>
 <attribute name="REVISION" value="A1" x="40" y="46" size="1.5" layer="16" font="vector" ratio="13" rot="MR180" align="center-right"/>
 <attribute name="REVISION" value="A1" x="40" y="46" size="1.5" layer="22" font="vector" ratio="13" rot="MR180" align="center-right"/>
+<attribute name="TITLE" value="COMMON EMITTER AMPLIFIER" x="10.5" y="48.2" size="1.5" layer="21" font="vector" ratio="12" align="center-left"/>
+<attribute name="TITLE" value="COMMON EMITTER AMPLIFIER" x="10.5" y="48.2" size="1.5" layer="1" font="vector" ratio="12" align="center-left"/>
 </element>
 <element name="C2" library="minipcb" package="C050-024X044" value="" x="18.5" y="8.5" smashed="yes">
