File: miniPCB/04/B/04B-005/04B-005.sch (EAGLE design)
At the start: 28 parts

Commit message: NM.23OCT2023
Other:
- note added: "NOTES:"
- moved on the sheet: C1, C2, C3, C4, C5, P1-1, P1-2, P1-3, P1-4, P1-5, Q1, R1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
