File: miniPCB/02/A/02A-007/02A-007.brd (EAGLE design)
At the start: 160 x 100 mm, 10 parts

Commit message: NM.04NOV2023
Parts:
- removed P1.: (no value), nolan:PCB_5
- removed R6: (no value), nolan:R0805
- added P1: (no value), minipcb:PINS_1X7
- added PCB1: (no value), minipcb:MINIPCB_00A_20X25
- added R2: (no value), minipcb:R0805
- D1, D2: device nolan:SOD80C -> minipcb:DO214AC
- Q1, Q2: device nolan:SOT23 -> minipcb:SOT23
- R1, R3, R4, R5: device nolan:R0805 -> minipcb:R0805
- moved R1 43.7 mm to (18.5, 10.0), turned to 180 degrees
- moved Q2 40.6 mm to (13.5, 14.0), turned to 270 degrees
- moved R5 37.7 mm to (19.0, 16.5), turned to 270 degrees
- moved R4 35.7 mm to (10.5, 14.0), turned to 90 degrees
- moved D2 34.3 mm to (8.00, 14.0), turned to 270 degrees
- moved Q1 34.1 mm to (13.5, 7.00), turned to 270 degrees
- moved R3 33.4 mm to (10.5, 7.00), turned to 270 degrees
- moved D1 29.6 mm to (8.00, 7.00), turned to 90 degrees
Connections:
- removed net N$2: P1..3
- removed net VCC: D1.C, P1..2, Q2.2, R3.1
- new net V+: D1.C, P1.2, Q1.2, R3.2
- net GND: now also P1.1, Q2.2, R4.1; no longer P1..1, Q1.2, R4.2
- net INPUT: now also P1.4; no longer P1..4
- net N$1: now also Q1.1, R3.1; no longer Q2.1, R3.2
- net N$3: now also P1.7, Q2.3, R5.1; no longer Q1.3, R5.2
- net N$4: now also Q2.1, R2.2, R4.2; no longer Q1.1, R4.1, R6.2
- net N$5: now also P1.6, Q1.3, R5.2; no longer P1..5, Q2.3, R5.1
- net N$6: now also P1.5, R2.1; no longer R6.1
Routing:
- net GND: track 0.00 -> 31.7 mm
- net V+: track 0.00 -> 20.6 mm
- net N$4: track 0.00 -> 18.5 mm
- net N$5: track 0.00 -> 15.6 mm, vias 0 -> 1
- net N$1: track 0.00 -> 14.8 mm
- net N$3: track 0.00 -> 13.5 mm, vias 0 -> 1
- net N$6: track 0.00 -> 3.05 mm
- net INPUT: track 0.00 -> 3.05 mm
Other:
- board outline removed
