File: miniPCB/02/A/02A-007/02A-007.sch (EAGLE design)
At the start: 10 parts, among them P1. MINIPCB_4INCH

Commit message: NM.04NOV2023
Parts:
- removed P1.: MINIPCB_4INCH, nolan:MINIPCB_4INCH
- removed R6: (no value), nolan:R-EU_1%_R0805
- added P1: (no value), minipcb:MINIPCB_7P
- added PCB1: (no value), minipcb:MINIPCB_0P00A-20X25
- added R2: (no value), minipcb:RESISTORSMD
- D1, D2: value (none) -> DIODESMD; device nolan:DIODE-SOD80C -> minipcb:DIODESMD
- Q1: device nolan:BJT_NPNBEC -> minipcb:BJT_PNPBEC; MFG_PN 2N3904 -> (none)
- Q2: device nolan:BJT_PNPBEC -> minipcb:BJT_NPNBEC; MFG_PN 2N3906 -> (none)
- R1, R4: device nolan:R-EU_1%_R0805 -> minipcb:RESISTORSMD; TOLERANCE 1% -> (none)
- R3: device nolan:R-EU_1%_R0805 -> minipcb:RESISTORSMD
- R5: device nolan:R-EU__R0805 -> minipcb:RESISTORSMD
Connections:
- removed net N$2: P1.3.1
- removed net VCC: D1.C, P1.1.1, Q2.E, R3.1
- new net V+: D1.C, P1-2.1, Q1.E, R3.2
- net GND: now also P1-1.1, Q2.E, R4.1; no longer P1.2.1, Q1.E, R4.2
- net INPUT: now also P1-4.1; no longer P1.4.1
- net N$1: now also Q1.B, R3.1; no longer Q2.B, R3.2
- net N$3: now also P1-7.1, Q2.C, R5.1; no longer Q1.C, R5.2
- net N$4: now also Q2.B, R2.2, R4.2; no longer Q1.B, R4.1, R6.2
- net N$5: now also P1-6.1, Q1.C, R5.2; no longer P1.5.1, Q2.C, R5.1
- net N$6: now also P1-5.1, R2.1; no longer R6.1
Other:
- note added: "NOTES:"
- note removed: "A"
- note removed: "Part Pad Pin Dir Net D1 A A pas N$1 C C pas VCC D2 A A pas GND C C pas N$4 P1. 1 1 io GND 2 1 io VCC 3 1 io N$2 4 1 io INPUT 5 1 io N$5 Q1 1 B pas N$4 2 E pas GND 3 C pas N$3 Q2 1 B pas N$1 2 E pas VCC 3 C pas N$5 R1 1 1 pas INPUT 2 2 pas N$1 R3 1 1 pas VCC 2 2 pas N$1 R4 1 1 pas N$4 2 2 pas GND R5 1 1 pas N$5 2 2 pas N$3 R6 1 1 pas N$6 2 2 pas N$4"
- note removed: "Part Value Device Package Description MFG_PN PACKAGE TOLERANCE C1 1u C-EU_C0805 C0805 CAPACITOR, European symbol C2 100n C-EU_C0805 C0805 CAPACITOR, European symbol C3 C-EU_C0805 C0805 CAPACITOR, European symbol D1 DIODE-SOD80C SOD80C DIODE D2 DIODE-SOD80C SOD80C DIODE P1. MINIPCB_4INCH PCB_5 Q1 BJT_NPNBEC SOT23 TRANSISTOR 2N3904 Q2 BJT_PNPBEC SOT23 TRANSISTOR 2N3906 R1 R-EU_1%_R0805 R0805 RESIST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"
