File: miniPCB/08/A/08A-005/08A-005.brd (EAGLE design)
At the start: 37 parts

Commit message: NM.04NOV2023
Parts:
- removed P1-: (no value), minipcb:MINIPCB_7P_50X50
- added P1: (no value), minipcb:PINS_6
- added PCB1: (no value), minipcb:MINIPCB_0P_50X75
- C10, C7, C8, C9: device minipcb:C050-024X044 -> minipcb:C5MM
- moved R3 58.5 mm to (66.5, 42.5), turned to 180 degrees
- moved R1 53.2 mm to (66.5, 25.5)
- moved R4 53.0 mm to (66.5, 4.50), turned to 180 degrees
- moved C4 47.6 mm to (53.0, 36.5), turned to 270 degrees
- moved C1 41.7 mm to (71.0, 34.0)
- moved TP3 41.6 mm to (58.5, 38.5)
- moved TP6 41.5 mm to (58.5, 34.0)
- moved R2 41.2 mm to (64.0, 36.5)
- moved TP13 37.6 mm to (58.5, 29.0), turned to 0 degrees
- moved TP4 35.9 mm to (58.5, 7.00)
- moved C8 34.0 mm to (45.0, 36.5), turned to 270 degrees
- moved C2 33.8 mm to (71.0, 12.0), turned to 90 degrees
- moved C9 31.0 mm to (44.0, 9.50), turned to 270 degrees
- moved C5 25.2 mm to (52.0, 9.50), turned to 270 degrees
- moved R5 23.8 mm to (64.0, 14.5), turned to 270 degrees
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Connections:
- net BIASA: now also C8.+; no longer C8.1
- net BIASB: now also C9.+; no longer C9.1
- net GND: now also C10.-, C7.-, C8.-, C9.-, P1.1; no longer C10.2, C7.2, C8.2, C9.2, P1-.1
- net IN: now also P1.4; no longer P1-.4
- net IN-: now also C10.+; no longer C10.1
- net OUTA: now also P1.5; no longer P1-.5
- net OUTB: now also P1.6; no longer P1-.7
- net V+: now also C7.+, P1.2; no longer C7.1, P1-.2
Routing:
- net V+: track 71.1 -> 0.00 mm
- net OUTA: track 54.2 -> 0.00 mm
- net OUTB: track 43.7 -> 0.00 mm
- net IN-: track 38.2 -> 0.00 mm
- net BIASB: track 35.9 -> 0.00 mm
- net R2.3: track 33.0 -> 0.00 mm, vias 1 -> 0
- net R5.3: track 24.1 -> 0.00 mm
- net BIASA: track 22.3 -> 0.00 mm
- net INA+: track 18.4 -> 0.00 mm
- net R2.1: track 16.6 -> 0.00 mm
- net R5.1: track 16.4 -> 0.00 mm
- net INB+: track 16.0 -> 0.00 mm
- net IN: track 9.72 -> 0.00 mm
Other:
- board text removed: "C1"
- board text removed: "C10"
- board text removed: "C2"
- board text removed: "C3"
- board text removed: "C4"
- board text removed: "C5"
- board text removed: "C6"
- board text removed: "C7"
- board text removed: "C8"
- board text removed: "C9"
- board text removed: "R1"
- board text removed: "R10"
- board text removed: "R11"
- board text removed: "R2"
- board text removed: "R3"
- board text removed: "R4"
- board text removed: "R5"
- board text removed: "R6"
- board text removed: "R7"
- board text removed: "R8"
- board text removed: "R9"
- board text removed: "TP1"
- board text removed: "TP10"
- board text removed: "TP11"
- board text removed: "TP12"
- board text removed: "TP13"
- board text removed: "TP14"
- board text removed: "TP2"
- board text removed: "TP3"
- board text removed: "TP4"
- board text removed: "TP5"
- board text removed: "TP6"
- board text removed: "TP7"
- board text removed: "TP8"
- board text removed: "TP9"
- board text removed: "U1"
