File: miniPCB/08/A/08A-005/08A-005.sch (EAGLE design)
At the start: 37 parts

Commit message: NM.04NOV2023
Parts:
- removed P1-: (no value), minipcb:MINIPCB_7P50
- added P1: (no value), minipcb:MINIPCB_6P
- added PCB1: (no value), minipcb:MINIPCB_0P50X75
- C10, C7, C8, C9: device minipcb:CAPACITORTHD -> minipcb:CAPACITOR_10
Connections:
- net GND: now also P1-1.1, U1-PWR.V-; no longer P1-1.1, U1P.V-
- net IN: now also P1-4.1; no longer P1-4.1
- net OUTA: now also P1-5.1; no longer P1-5.1
- net OUTB: now also P1-6.1; no longer P1-7.1
- net V+: now also P1-2.1, U1-PWR.V+; no longer P1-2.1, U1P.V+
Other:
- note added: "NOTES:"
- moved on the sheet: C1, C10, C2, C3, C4, C5, C6, C7, C8, C9, R1, R10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
