File: miniPCB/04/A/04A-020/04A-020.sch (EAGLE design)
At the start: 41 parts, among them U1 OPAMP_QUADTHD

Commit message: NM.14JAN2023
Parts:
- P1-: PART_NUMBER X04A-020-A -> X04A-020-A-XB
Connections:
- net GND: now also U1-PWR.V-; no longer U1P.V-
- net V+: now also U1-PWR.V+; no longer U1P.V+

Commit message: NM.07MAR2024
Parts:
- removed P1-: (no value), minipcb:MINIPCB_7P50X100
- added P1: (no value), minipcb:MINIPCB_7P
- added R15, R16, R18: (no value), minipcb:RESISTOR10MM
- added R17: (no value), minipcb:TRIMPOT0.100THD
- added U2: CLASSIC-50X100, miniPCB_BOARDS:CLASSIC-50X100
- C2, C4, C7: device minipcb:CAPACITORTHD -> minipcb:CAPACITOR_10
- R1, R4: device minipcb:TRIMPOT0.100THD -> minipcb:RESISTOR10MM
- R3, R7: device minipcb:RESISTOR10MM -> minipcb:TRIMPOT0.100THD
Connections:
- new net N$12: R13.1, R17.S
- new net N$13: P1-4.1, R1.2
- new net N$14: P1-5.1, R2.2
- net BIAS: now also C5.+, R7.S; no longer C2.+, R4.S
- net GND: now also P1-1.1, R8.1, TP11.1; no longer P1-1.1, R5.1, TP14.1
- net N$1: now also R12.1, R15.1, TP13.1; no longer R10.1, R11.1, TP11.1
- net N$10: now also R3.A, R4.2; no longer R1.A, R2.2
- net N$11: now also P1-6.1, R18.1; no longer P1-5.1, R14.1
- net N$2: now also P1-7.1, R15.2, R16.2; no longer P1-7.1, R11.2, R13.2
- net N$3: now also R2.1; no longer P1-4.1
- net N$4: now also R1.1; no longer P1-6.1
- net N$5: now also R3.S, R5.1, R9.2; no longer R1.S, R6.1, R7.2
- net N$6: now also R10.2, R4.1, R5.2; no longer R2.1, R6.2, R8.2
- net N$7: now also R11.2, R9.1; no longer R7.1, R9.2
- net N$8: now also R10.1, R12.2; no longer R10.2, R8.1
- net N$9: now also R16.1, TP14.1; no longer R13.1, TP12.1
- net NC: now also P1-3.1; no longer P1-3.1
- net OUT: now also R14.1, R17.A, R18.2; no longer R12.1, R14.2
- net POT.1: now also R7.A, R8.2; no longer R4.A, R5.2
- net POT.3: now also R6.1, R7.E; no longer R3.1, R4.E
- net V+: now also C2.+, P1-2.1, R6.2, TP10.1; no longer C5.+, P1-2.1, R3.2, TP13.1
- net VFB: now also R11.1, R13.2, R14.2, TP12.1; no longer R12.2, R9.1, TP10.1
Other:
- moved on the sheet: C1, C2, C3, C4, C5, C6, C7, C8, R10, R11, R12, R13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
