File: miniPCB/04/B/04B-355/04B-355.brd (EAGLE design)
At the start: 45 parts

Commit message: NM.26NOV2024
Parts:
- moved R19 228.8 mm to (-19.1, 92.7)
- moved R18 207.4 mm to (-82.5, 86.4)
- moved R17 201.8 mm to (-69.8, 86.4)
- moved TP9 186.0 mm to (-80.0, 91.4)
- moved C12 185.5 mm to (-48.3, 73.7)
- moved R15 183.2 mm to (-57.1, 86.4)
- moved C11 180.9 mm to (-38.1, 73.7)
- moved R10 169.5 mm to (-69.8, 80.0)
- moved C9 162.4 mm to (-27.9, 73.7)
- moved R5 158.0 mm to (-19.1, 80.0)
- moved TP8 155.4 mm to (-73.7, 91.4)
- moved R16 151.9 mm to (-53.3, 66.0)
- moved C10 143.2 mm to (-19.1, 57.1)
- moved C5 138.6 mm to (-83.8, 66.0), turned to 0 degrees
- moved C7 137.1 mm to (-17.8, 73.7)
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Other:
- board outline added: 160 x 100 mm
