File: miniPCB/05/A/05A-010/05A-010.brd (EAGLE design)
At the start: 6 parts

Commit message: NM.26OCT2023
Connections:
- net N$1 renamed INPUT
- net N$3 renamed OUTPUT
Changed lines of the file:
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@@
 <element name="PCB1" library="minipcb" package="MINIPCB_00A_20X33" value="" x="0" y="0" smashed="yes">
 <attribute name="CIRCUIT_CATEGORY" value="CIRCUIT CATEGORY" x="45.72" y="-1.27" size="1.778" layer="27" display="off"/>
+<attribute name="PART_NUMBER" value="" x="27" y="2" size="1.5" layer="22" font="vector" ratio="13" rot="MR180" align="center-right"/>
 <attribute name="PART_NUMBER" value="" x="27" y="2" size="1.5" layer="16" font="vector" ratio="13" rot="MR180" align="center-right"/>
-<attribute name="PART_NUMBER" value="" x="27" y="2" size="1.5" layer="22" font="vector" ratio="13" rot="MR180" align="center-right"/>
 <attribute name="REVISION" value="A1" x="45.72" y="-1.27" size="1.778" layer="27" display="off"/>
 <attribute name="TITLE" value="TITLE" x="45.72" y="-1.27" size="1.778" layer="27" display="off"/>
@@
 <wire x1="7.67" y1="12.83" x2="7.67" y2="17.98" width="0.5" layer="16"/>
 </signal>
-<signal name="N$1">
+<signal name="INPUT">
 <contactref element="P1" pad="4"/>
 <contactref element="R1" pad="1"/>
@@
 <wire x1="17" y1="3.5" x2="19.5" y2="6" width="0.5" layer="16"/>
 </signal>
-<signal name="N$3">
+<signal name="OUTPUT">
 <contactref element="R2" pad="2"/>
 <contactref element="C2" pad="1"/>

Commit message: Attempting to fix my Git merge error.
Connections:
- net INPUT renamed N$1
- net OUTPUT renamed N$3
Changed lines of the file:
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@@
 <element name="PCB1" library="minipcb" package="MINIPCB_00A_20X33" value="" x="0" y="0" smashed="yes">
 <attribute name="CIRCUIT_CATEGORY" value="CIRCUIT CATEGORY" x="45.72" y="-1.27" size="1.778" layer="27" display="off"/>
+<attribute name="PART_NUMBER" value="" x="27" y="2" size="1.5" layer="16" font="vector" ratio="13" rot="MR180" align="center-right"/>
 <attribute name="PART_NUMBER" value="" x="27" y="2" size="1.5" layer="22" font="vector" ratio="13" rot="MR180" align="center-right"/>
-<attribute name="PART_NUMBER" value="" x="27" y="2" size="1.5" layer="16" font="vector" ratio="13" rot="MR180" align="center-right"/>
 <attribute name="REVISION" value="A1" x="45.72" y="-1.27" size="1.778" layer="27" display="off"/>
 <attribute name="TITLE" value="TITLE" x="45.72" y="-1.27" size="1.778" layer="27" display="off"/>
@@
 <wire x1="7.67" y1="12.83" x2="7.67" y2="17.98" width="0.5" layer="16"/>
 </signal>
-<signal name="INPUT">
+<signal name="N$1">
 <contactref element="P1" pad="4"/>
 <contactref element="R1" pad="1"/>
@@
 <wire x1="17" y1="3.5" x2="19.5" y2="6" width="0.5" layer="16"/>
 </signal>
-<signal name="OUTPUT">
+<signal name="N$3">
 <contactref element="R2" pad="2"/>
 <contactref element="C2" pad="1"/>
