File: miniPCB/08/C/08C-005/08C-005.sch (EAGLE design)
At the start: 32 parts

Commit message: Attempting to fix my Git merge error.
Parts:
- removed P1: (no value), minipcb:MINIPCB_7P
- removed PCB1: (no value), minipcb:MINIPCB_0P50X50
- added P1-: (no value), minipcb:MINIPCB_7P50
Connections:
- net GND: now also P1-1.1, P1-6.1, U1P.V-; no longer P1-1.1, P1-5.1, U1-PWR.V-
- net N$2: now also P1-4.1; no longer P1-4.1
- net OUT+: now also P1-7.1; no longer P1-7.1
- net OUT-: now also P1-5.1; no longer P1-6.1
- net V+: now also P1-2.1, U1P.V+; no longer P1-2.1, U1-PWR.V+
Other:
- note removed: "NOTES:"
- moved on the sheet: C1, C10, C2, C3, C4, C5, C6, C7, C8, C9, Q1, R1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

Commit message: Attempting to fix my Git merge error.
Parts:
- removed P1-: (no value), minipcb:MINIPCB_7P50
- added P1: (no value), minipcb:MINIPCB_7P
- added PCB1: (no value), minipcb:MINIPCB_0P50X50
Connections:
- net GND: now also P1-1.1, P1-5.1, U1-PWR.V-; no longer P1-1.1, P1-6.1, U1P.V-
- net N$2: now also P1-4.1; no longer P1-4.1
- net OUT+: now also P1-7.1; no longer P1-7.1
- net OUT-: now also P1-6.1; no longer P1-5.1
- net V+: now also P1-2.1, U1-PWR.V+; no longer P1-2.1, U1P.V+
Other:
- note added: "NOTES:"
- moved on the sheet: C1, C10, C2, C3, C4, C5, C6, C7, C8, C9, Q1, R1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
