File: miniPCB/11/A/11A-001/11A-001.brd (EAGLE design)
At the start: 100 x 100 mm, 74 parts, among them J1 VDD SELECTOR, J3 ICSP, J4 PICKIT3, J7 2.1 MM, U1 VIVA_UTSA-KEYPADV5, U2 VIVA_USB-TTL, U3 PIC16F1829, U4 VIVA-HEADER-I2C-RA, U5 VIVA_PIC16BOARD, U6 ATMEGA328-AU, U7 VIVA_USB-TTL, U8 3.3V, U9 5.0V

Commit message: NM.09AUG2023
Parts:
- removed R17: 10k, utsa:R0805
- added C22, C23: (no value), utsa:C0805
- added D7: (no value), utsa:DO214AC
- added J6: (no value), utsa:VIVA-HEADER-ADC-8P
- C11: value 100p -> 100n
- C12: value 1u -> 100p
- C13: value 10u -> 100n
- C14: value (none) -> 1u
- C15: value (none) -> 100n
- C18, C19: value 100n -> (none)
- C5: value 1u -> (none)
- C6: value 32 -> 100n
- C9: value 1u -> 10u
- J1: value VDD SELECTOR -> PICKIT3; device utsa:PINS_3 -> nolan-viva:PICKIT3
- J2: device utsa:VIVA-HEADER-12P -> utsa:VIVA-HEADER-ADC-PIC16
- J4: value PICKIT3 -> (none); device nolan-viva:PICKIT3 -> utsa:VIVA-HEADER-ADC-8P
- J5: device utsa:VIVA-HEADER-ADC-PIC16 -> utsa:VIVA-HEADER-ADC-8P
- J8: value (none) -> VDD SELECTOR; device utsa:VIVA-HEADER-ADC-8P -> utsa:PINS_3
- R1, R2, R3: value 150 -> 180
- R11: value 10R -> 10k
- R12, R16: value 10k -> 180
- R14: value 180 -> 10k
- R15: value 1k -> 10R
- R5: value 2k2 -> 10k
- R7: value 10k -> 2k2
- R8, R9: value 10k -> 4k7
- U6: value ATMEGA328-AU -> ATMEGA328P-AU
- moved J2 97.7 mm to (96.5, 21.5), turned to 270 degrees
- moved J4 89.7 mm to (58.4, 91.5)
- moved J8 88.0 mm to (5.00, 39.5)
- moved R7 86.5 mm to (90.5, 72.5), turned to 270 degrees
- moved C5 81.9 mm to (86.5, 72.5), turned to 270 degrees
- moved J1 79.4 mm to (76.0, 3.50)
- moved J5 62.3 mm to (96.5, 83.8), turned to 180 degrees
- moved D3 58.6 mm to (17.0, 36.0), turned to 0 degrees
- moved R12 56.3 mm to (69.5, 61.5), turned to 0 degrees
- moved R15 56.2 mm to (60.5, 79.5)
- moved R9 56.0 mm to (26.5, 22.0)
- moved C6 53.5 mm to (15.5, 12.0), turned to 270 degrees
- moved C20 53.0 mm to (29.5, 91.5), turned to 0 degrees
- moved D6 50.2 mm to (17.0, 38.5)
- moved D4 45.9 mm to (13.0, 94.5), turned to 0 degrees
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- renumbered REV-A1 to -, U$3 to $3_73_$
Connections:
- removed net AT_RST_BTN: B3.3.B, B3.4.B, R13.1, R9.2
- removed net N$36: C14.1, C17.1, D1.C, D3.C, U8.3, U9.3
- removed net N$38: LED3.A, R15.2
- removed net N$45: C18.1, U7.2.DTR
- removed net N$46: C15.1, D2.A, U8.2, U8.4.TAB
- removed net N$47: D3.A, J7.TIP
- removed net N$48: D4.A, U7.1.3V3
- removed net N$49: C16.1, D6.A, U9.2, U9.4.TAB
- removed net N$51: D5.A, U2.1.3V3
- new net 3V3: C22.1, D4.A, U8.2, U8.4.TAB
- new net 5V0: C23.1, D7.A, U9.2, U9.4.TAB
- new net AT-USB-3V3: D2.A, U7.1.3V3
- new net AT-USB-5V: D5.A, U7.6.5V
- new net AT_DTR_CAP: C15.1, U7.2.DTR
- new net LED_POWER: LED3.A, R16.2
- new net N$33: J5.11, J5.6
- new net N$34: J5.10, J5.7
- new net N$35: J5.8, J5.9
- new net PIC-USB-3V3: D3.A, U2.1.3V3
- new net PIC-USB-5V: D6.A, U2.6.5V
- new net UNREG_IN: D1.A, J7.TIP
- new net UNREG_IN_POLARITY_PROTECTED: C18.1, C19.1, C20.1, C21.1, D1.C, U8.3, U9.3
- net +3V3: now also D3.C, J8.1; no longer D5.C, J1.1
- net +5V: now also D5.C, D7.C, J8.3; no longer D1.A, J1.3, U2.6.5V, U7.6.5V
- net ADC6: now also J6.8, J6.9; no longer J8.7
- net ADC7: now also J6.10, J6.7; no longer J8.8
- net AT_RST: now also C15.2; no longer C18.2
- net AT_RST_CAP: now also B4.3.B, B4.4.B, C13.1, R13.1, R14.2; no longer C9.1, R10.2, R9.1
- net AT_SCK: now also R12.1; no longer R14.1
- net AVCC: now also C12.1, C14.1, R15.2; no longer C10.1, C11.1, R11.2
- net B1-CAP: now also R5.2; no longer R12.2
- net GND: now also C18.2, C22.2, C23.2, J1.3, J4.1, J4.16, J5.16, J6.1, J6.16; no longer C15.2, J4.3, J8.1
- net ICSP_CLK: now also J1.5; no longer J4.5
- net ICSP_DAT: now also J1.4; no longer J4.4
- net MCLR: now also J1.1, R8.2; no longer J4.1, R7.2
- net MCLR_CAP: now also C6.1, R8.1, R9.2; no longer C5.1, R7.1, R8.2
- net N$37: now also R12.2; no longer R14.2
- net PB0: now also J5.14, J5.3; no longer J2.9
- net PB1: now also J5.13, J5.4; no longer J2.10
- net PB2: now also J5.12, J5.5; no longer J2.11
- net PC0: now also J6.11, J6.6; no longer J8.3
- net PC1: now also J6.12, J6.5; no longer J8.4
- net PC2: now also J6.13, J6.4; no longer J8.6
- net PC3: now also J6.14, J6.3; no longer J8.5
- net PD2: now also J4.14, J4.3; no longer J2.3
- net PD3: now also J4.13, J4.4; no longer J2.4
- net PD4: now also J4.12, J4.5, R10.1; no longer J2.6, R17.1
- net PD4-CAP: now also B3.3.B, B3.4.B, C11.1, R10.2, R11.2; no longer B4.3.B, B4.4.B, C19.1, R16.2, R17.2
- net PD5: now also J4.11, J4.6; no longer J2.5
- net PD6: now also J4.10, J4.7; no longer J2.7
- net PD7: now also J4.8, J4.9; no longer J2.8
- net RB5: now also J2.5; no longer J5.5
- net RB7: now also R4.1; no longer R12.1
- net RC2: now also J2.3; no longer J5.3
- net RC3: now also J2.4; no longer J5.4
- net SCL: now also R7.2; no longer R6.2
- net SDA: now also R6.2; no longer R5.2
- net VDD: now also C10.1, C16.1, C17.1, C5.1, C9.1, J4.15, J5.15, J6.15, J6.2, R14.1, R7.1, R9.1; no longer C12.1, C13.1, C20.1, C21.1, C6.1, R10.1, R4.1, R8.1
Routing:
- net VDD: track 177.4 -> 462.8 mm, vias 20 -> 24
- net SCL: track 0.00 -> 183.3 mm, vias 0 -> 6
- net SDA: track 0.00 -> 171.1 mm, vias 0 -> 6
- net RC3: track 0.00 -> 90.0 mm, vias 0 -> 2
- net ICSP_DAT: track 0.00 -> 61.8 mm, vias 0 -> 2
- net ICSP_CLK: track 0.00 -> 60.1 mm, vias 0 -> 2
- net N$46: track 56.1 -> 0.00 mm, vias 2 -> 0
- net RA4: track 0.00 -> 52.1 mm
- net PD4: track 0.00 -> 50.5 mm, vias 0 -> 2
- net RB5: track 0.00 -> 48.4 mm
- net PD5: track 0.00 -> 48.3 mm, vias 0 -> 1
- net AT_RST: track 2.00 -> 49.8 mm, vias 0 -> 1
- net RC2: track 0.00 -> 47.4 mm
- net PB0: track 0.00 -> 46.0 mm
- net RC0: track 0.00 -> 46.0 mm
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Other:
- board text added: "ATmega328P-AU"
- board text added: "C1"
- board text added: "C10"
- board text added: "C11"
- board text added: "C12"
- board text added: "C13"
- board text added: "C14"
- board text added: "C15"
- board text added: "C16"
- board text added: "C17"
- board text added: "C18"
- board text added: "C19"
- board text added: "C2"
- board text added: "C20"
- board text added: "C21"
- board text added: "C22"
- board text added: "C23"
- board text added: "C3"
- board text added: "C4"
- board text added: "C5"
- board text added: "C6"
- board text added: "C7"
- board text added: "C8"
- board text added: "C9"
- board text added: "D1"
- board text added: "D2"
- board text added: "D3"
- board text added: "D4"
- board text added: "D5"
- board text added: "D6"
- board text added: "D7"
- board text added: "J3"
- board text added: "J7"
- board text added: "J8"
- board text added: "LED1"
- board text added: "LED2"
- board text added: "LED3"
- board text added: "R1"
- board text added: "R10"
- board text added: "R11"
- board text added: "R12"
- board text added: "R13"
- board text added: "R14"
- board text added: "R15"
- board text added: "R16"
- board text added: "R2"
- board text added: "R3"
- board text added: "R4"
- board text added: "R5"
- board text added: "R6"
- board text added: "R7"
- board text added: "R8"
- board text added: "R9"
- board text added: "REV A1"
- board text added: "U3"
- board text added: "U6"
- board text added: "U8"
- board text added: "U9"
- board text added: "Y1"
- board text removed: "ATmega328"

Commit message: NM.07MAR2024
Parts:
- added C24: 1u, utsa:C0805
Connections:
- new net AREF: C24.1, U6.20
- net GND: now also C24.2; no longer U6.20
Routing:
- net GND: track 16.4 -> 10.0 mm, vias 119 -> 123
- net AREF: track 0.00 -> 2.34 mm
Other:
- board text added: "C24"
- board text added: "REV A2"
- board text removed: "REV A1"

Commit message: Attempting to fix my Git merge error.
Parts:
- added DRILEGEND: (no value), drilegend:DRILEGEND
- moved D4 1.50 mm to (13.0, 96.0)
- moved D1 1.00 mm to (13.0, 92.5)
- moved D7 0.50 mm to (13.0, 89.0)
Routing:
- net +3V3: track 85.7 -> 87.2 mm
- net 3V3: track 18.3 -> 19.5 mm
- net UNREG_IN_POLARITY_PROTECTED: track 33.9 -> 34.5 mm
- net 5V0: track 18.5 -> 19.0 mm
- net GND: vias 123 -> 209

Commit message: NM.21APR2024
Parts:
- removed DRILEGEND: (no value), drilegend:DRILEGEND
Changed lines of the file:
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@@
 <layer number="21" name="tPlace" color="7" fill="1" visible="yes" active="yes"/>
 <layer number="22" name="bPlace" color="7" fill="1" visible="yes" active="yes"/>
-<layer number="23" name="tOrigins" color="15" fill="1" visible="no" active="yes"/>
+<layer number="23" name="tOrigins" color="15" fill="1" visible="yes" active="yes"/>
 <layer number="24" name="bOrigins" color="15" fill="1" visible="yes" active="yes"/>
 <layer number="25" name="tNames" color="7" fill="1" visible="yes" active="yes"/>
@@
 <layer number="42" name="bRestrict" color="1" fill="10" visible="yes" active="yes"/>
 <layer number="43" name="vRestrict" color="2" fill="10" visible="yes" active="yes"/>
-<layer number="44" name="Drills" color="7" fill="1" visible="no" active="yes"/>
-<layer number="45" name="Holes" color="7" fill="1" visible="no" active="yes"/>
+<layer number="44" name="Drills" color="7" fill="1" visible="yes" active="yes"/>
+<layer number="45" name="Holes" color="7" fill="1" visible="yes" active="yes"/>
 <layer number="46" name="Milling" color="3" fill="1" visible="yes" active="yes"/>
 <layer number="47" name="Measures" color="7" fill="1" visible="yes" active="yes"/>
@@
 <attribute name="VALUE" x="54.3" y="79.5" size="1.27" layer="27" ratio="12" rot="R90" align="center"/>
 </element>
-<element name="DRILEGEND" library="drilegend" package="DRILEGEND" value="" x="-27.016" y="-31.825996875" smashed="yes"/>
 </elements>
 <signals>

Commit message: NM.22APR2024
Routing:
- net AT_DTR_CAP: track 34.6 -> 31.7 mm
- net N$16: track 0.00 -> 1.91 mm
- net XTAL1: track 9.51 -> 7.81 mm
- net AT-USB-3V3: vias 1 -> 0
Changed lines of the file:
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@@
 <setting verticaltext="up"/>
 </settings>
-<grid distance="0.5" unitdist="mm" unit="mm" style="dots" multiple="1" display="yes" altdistance="0.025" altunitdist="inch" altunit="inch"/>
+<grid distance="1" unitdist="mm" unit="mm" style="dots" multiple="1" display="yes" altdistance="0.025" altunitdist="inch" altunit="inch"/>
 <layers>
 <layer number="1" name="Top" color="4" fill="1" visible="yes" active="yes"/>
@@
 <wire x1="22" y1="90.008" x2="22" y2="88.992" width="0.1016" layer="145"/>
 <wire x1="21.492" y1="89.5" x2="22.508" y2="89.5" width="0.1016" layer="145"/>
-<wire x1="15" y1="65.008" x2="15" y2="63.992" width="0.1016" layer="145"/>
-<wire x1="14.492" y1="64.5" x2="15.508" y2="64.5" width="0.1016" layer="145"/>
 <wire x1="62.980759375" y1="74.488759375" x2="62.980759375" y2="73.472759375" width="0.1016" layer="145"/>
 <wire x1="62.472759375" y1="73.980759375" x2="63.488759375" y2="73.980759375" width="0.1016" layer="145"/>
@@
 </element>
 <element name="J5" library="utsa" package="VIVA-HEADER-ADC-8P" value="" x="96.52" y="83.82" smashed="yes" rot="R180">
-<attribute name="P3" value="PB0/D7" x="92.075" y="85.59" size="1.27" layer="21" font="vector" ratio="15" rot="R90"/>
+<attribute name="P3" value="PB0/D8" x="92.075" y="85.59" size="1.27" layer="21" font="vector" ratio="15" rot="R90"/>
 <attribute name="P4" value="PB1/D9" x="89.535" y="85.59" size="1.27" layer="21" font="vector" ratio="15" rot="R90"/>
 <attribute name="P5" value="PB2/D10" x="86.995" y="85.59" size="1.27" layer="21" font="vector" ratio="15" rot="R90"/>
@@
 <contactref element="C15" pad="2"/>
 <contactref element="J3" pad="5"/>
-<wire x1="43.95" y1="73.5" x2="43.95" y2="75.5" width="0.5" layer="1"/>
+<wire x1="43.95" y1="73.5" x2="43.95" y2="75.5" width="0.3" layer="1"/>
 <wire x1="43.95" y1="72.4" x2="43.95" y2="73.5" width="0.3" layer="1"/>
 <wire x1="71.12" y1="71.46" x2="69.16" y2="69.5" width="0.3" layer="16"/>
@@
 <contactref element="Y1" pad="3"/>
 <contactref element="U6" pad="7"/>
-<wire x1="57.3" y1="63.1" x2="58" y2="63.1" width="0.3" layer="1"/>
-<wire x1="58" y1="63.1" x2="58.5" y2="63.6" width="0.3" layer="1"/>
-<wire x1="58.5" y1="63.6" x2="58.5" y2="65.3" width="0.3" layer="1"/>
-<wire x1="58.5" y1="65.3" x2="57.9" y2="65.9" width="0.3" layer="1"/>
-<wire x1="57.9" y1="65.9" x2="56.7" y2="65.9" width="0.3" layer="1"/>
-<wire x1="56.7" y1="65.9" x2="56" y2="66.6" width="0.3" layer="1"/>
+<wire x1="57.3" y1="63.1" x2="56.6" y2="63.1" width="0.3" layer="1"/>
+<wire x1="56.6" y1="63.1" x2="56.2" y2="63.5" width="0.3" layer="1"/>
+<wire x1="56.2" y1="66.4" x2="56.2" y2="63.5" width="0.3" layer="1"/>
+<wire x1="56.2" y1="66.4" x2="56" y2="66.6" width="0.3" layer="1"/>
 <wire x1="56" y1="66.6" x2="56" y2="67.75" width="0.3" layer="1"/>
 <wire x1="58.3" y1="61.3" x2="57.3" y2="62.3" width="0.25" layer="1"/>
@@
 <contactref element="Y1" pad="1"/>
 <contactref element="U6" pad="8"/>
-<wire x1="57.1" y1="66.5" x2="58.3" y2="66.5" width="0.3" layer="1"/>
-<wire x1="58.3" y1="66.5" x2="59.2" y2="65.6" width="0.3" layer="1"/>
-<wire x1="59.2" y1="65.6" x2="59.2" y2="65.2" width="0.3" layer="1"/>
-<wire x1="59.2" y1="65.2" x2="59.45" y2="64.95" width="0.3" layer="1"/>
-<wire x1="59.45" y1="64.95" x2="59.7" y2="64.7" width="0.3" layer="1"/>
+<wire x1="57.1" y1="66.5" x2="58.6" y2="66.5" width="0.3" layer="1"/>
+<wire x1="58.6" y1="66.5" x2="59.7" y2="65.4" width="0.3" layer="1"/>
+<wire x1="59.6" y1="64.8" x2="59.7" y2="64.9" width="0.3" layer="1"/>
+<wire x1="59.7" y1="65.4" x2="59.7" y2="64.9" width="0.3" layer="1"/>
+<wire x1="59.45" y1="64.95" x2="59.6" y2="64.8" width="0.3" layer="1"/>
+<wire x1="59.6" y1="64.8" x2="59.7" y2="64.7" width="0.3" layer="1"/>
 <wire x1="57.1" y1="66.5" x2="56.8" y2="66.8" width="0.3" layer="1"/>
 <wire x1="56.8" y1="66.8" x2="56.8" y2="67.75" width="0.3" layer="1"/>
@@
 <contactref element="R14" pad="2"/>
 <wire x1="42.05" y1="79.5" x2="41.000003125" y2="79.500003125" width="0.5" layer="1"/>
-<wire x1="42.05" y1="79.5" x2="42.05" y2="75.5" width="0.5" layer="1"/>
-<wire x1="42.05" y1="79.5" x2="42.05" y2="77.5" width="0.5" layer="1"/>
+<wire x1="42.05" y1="79.5" x2="42.05" y2="75.5" width="0.3" layer="1"/>
+<wire x1="42.05" y1="79.5" x2="42.05" y2="77.5" width="0.3" layer="1"/>
 <wire x1="41.000003125" y1="79.500003125" x2="39.499996875" y2="79.500003125" width="0.5" layer="1"/>
 <wire x1="39.499996875" y1="79.500003125" x2="37" y2="82" width="0.5" layer="1"/>
@@
 <contactref element="U7" pad="2.DTR"/>
 <contactref element="C15" pad="1"/>
-<wire x1="19" y1="61.96" x2="17.54" y2="61.96" width="0.5" layer="1"/>
-<wire x1="17.54" y1="61.96" x2="16.5" y2="63" width="0.5" layer="1"/>
-<wire x1="16.5" y1="63" x2="16.5" y2="66" width="0.5" layer="1"/>
-<wire x1="16.5" y1="66" x2="17.5" y2="67" width="0.5" layer="1"/>
-<wire x1="17.5" y1="67" x2="18.5" y2="67" width="0.5" layer="1"/>
-<wire x1="18.5" y1="67" x2="25" y2="73.5" width="0.5" layer="1"/>
-<wire x1="25" y1="73.5" x2="42.05" y2="73.5" width="0.5" layer="1"/>
+<wire x1="19" y1="61.96" x2="20.36" y2="61.96" width="0.3" layer="1"/>
+<wire x1="20.36" y1="61.96" x2="20.9" y2="62.5" width="0.3" layer="1"/>
+<wire x1="25.3" y1="73.5" x2="42.05" y2="73.5" width="0.3" layer="1"/>
+<wire x1="20.9" y1="62.5" x2="20.9" y2="69.1" width="0.3" layer="1"/>
+<wire x1="20.9" y1="69.1" x2="25.3" y2="73.5" width="0.3" layer="1"/>
 </signal>
 <signal name="3V3">
@@
 <wire x1="19" y1="45" x2="10" y2="54" width="0.5" layer="1"/>
 <wire x1="10" y1="63.5" x2="11" y2="64.5" width="0.5" layer="1"/>
-<wire x1="11" y1="64.5" x2="15" y2="64.5" width="0.5" layer="1"/>
-<via x="15" y="64.5" extent="1-16" drill="0.5" diameter="0.9"/>
-<wire x1="15" y1="64.5" x2="19" y2="64.5" width="0.5" layer="16"/>
+<wire x1="11" y1="64.5" x2="19" y2="64.5" width="0.5" layer="1"/>
 <wire x1="10" y1="54" x2="10" y2="63.5" width="0.5" layer="1"/>
 </signal>
@@
 <wire x1="54.3" y1="77.5" x2="54.3" y2="78.55" width="0.3" layer="1"/>
 </signal>
+<signal name="N$16">
+<wire x1="59.2" y1="63.4" x2="59" y2="63.4" width="0.3" layer="1"/>
+<wire x1="59" y1="63.4" x2="58" y2="64.4" width="0.3" layer="1"/>
+<wire x1="58" y1="64.4" x2="57.7" y2="64.4" width="0.3" layer="1"/>
+</signal>
 </signals>
