File: miniPCB/11/A/11A-001/11A-001.sch (EAGLE design)
At the start: 73 parts, among them J1 VDD SELECTOR, J3 ICSP, J4 PICKIT3, J7 2.1 MM, U1 VIVA_UTSA-KEYPADV5, U2 VIVA_USB-TTL, U3 PIC16F1829, U4 VIVA-HEADER-I2C-RA, U5 VIVA_PIC16BOARD, U6 ATMEGA328-AU, U7 VIVA_USB-TTL, U8 3.3V, U9 5.0V

Commit message: NM.09AUG2023
Parts:
- removed R17: 10k, utsa:R-EU__R0805
- removed REV-A1: 11A-001, utsa:PCB_100X100
- added -: 11A-001, utsa:PCB_100X100
- added C22, C23: (no value), utsa:C0805
- added D7: (no value), utsa:DIODE-DO214AC
- added J6: (no value), utsa:VIVA-HEADER-ADC-8P
- C10: device utsa:C-EU_C0805 -> utsa:C0805
- C11: value 100p -> 100n; device utsa:C-EU_C0805 -> utsa:C0805
- C12: value 1u -> 100p; device utsa:C0805 -> utsa:C-EU_C0805
- C13: value 10u -> 100n
- C14: value (none) -> 1u; device utsa:C0805 -> utsa:C-EU_C0805
- C15: value (none) -> 100n
- C18, C19: value 100n -> (none)
- C5: value 1u -> (none)
- C6: value 32 -> 100n
- C9: value 1u -> 10u
- J1: value VDD SELECTOR -> PICKIT3; device utsa:PINS_3_2.54 -> nolan-viva:PICKIT3
- J2: device utsa:VIVA-HEADER-12P -> utsa:VIVA-HEADER-ADC-PIC16; P10 PB1/D9 -> (none); P11 PB2/D10 -> (none); P12 NC -> (none); P3 PD2/D2 -> (none); P4 PD3/D3 -> (none); P5 PD4/D4 -> (none); P6 PD5/D5 -> (none); P7 PD6/D6 -> (none); P8 PD7/D7 -> (none); P9 PB0/D8 -> (none)
- J4: value PICKIT3 -> (none); device nolan-viva:PICKIT3 -> utsa:VIVA-HEADER-ADC-8P; P3 (none) -> PD2/D2; P4 (none) -> PD3/D3; P5 (none) -> PD4/D4; P6 (none) -> PD5/D5; P7 (none) -> PD6/D6; P8 (none) -> PD7/D7
- J5: device utsa:VIVA-HEADER-ADC-PIC16 -> utsa:VIVA-HEADER-ADC-8P; P3 (none) -> PB0/D7; P4 (none) -> PB1/D9; P5 (none) -> PB2/D10; P6 (none) -> A; P7 (none) -> B; P8 (none) -> C
- J8: value (none) -> VDD SELECTOR; device utsa:VIVA-HEADER-ADC-8P -> utsa:PINS_3_2.54; P3 PC0/A0 -> (none); P4 PC1/A1 -> (none); P5 PC2/A2 -> (none); P6 PC3/A3 -> (none); P7 ADC6/A6 -> (none); P8 ADC7/A7 -> (none)
- R1, R2, R3: value 150 -> 180
- R11: value 10R -> 10k
- R12, R16: value 10k -> 180
- R14: value 180 -> 10k
- R15: value 1k -> 10R
- R5: value 2k2 -> 10k
- R7: value 10k -> 2k2
- R8, R9: value 10k -> 4k7
- U6: value ATMEGA328-AU -> ATMEGA328P-AU
- renumbered U$3 to $3_73_$
Connections:
- removed net AT_RST_BTN: B3.2, R13.1, R9.2
- removed net N$36: C14.+, C17.+, D1.C, D3.C, U8.IN, U9.IN
- removed net N$38: LED3.A, R15.2
- removed net N$45: C18.+, U7.(2)DTR
- removed net N$46: C15.+, D2.A, U8.OUT
- removed net N$47: D3.A, J7.TIP
- removed net N$48: D4.A, U7.(1)3V3
- removed net N$49: C16.+, D6.A, U9.OUT
- removed net N$51: D5.A, U2.(1)3V3
- new net 3V3: C22.+, D4.A, U8.OUT
- new net 5V0: C23.+, D7.A, U9.OUT
- new net AT-USB-3V3: D2.A, U7.(1)3V3
- new net AT-USB-5V: D5.A, U7.(6)5V
- new net AT_DTR_CAP: C15.+, U7.(2)DTR
- new net LED_POWER: LED3.A, R16.2
- new net N$33: J5.6.ADC3
- new net N$34: J5.7.ADC4
- new net N$35: J5.8.ADC5
- new net PIC-USB-3V3: D3.A, U2.(1)3V3
- new net PIC-USB-5V: D6.A, U2.(6)5V
- new net UNREG_IN: D1.A, J7.TIP
- new net UNREG_IN_POLARITY_PROTECTED: C18.+, C19.+, C20.+, C21.+, D1.C, U8.IN, U9.IN
- net +3V3: now also D3.C, J8.1; no longer D5.C, J1.1
- net +5V: now also D5.C, D7.C, J8.3; no longer D1.A, J1.3, U2.(6)5V, U7.(6)5V
- net ADC6: now also J6.8.ADC5; no longer J8.5.ADC3
- net ADC7: now also J6.7.ADC4; no longer J8.5.ADC4
- net AT_RST: now also C15.-; no longer C18.-
- net AT_RST_CAP: now also B4.2, C13.+, R13.1, R14.2; no longer C9.+, R10.2, R9.1
- net AT_SCK: now also R12.1; no longer R14.1
- net AVCC: now also C12.1, C14.1, R15.2; no longer C10.1, C11.1, R11.2
- net B1-CAP: now also R5.2; no longer R12.2
- net GND: now also C10.-, C11.-, C12.2, C14.2, C18.-, C22.-, C23.-, J1.3.VSS(GND), J4.1.GND, J6.1.GND; no longer C10.2, C11.2, C12.-, C14.-, C15.-, J4.3.VSS(GND), J8.1.GND
- net ICSP_CLK: now also J1.5.PGC; no longer J4.5.PGC
- net ICSP_DAT: now also J1.4.PGD; no longer J4.4.PGD
- net MCLR: now also J1.1.MCLR, R8.2; no longer J4.1.MCLR, R7.2
- net MCLR_CAP: now also C6.+, R8.1, R9.2; no longer C5.+, R7.1, R8.2
- net N$37: now also R12.2; no longer R14.2
- net PB0: now also J5.3.ADC0; no longer J2.5.ADC5
- net PB1: now also J5.4.ADC1; no longer J2.5.ADC6
- net PB2: now also J5.5.ADC2; no longer J2.5.ADC7
- net PC0: now also J6.6.ADC3; no longer J8.3.ADC0
- net PC1: now also J6.5.ADC2; no longer J8.4.ADC1
- net PC2: now also J6.4.ADC1; no longer J8.5.ADC2
- net PC3: now also J6.3.ADC0; no longer J8.5.ADC1
- net PD2: now also J4.3.ADC0; no longer J2.3.ADC0
- net PD3: now also J4.4.ADC1; no longer J2.4.ADC1
- net PD4: now also J4.5.ADC2, R10.1; no longer J2.5.ADC2, R17.1
- net PD4-CAP: now also B3.2, C11.+, R10.2, R11.2; no longer B4.2, C19.+, R16.2, R17.2
- net PD5: now also J4.6.ADC3; no longer J2.5.ADC1
- net PD6: now also J4.7.ADC4; no longer J2.5.ADC3
- net PD7: now also J4.8.ADC5; no longer J2.5.ADC4
- net RB5: now also J2.5.ADC2; no longer J5.5.ADC2
- net RB7: now also R4.1; no longer R12.1
- net RC2: now also J2.3.ADC0; no longer J5.3.ADC0
- net RC3: now also J2.4.ADC1; no longer J5.4.ADC1
- net SCL: now also R7.2; no longer R6.2
- net SDA: now also R6.2; no longer R5.2
- net VDD: now also C10.+, C16.+, C17.+, C5.+, C9.+, J1.2.VDD(PWR), J4.2.VDD, J6.2.VDD, J8.2, R14.1, R7.1, R9.1; no longer C12.+, C13.+, C20.+, C21.+, C6.+, J1.2, J4.2.VDD(PWR), J8.2.VDD, R10.1, R4.1, R8.1
Other:
- note added: "3.3V LINEAR REGULATOR"
- note added: "5.0V LINEAR REGULATOR"
- note added: "FIDUCIALS"
- note added: "INPUT CAPACITANCE"
- note added: "LOGO"
- note added: "NOTES: THIS PROJECT WAS CREATED IN SUPPORT OF UTSA ENGINEERING CURRICULUM. PROJECT REVISION HISTORY: v1.0, AUG.2014 INITIAL RELEASE v2.0, JAN.2015 ADDED PROTOTYPING AREA v3.0, AUG.2015 ADDED HIGH-SIDE TRANSISTOR SWITCH ADDED ABC CAPACITANCE TOUCH BUTTONS v4.0, AUG.2018 CONVERTED TO SURFACE MOUNT REPLACED ABC WITH UTSA FOR CAPACITANCE TOUCH BUTTONS v5.1, JAN.2022 EXPANDED TO 100 x 100 mm ADDED ATm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"
- note added: "POWER INDICATOR LED"
- note added: "POWER STEERING"
- note added: "VDD SELECTION JUMPER"
- note removed: "Fiducial"
- note removed: "v5.1, JAN.2022 EXPANDED TO 100 x 100 mm ADDED ATmega328P REMOVED HIGH-SIDE TRANSISTOR SWITCH v5.2, MAY.2022 ADDED ATMEGA BUTTON CHANGED OLED DISPLAY ADDED DTR CAPACITOR v5.3, JUNE.2023 UPDATED ATmega328P PIN BREAKOUTS UPDATED FOOTPRINTS AND SILKSCREEN FOR HIGHER DENSITY LAYOUT"
- moved on the sheet: B3, B4, C1, C13, C16, C17, C2, C20, C21, C3, C5, C6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

Commit message: NM.07MAR2024
Parts:
- added C24: 1u, utsa:C-EU_C0805
Connections:
- new net AREF: C24.1, U6.AREF
- net GND: now also C24.2; no longer U6.AREF

Commit message: NM.22APR2024
Parts:
- J5: P3 PB0/D7 -> PB0/D8
Changed lines of the file:
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@@
 </part>
 <part name="J5" library="utsa" deviceset="VIVA-HEADER-ADC-8P" device="">
-<attribute name="P3" value="PB0/D7"/>
+<attribute name="P3" value="PB0/D8"/>
 <attribute name="P4" value="PB1/D9"/>
 <attribute name="P5" value="PB2/D10"/>
