File: miniPCB/14/A/14A-05/14A-05.brd (EAGLE design)
At the start: 3.8 x 86.4 mm, 55 parts, among them J3 ICSP, U2 UCC287502DBVR, U3 TLP181(GB,F), U6 ATMEGA328P-AU, U7 VIVA_USB-TTL

Commit message: NM.26NOV2024
Parts:
- removed B3, B4: (no value), nolan-utsa:6X6MM
- removed C10, C14, C24: 1u, utsa:C0805
- removed C11, C13, C15: 100n, utsa:C0805
- removed C12: 100p, utsa:C0805
- removed C2, C7: 15p, utsa:C0603
- removed C9: 10u, utsa:C0805
- removed J3: ICSP, utsa:PINS_6-2X3_AT
- removed LED2: (no value), utsa:SML0805
- removed Q1: (no value), minipcb:SOT23
- removed R1, R2: (no value), minipcb:R0402
- removed R13, R14, R5, R6: 10k, utsa:R0805
- removed R3: 10R, utsa:R0805
- removed R4: 180, utsa:R0805
- removed U6: ATMEGA328P-AU, utsa:32A_ATM
- removed U7: VIVA_USB-TTL, utsa:VIVA_USB_TTL_SUBTEXT
- removed Y1: (no value), utsa:TXC7M2
Connections:
- removed net ADC6: U6.19
- removed net ADC7: U6.22
- removed net AREF: C24.1, U6.20
- removed net AT-USB-3V3: U7.1.3V3
- removed net AT-USB-5V: U7.6.5V
- removed net AT_DTR_CAP: C15.1, U7.2.DTR
- removed net AT_MISO: J3.1, U6.16
- removed net AT_MOSI: J3.4, U6.15
- removed net AT_RST: C15.2, J3.5, R13.2, U6.29
- removed net AT_RST_CAP: B4.3.B, B4.4.B, C13.1, R13.1, R14.2
- removed net AT_RXD: U6.30, U7.4.RDO
- removed net AT_SCK: J3.3, R4.1, U6.17
- removed net AT_TXD: U6.31, U7.3.RXI
- removed net AVCC: C12.1, C14.1, R3.2, U6.18
- removed net N$1: Q1.1, R1.2, R2.2
- removed net N$37: LED2.A, R4.2
- removed net PB0: U6.12
- removed net PB1: U6.13
- removed net PB2: U6.14
- removed net PC0: U6.23
- removed net PC1: U6.24
- removed net PC2: U6.25
- removed net PC3: U6.26
- removed net PD2: U6.32
- removed net PD3: U6.1
- removed net PD4: R6.1, U6.2
- removed net PD4-CAP: B3.3.B, B3.4.B, C11.1, R5.2, R6.2
- removed net PD5: U6.9
- removed net PD6: U6.10
- removed net PD7: U6.11
- removed net SCL: U6.28
- removed net SDA: U6.27
- removed net XTAL1: C7.2, U6.7, Y1.3
- removed net XTAL2: C2.2, U6.8, Y1.1
- net GND: no longer B3.1.A, B3.2.A, B4.1.A, B4.2.A, C10.2, C11.2, C12.2, C13.2, C14.2, C2.1, C24.2, C7.1, C9.2, J3.6, LED2.C, Q1.2, R2.1, U6.21, U6.3, U6.5, U7.5.GND
- net VDD: no longer C10.1, C9.1, J3.2, R14.1, R3.1, R5.1, U6.4, U6.6
Routing:
- net GND: track 2.40 -> 0.00 mm
