File: miniPCB/14/A/14A-05/14A-05.sch (EAGLE design)
At the start: 55 parts, among them J3 ICSP, U2 UCC287502DBVR, U3 TLP181(GB,F), U6 ATMEGA328P-AU, U7 VIVA_USB-TTL

Commit message: NM.26NOV2024
Parts:
- removed B3, B4: (no value), nolan-utsa:PUSHBUTTON6X6MM
- removed C10: 1u, utsa:C0805
- removed C11, C13, C15: 100n, utsa:C0805
- removed C12: 100p, utsa:C-EU_C0805
- removed C14, C24: 1u, utsa:C-EU_C0805
- removed C2, C7: 15p, utsa:C0603
- removed C9: 10u, utsa:C0805
- removed J3: ICSP, utsa:PINS_6-2X3_AT
- removed LED2: (no value), utsa:LEDSML0805
- removed Q1: (no value), minipcb:MOSFET-NSOT23
- removed R1, R2: (no value), minipcb:RESISTOR0402
- removed R13, R14, R5, R6: 10k, utsa:R-EU__R0805
- removed R3: 10R, utsa:R-EU__R0805
- removed R4: 180, utsa:R-EU__R0805
- removed U6: ATMEGA328P-AU, utsa:ATMEGA328-AU
- removed U7: VIVA_USB-TTL, utsa:VIVA_USB-TTL
- removed Y1: (no value), utsa:CRYSTAL-3225_4P
Connections:
- removed net ADC6: U6.ADC6
- removed net ADC7: U6.ADC7
- removed net AREF: C24.1, U6.AREF
- removed net AT-USB-3V3: U7.(1)3V3
- removed net AT-USB-5V: U7.(6)5V
- removed net AT_DTR_CAP: C15.+, U7.(2)DTR
- removed net AT_MISO: J3.1, U6.PB4
- removed net AT_MOSI: J3.4, U6.PB3
- removed net AT_RST: C15.-, J3.5, R13.2, U6.PC6
- removed net AT_RST_CAP: B4.2, C13.+, R13.1, R14.2
- removed net AT_RXD: U6.PD0, U7.(4)MCU.RX
- removed net AT_SCK: J3.3, R4.1, U6.PB5
- removed net AT_TXD: U6.PD1, U7.(3)MCU.TX
- removed net AVCC: C12.1, C14.1, R3.2, U6.AVCC
- removed net N$1: Q1.G, R1.2, R2.2
- removed net N$37: LED2.A, R4.2
- removed net PB0: U6.PB0
- removed net PB1: U6.PB1
- removed net PB2: U6.PB2
- removed net PC0: U6.PC0
- removed net PC1: U6.PC1
- removed net PC2: U6.PC2
- removed net PC3: U6.PC3
- removed net PD2: U6.PD2
- removed net PD3: U6.PD3
- removed net PD4: R6.1, U6.PD4
- removed net PD4-CAP: B3.2, C11.+, R5.2, R6.2
- removed net PD5: U6.PD5
- removed net PD6: U6.PD6
- removed net PD7: U6.PD7
- removed net SCL: U6.PC5
- removed net SDA: U6.PC4
- removed net XTAL1: C7.+, U6.PB6, Y1.2
- removed net XTAL2: C2.+, U6.PB7, Y1.1
- net GND: no longer B3.1, B4.1, C10.-, C11.-, C12.2, C13.-, C14.2, C2.-, C24.2, C7.-, C9.-, J3.6, LED2.C, Q1.S, R2.1, U6.GND, U6.GND_2, U6.GND_3, U7.(5)GND
- net VDD: no longer C10.+, C9.+, J3.2, R14.1, R3.1, R5.1, U6.VCC, U6.VCC_2
Other:
- note removed: "ATmega MICROCONTROLLER"
- note removed: "GENERAL PURPOSE BUTTON"
- note removed: "PROGRAMMING HEADER"
- note removed: "RESET BUTTON"
