File: miniPCB/20/A/20A-20/20A-20.brd (EAGLE design)
At the start: 116 parts, among them J1 XE-1109-001, J2 XE-1109-001, J3 ICSP, J5 105313-1102, J6 105313-1102, K1 RZ03-1A4-D005, U10 TLP181(GB,F), U11 TLP181(GB,F), U2 ADUM1250ARZ, U4 ADUM1250ARZ, U7 ATMEGA328P-AU, U8 VIVA_USB-TTL, U9 TLP181(GB,F)

Commit message: NM.23NOV2024
Parts:
- moved J4 16.0 mm to (95.5, 12.0)
- moved U11 15.0 mm to (63.1, 33.1)
- moved U10 15.0 mm to (63.2, 23.5)
- moved R36 14.2 mm to (57.0, 25.2), turned to 180 degrees
- moved R39 14.0 mm to (56.9, 34.6), turned to 180 degrees
- moved R33 13.3 mm to (40.0, 48.5)
- moved U9 13.3 mm to (45.5, 46.0)
- moved R34 13.3 mm to (70.0, 25.8), turned to 0 degrees
- moved R37 13.3 mm to (70.1, 35.4), turned to 0 degrees
- moved J6 13.0 mm to (90.6, 32.1)
- moved D4 13.0 mm to (72.7, 21.5)
- moved D5 13.0 mm to (72.6, 31.1)
- moved J5 13.0 mm to (90.7, 22.5)
- moved Q2 13.0 mm to (80.7, 21.5)
- moved Q3 13.0 mm to (80.6, 31.1)
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Connections:
- removed net ACTIVE_LOW: R33.1, R36.1, R39.1, U10.1, U11.1, U9.1
- removed net PD5: U7.9
- removed net PD6: U7.10
- removed net PD7: U7.11
- new net DCBUS: R33.1, U7.11, U9.1
- new net FAN: R39.1, U11.1, U7.10
- new net HEATER: R36.1, U10.1, U7.9
- new net N$36: R31.1, U9.6
- new net N$39: R37.1, U11.6
- net GNDB: now also J4.1, J4.2, J4.3, J4.4; no longer U10.4, U11.4, U9.4
- net N$28: now also U10.4; no longer R34.1, U10.6
- net N$29: now also U9.4; no longer R31.1, U9.6
- net N$30: now also D6.C, K1.A2, R31.2
- net N$33: now also U11.4; no longer R37.1, U11.6
- net N$35: now also R34.1, U10.6; no longer J4.1, J4.2, J4.3, J4.4, K1.14.1, K1.14.2
- net V+: now also K1.14.1, K1.14.2; no longer D6.C, K1.A2, R31.2
Routing:
- net N$30: track 0.00 -> 8.04 mm, vias 0 -> 1
- net N$31: track 0.00 -> 7.41 mm
- net ACTIVE_LOW: track 7.10 -> 0.00 mm
- net GNDB: track 25.8 -> 21.2 mm, vias 0 -> 9
- net GND: track 42.6 -> 46.8 mm, vias 18 -> 21
- net N$36: track 0.00 -> 3.84 mm
- net N$39: track 0.00 -> 3.19 mm
- net N$35: track 0.00 -> 3.07 mm
- net DCBUS: track 0.00 -> 2.37 mm
- net HEATER: track 0.00 -> 2.16 mm
- net N$33: track 12.2 -> 10.1 mm
- net N$28: track 12.2 -> 10.1 mm
- net FAN: track 0.00 -> 2.12 mm
- net V+: track 4.65 -> 3.10 mm, vias 3 -> 2
- net VDD: track 44.4 -> 42.9 mm
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- added copper zone on layer 1, net GNDB
- added copper zone on layer 2, net GNDB
- added copper zone on layer 2, net N$30
- added copper zone on layer 15, net V+
Other:
- board text added: "FAN"
- board text added: "HEATER"

Commit message: NM.26NOV2024
Parts:
- added C37, C38, C39, C41, C43, C48, C51, C53, C56, C58: 100n, minipcb:C0402
- added C40, C45, C46: 10u, minipcb:C0805
- added C42, C44, C49, C50, C54, C55, C59: 4u7, minipcb:C0402
- added C47, C52: 470p, minipcb:C0402
- added C57: 4n7, minipcb:C0402
- added FL10, FL9: BLM03HG601SZ1D, minipcb:R0402
- added J8: (no value), utsa:PJ-102A
- added J9: NANOFIT, utsa:PINS_4_NANOFIT_RA
- added P1, P2, P3, P4: (no value), minipcb:BANNAN_JACK_4MM_H
- added R40, R41, R43, R44: 4k7, minipcb:R0402
- added R42, R47, R48, R51, R52: DNP, minipcb:R0402
- added R45, R49: WSL2010R5000DEA, utsa:R5025
- added R46, R50: 22, minipcb:R0402
- added R53, R54: 60, minipcb:R0402
- added R55: 300, minipcb:R0402
- added U12: ADUM1250ARZ, 16A-01:SOIC127P600X175-8N
- added U13: ADUM6280, 16A-01:SOIC127P600X175-8N
- added U14, U16: ADC121C027CIMK, utsa:SOT23-6
- added U15, U17: INA181, utsa:SOT23-6
- added U18: MCP2561FD-E/MF, utsa:SON65P300X300X100-9N
- U6: value (none) -> ADUM6280
Connections:
- new net CAN-RX: U18.4
- new net CAN-STBY: U18.8
- new net CAN-TX: U18.1
- new net CANH: J9.3, R54.2, U18.7
- new net CANL: J9.2, R53.2, U18.6
- new net CURRENT-SENSE+: Q2.3, Q3.3, R45.2, U15.3
- new net CURRENT-SENSE-: J4.1, J4.2, J4.3, J4.4, R45.1, U15.4
- new net ISO-SCL: R41.1, U12.6, U14.5
- new net ISO-SDA: R40.1, U12.7, U14.6
- new net LEAKAGE-CURRENT+: P4.1, P4.2, R49.2, U17.3
- new net LEAKAGE-CURRENT-: P3.1, P3.2, R49.1, U17.4
- new net N$41: R42.2, R43.1, U13.8
- new net N$42: C37.2, FL9.2, U13.5, U13.7
- new net N$43: C37.1, FL10.2, U13.6
- new net N$44: C47.1, R46.2, U14.3
- new net N$45: R46.1, U15.1
- new net N$46: R47.1, R48.1, U14.4
- new net N$47: C52.1, R50.2, U16.3
- new net N$48: R50.1, U17.1
- new net N$49: R51.1, R52.1, U16.4
- new net N$50: J8.TIP
- new net N$51: P1.1, P1.2, P2.1, P2.2
- new net N$52: R55.1, U18.5
- new net N$53: C57.1, R53.1, R54.1, R55.2
- new net VBUS: J9.4
- new net VISO2: C38.1, C41.1, C42.1, C45.1ASD, C48.1, C49.1, C50.1, C51.1, FL10.1, R40.2, R41.2, R43.2, R47.2, U12.8, U14.1, U15.6
- net GND: now also C39.2, C40.2ASDF, C43.2, C44.2, C46.2ASDF, C52.2, C53.2, C54.2, C55.2, C56.2, C57.2, C58.2, C59.2, J8.RING, J9.1, R52.2, U12.4, U13.2, U13.4, U16.2, U17.2, U17.5, U18.2, U18.9
- net GNDB: now also C38.2, C41.2, C42.2, C45.2ASDF, C47.2, C48.2, C49.2, C50.2, C51.2, FL9.1, R42.1, R48.2, U14.2, U15.2, U15.5; no longer J4.1, J4.2, J4.3, J4.4, Q2.3, Q3.3
- net PDIS: now also R44.1, U13.1
- net SCL: now also U12.3, U16.5
- net SDA: now also U12.2, U16.6
- net VDD: now also C39.1, C40.1ASD, C43.1, C44.1, C46.1ASD, C53.1, C54.1, C55.1, C56.1, C58.1, C59.1, R44.2, R51.2, U12.1, U13.3, U16.1, U17.6, U18.3
Routing:
- net GND: track 46.8 -> 80.7 mm, vias 21 -> 31
- net ISO-SDA: track 0.00 -> 25.9 mm, vias 0 -> 2
- net VDD: track 42.9 -> 67.7 mm, vias 13 -> 19
- net ISO-SCL: track 0.00 -> 24.4 mm, vias 0 -> 2
- net VISO2: track 0.00 -> 19.4 mm, vias 0 -> 6
- net GNDB: track 21.2 -> 33.1 mm
- net N$42: track 0.00 -> 8.53 mm, vias 0 -> 2
- net LEAKAGE-CURRENT-: track 0.00 -> 4.60 mm
- net LEAKAGE-CURRENT+: track 0.00 -> 4.60 mm
- net CANH: track 0.00 -> 4.36 mm, vias 0 -> 1
- net CURRENT-SENSE-: track 0.00 -> 3.87 mm
- net CURRENT-SENSE+: track 0.00 -> 3.87 mm
- net N$44: track 0.00 -> 3.34 mm
- net N$47: track 0.00 -> 3.34 mm
- net N$41: track 0.00 -> 3.28 mm
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- added copper zone on layer 1, net CURRENT-SENSE+
- added copper zone on layer 1, net CURRENT-SENSE-
- added copper zone on layer 1, net LEAKAGE-CURRENT+
- added copper zone on layer 1, net LEAKAGE-CURRENT-
- added copper zone on layer 1, net N$51
- added copper zone on layer 15, net VISO2
- removed copper zone on layer 1, net GNDB
Other:
- board text added: "DC+(1)"
- board text added: "DC+(2)"
- board text added: "DC-(1)"
- board text added: "DC-(2)"
- board text added: "DUT+"
- board text added: "DUT-"
