File: miniPCB/20/A/20A-20/20A-20.sch (EAGLE design)
At the start: 116 parts, among them J1 XE-1109-001, J2 XE-1109-001, J3 ICSP, J5 105313-1102, J6 105313-1102, K1 RZ03-1A4-D005, U10 TLP181(GB,F), U11 TLP181(GB,F), U2 ADUM1250ARZ, U4 ADUM1250ARZ, U7 ATMEGA328P-AU, U8 VIVA_USB-TTL, U9 TLP181(GB,F)

Commit message: NM.23NOV2024
Connections:
- removed net ACTIVE_LOW: R33.1, R36.1, R39.1, U10.A, U11.A, U9.A
- removed net PD5: U7.PD5
- removed net PD6: U7.PD6
- removed net PD7: U7.PD7
- new net DCBUS: R33.1, U7.PD7, U9.A
- new net FAN: R39.1, U11.A, U7.PD6
- new net HEATER: R36.1, U10.A, U7.PD5
- new net N$36: R31.1, U9.CT
- new net N$39: R37.1, U11.CT
- net GNDB: now also J4.1; no longer U10.ET, U11.ET, U9.ET
- net N$28: now also U10.ET; no longer R34.1, U10.CT
- net N$29: now also U9.ET; no longer R31.1, U9.CT
- net N$30: now also D6.C, K1.A2, R31.2
- net N$33: now also U11.ET; no longer R37.1, U11.CT
- net N$35: now also R34.1, U10.CT; no longer J4.1, K1.14
- net V+: now also K1.14; no longer D6.C, K1.A2, R31.2
Other:
- moved on the sheet: D4, D5, J4, J5, J6, Q2, Q3, R31, R33, R34, R35, R36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

Commit message: NM.26NOV2024
Parts:
- added C37, C38, C39, C41, C43, C48, C51, C53, C56, C58: 100n, minipcb:CAPACITOR0402
- added C40, C45, C46: 10u, minipcb:CAPACITORSMD
- added C42, C44, C49, C50, C54, C55, C59: 4u7, minipcb:CAPACITOR0402
- added C47, C52: 470p, minipcb:CAPACITOR0402
- added C57: 4n7, minipcb:CAPACITOR0402
- added FL10, FL9: BLM03HG601SZ1D, minipcb:BLM03HG601SZ1D
- added J8: (no value), utsa:2.1MMJACKTHM
- added J9: NANOFIT, utsa:PINS_4-NANOFIT
- added P1, P2, P3, P4: (no value), minipcb:PINS_1571-0500
- added R40, R41, R43, R44: 4k7, minipcb:RESISTOR0402
- added R42, R47, R48, R51, R52: DNP, minipcb:RESISTOR0402
- added R45, R49: WSL2010R5000DEA, utsa:R-EU_R5025
- added R46, R50: 22, minipcb:RESISTOR0402
- added R53, R54: 60, minipcb:RESISTOR0402
- added R55: 300, minipcb:RESISTOR0402
- added U12: ADUM1250ARZ, 16A-01:ADUM1250ARZ
- added U13: ADUM6280, 16A-01:ADUM6280
- added U14, U16: ADC121C027CIMK, utsa:ADC121C027CIMK
- added U15, U17: INA181, utsa:INAX81
- added U18: MCP2561FD-E/MF, utsa:MCP2561FD-E/MF
- U6: value (none) -> ADUM6280
Connections:
- new net CAN-RX: U18.RX
- new net CAN-STBY: U18.STBY
- new net CAN-TX: U18.TX
- new net CANH: J9.3, R54.2, U18.CANH
- new net CANL: J9.2, R53.2, U18.CANL
- new net CURRENT-SENSE+: Q2.S, Q3.S, R45.2, U15.3.IN+
- new net CURRENT-SENSE-: J4.1, R45.1, U15.4.IN-
- new net ISO-SCL: R41.1, U12.SCL2, U14.5.SCL
- new net ISO-SDA: R40.1, U12.SDA2, U14.6.SDA
- new net LEAKAGE-CURRENT+: P4.1, R49.2, U17.3.IN+
- new net LEAKAGE-CURRENT-: P3.1, R49.1, U17.4.IN-
- new net N$41: R42.2, R43.1, U13.VSEL
- new net N$42: C37.-, FL9.2, U13.GNDISO
- new net N$43: C37.+, FL10.2, U13.VISO
- new net N$44: C47.+, R46.2, U14.3.VIN
- new net N$45: R46.1, U15.1.OUT
- new net N$46: R47.1, R48.1, U14.4.ADDR
- new net N$47: C52.+, R50.2, U16.3.VIN
- new net N$48: R50.1, U17.1.OUT
- new net N$49: R51.1, R52.1, U16.4.ADDR
- new net N$50: J8.TIP
- new net N$51: P1.1, P2.1
- new net N$52: R55.1, U18.SPLIT
- new net N$53: C57.+, R53.1, R54.1, R55.2
- new net VBUS: J9.4
- new net VISO2: C38.+, C41.+, C42.+, C45.+, C48.+, C49.+, C50.+, C51.+, FL10.1, R40.2, R41.2, R43.2, R47.2, U12.VDD2, U14.1.VA, U15.6.VS
- net GND: now also C39.-, C40.-, C43.-, C44.-, C46.-, C52.-, C53.-, C54.-, C55.-, C56.-, C57.-, C58.-, C59.-, J8.RING, J9.1, R52.2, U12.GND1, U13.GND1, U16.2.GND, U17.2.GND, U17.5.REF, U18.VSS
- net GNDB: now also C38.-, C41.-, C42.-, C45.-, C47.-, C48.-, C49.-, C50.-, C51.-, FL9.1, R42.1, R48.2, U14.2.GND, U15.2.GND, U15.5.REF; no longer J4.1, Q2.S, Q3.S
- net PDIS: now also R44.1, U13.PDIS
- net SCL: now also U12.SCL1, U16.5.SCL
- net SDA: now also U12.SDA1, U16.6.SDA
- net VDD: now also C39.+, C40.+, C43.+, C44.+, C46.+, C53.+, C54.+, C55.+, C56.+, C58.+, C59.+, R44.2, R51.2, U12.VDD1, U13.VDDP, U16.1.VA, U17.6.VS, U18.VDD
